Commit message: add arm glb

File: galbot_foxtrot_description/xacro/arm.xacro (robot description, xacro)
@@ -20,5 +20,5 @@
 			<visual>
 				<geometry>
-					<mesh filename="file://$(find galbot_foxtrot_description)/meshes/visual/arm/link1.obj"
+					<mesh filename="file://$(find galbot_foxtrot_description)/meshes/visual/arm/link1.glb"
 								scale="1 ${direction} 1"/>
 				</geometry>
@@ -49,5 +49,5 @@
 				<geometry>
 					<mesh
-							filename="file://$(find galbot_foxtrot_description)/meshes/visual/arm/link2.obj"
+							filename="file://$(find galbot_foxtrot_description)/meshes/visual/arm/link2.glb"
 							scale="1 ${direction} 1"/>
 				</geometry>
@@ -76,5 +76,5 @@
 			<visual>
 				<geometry>
-					<mesh filename="file://$(find galbot_foxtrot_description)/meshes/visual/arm/link3.obj"
+					<mesh filename="file://$(find galbot_foxtrot_description)/meshes/visual/arm/link3.glb"
 								scale="1 ${direction} 1"/>
 				</geometry>
@@ -103,5 +103,5 @@
 			<visual>
 				<geometry>
-					<mesh filename="file://$(find galbot_foxtrot_description)/meshes/visual/arm/link4.obj"
+					<mesh filename="file://$(find galbot_foxtrot_description)/meshes/visual/arm/link4.glb"
 								scale="1 ${direction} 1"/>
 				</geometry>
@@ -131,5 +131,5 @@
 				<geometry>
 					<mesh
-							filename="file://$(find galbot_foxtrot_description)/meshes/visual/arm/link5.obj"/>
+							filename="file://$(find galbot_foxtrot_description)/meshes/visual/arm/link5.glb"/>
 				</geometry>
 			</visual>
@@ -157,5 +157,5 @@
 			<visual>
 				<geometry>
-					<mesh filename="file://$(find galbot_foxtrot_description)/meshes/visual/arm/link6.obj"
+					<mesh filename="file://$(find galbot_foxtrot_description)/meshes/visual/arm/link6.glb"
 								scale="1 ${direction} 1"/>
 				</geometry>
@@ -184,5 +184,5 @@
 			<visual>
 				<geometry>
-					<mesh filename="file://$(find galbot_foxtrot_description)/meshes/visual/arm/link7.obj"
+					<mesh filename="file://$(find galbot_foxtrot_description)/meshes/visual/arm/link7.glb"
 								scale="1 ${direction} 1"/>
 				</geometry>
@@ -202,9 +202,9 @@
 			<limit acceleration="2" effort="10" jerk="12" lower="-1.5382" upper="1.5382" velocity="1.5"/>
 		</joint>
-		<joint name="${prefix}camera_joint" type="fixed">
+		<joint name="${prefix}camera_stand_joint" type="fixed">
 			<parent link="${prefix}link7"/>
-			<child link="${prefix}wrist_camera_link"/>
-		</joint>
-		<link name="${prefix}wrist_camera_link">
+			<child link="${prefix}wrist_camera_stand"/>
+		</joint>
+		<link name="${prefix}wrist_camera_stand">
 			<inertial>
 				<origin xyz="-0.0621229724155358 -0.0628379837355285 -0.00140310958315455"/>
@@ -215,11 +215,5 @@
 			<visual>
 				<geometry>
-					<mesh filename="file://$(find galbot_foxtrot_description)/meshes/visual/arm/d405_stand.obj"/>
-				</geometry>
-			</visual>
-			<visual>
-				<origin xyz="-0.0822 0 -0.06842" rpy="-1.5708 3.2315926 0"/>
-				<geometry>
-					<mesh filename="file://$(find sensor_models)/meshes/d405/d405.obj"/>
+					<mesh filename="file://$(find galbot_foxtrot_description)/meshes/visual/arm/d405_stand.glb"/>
 				</geometry>
 			</visual>
@@ -229,4 +223,16 @@
 				</geometry>
 			</collision>
+		</link>
+		<joint name="${prefix}camera_joint" type="fixed">
+			<origin xyz="-0.0822 0 -0.06842" rpy="0 ${PI/2 - 0.09} ${PI}"/>
+			<parent link="${prefix}wrist_camera_stand"/>
+			<child link="${prefix}wrist_camera"/>
+		</joint>
+		<link name="${prefix}wrist_camera">
+			<visual>
+				<geometry>
+					<mesh filename="file://$(find sensor_models)/meshes/realsense/d405.glb"/>
+				</geometry>
+			</visual>
 		</link>
 	</xacro:macro>
