Commit message: add ros2 control support for golf

File: galbot_foxtrot_description/xacro/component.xacro (robot description, xacro)
@@ -1,4 +1,4 @@
 <?xml version="1.0" ?>
-<robot name="Hitbot Gripper" xmlns:xacro="http://www.ros.org/wiki/xacro">
+<robot name="Arms_Default" xmlns:xacro="http://www.ros.org/wiki/xacro">
   <xacro:property name="PI" value="3.141592653589793"/>
   <xacro:arg name="type" default="base"/>
@@ -28,26 +28,24 @@
     <xacro:include filename="$(find galbot_one_description)/xacro/components/body.xacro"/>
   </xacro:if>
+  <xacro:if value="${'$(arg type)' == 'head'}">
+    <link name="base_link"/>
+    <xacro:include filename="$(find galbot_foxtrot_description)/xacro/components/head.xacro"/>
+    <xacro:galbot_foxtrot_head parent_link="base_link"/>
+  </xacro:if>
   <xacro:if value="${'$(arg type)' == 'arm'}">
-    <!-- Use a single base_link as root to avoid multiple roots for robot_state_publisher -->
-    <link name="base_link"/>
-    <joint name="arm_base_joint" type="fixed">
-      <origin rpy="${PI/2} 0 0"/>
-      <parent link="base_link"/>
-      <child link="arm_base"/>
-    </joint>
+    <xacro:include filename="$(find galbot_foxtrot_description)/xacro/components/arm.xacro"/>
     <link name="arm_base"/>
-    <joint name="left_arm_mount_joint" type="fixed">
-      <origin rpy="0 ${PI} 0" xyz="0 0 -0.13"/>
+    <joint name="torso_left_mount_joint" type="fixed">
+      <origin rpy="0 1.5707963267948966 0" xyz="0.20843 0 0"/>
       <parent link="arm_base"/>
       <child link="left_base_link"/>
     </joint>
-    <joint name="right_arm_mount_joint" type="fixed">
-      <origin  xyz="0 0 0.13"/>
+    <joint name="torso_right_mount_joint" type="fixed">
+      <origin rpy="3.141592653589793 1.5707963267948966 0" xyz="-0.20843 0 0"/>
       <parent link="arm_base"/>
       <child link="right_base_link"/>
     </joint>
-    <xacro:include filename="$(find galbot_one_description)/xacro/components/arm.xacro"/>
-    <xacro:galbot_one_arm name="left" direction="1"/>
-    <xacro:galbot_one_arm name="right" direction="-1"/>
+    <xacro:Arm name="right" direction="-1" camera="none"/>
+    <xacro:Arm name="left" camera="none"/>
   </xacro:if>
 </robot>

File: galbot_foxtrot_description/xacro/components/body.xacro (robot description, xacro)
@@ -3,4 +3,5 @@
 	<xacro:property name="PI" value="3.141592653589793"/>
 	<xacro:property name="collider_type" value="$(arg collider)"/>
+	<xacro:arg name="enable_joint5" default="false"/>
 <joint name="leg_joint" type="fixed">
 		<parent link="omni_chassis_leg_mount_link"/>
@@ -32,5 +33,5 @@
 	</link>
 	<joint name="body_joint1" type="revolute">
-		<origin rpy="1.5707963267948966 -0.385 3.141592653589793"/>
+		<origin rpy="${PI/2} -0.385 ${PI}"/>
 		<parent link="leg_base_link"/>
 		<child link="leg_link1"/>
@@ -57,5 +58,5 @@
 	</link>
 	<joint name="body_joint2" type="revolute">
-		<origin rpy="3.141592653589793 0 2.7566" xyz="0.45 0 0"/>
+		<origin rpy="${PI} 0 2.7566" xyz="0.45 0 0"/>
 		<parent link="leg_link1"/>
 		<child link="leg_link2"/>
@@ -81,5 +82,5 @@
 	</link>
 	<joint name="body_joint3" type="revolute">
-		<origin rpy="3.141592653589793 0 3.141592653589793" xyz="0.39 0 0"/>
+		<origin rpy="${PI} 0 ${PI}" xyz="0.39 0 0"/>
 		<parent link="leg_link2"/>
 		<child link="leg_link3"/>
@@ -100,5 +101,5 @@
 	</link>
 	<joint name="body_joint4" type="revolute">
-		<origin rpy="-1.5707963267948966 -1.5707963267948966 0" xyz="0 0.224 0"/>
+		<origin rpy="-${PI/2} -${PI/2} 0" xyz="0 0.224 0"/>
 		<parent link="leg_link3"/>
 		<child link="leg_link4"/>
@@ -106,16 +107,39 @@
 		<limit effort="30" lower="-1.5906" upper="1.5906" velocity="1"/>
 	</joint>
-	<link name="leg_end_effector_mount_link">
-		<inertial>
-			<origin xyz="0.0 0.032369999999999996 0.03006"/>
-			<mass value="0.41"/>
-			<inertia ixx="0.00142201" ixy="0.0" ixz="0.0" iyy="0.00132398" iyz="0.00023940999999999999" izz="0.00156199"/>
-		</inertial>
-	</link>
-	<joint name="leg_end_effector_mount_joint" type="fixed">
-		<origin rpy="1.5707963267948966 0 0"/>
-		<parent link="leg_link4"/>
-		<child link="leg_end_effector_mount_link"/>
-	</joint>
+	<xacro:if value="$(arg enable_joint5)">
+		<link name="leg_link5">
+			<inertial>
+				<origin xyz="0.0 0.032369999999999996 0.03006"/>
+				<mass value="0.41"/>
+				<inertia ixx="0.00142201" ixy="0.0" ixz="0.0" iyy="0.00132398" iyz="0.00023940999999999999" izz="0.00156199"/>
+			</inertial>
+		</link>
+		<joint name="body_joint5" type="revolute">
+			<origin rpy="${PI/2} 0 0"/>
+			<parent link="leg_link4"/>
+			<child link="leg_link5"/>
+			<axis xyz="0 0 1"/>
+			<limit effort="30" lower="-0.1645" upper="0.1645" velocity="1"/>
+		</joint>
+		<link name="leg_end_effector_mount_link"/>
+		<joint name="leg_end_effector_mount_joint" type="fixed">
+			<parent link="leg_link5"/>
+			<child link="leg_end_effector_mount_link"/>
+		</joint>
+	</xacro:if>
+	<xacro:unless value="$(arg enable_joint5)">
+		<link name="leg_end_effector_mount_link">
+			<inertial>
+				<origin xyz="0.0 0.032369999999999996 0.03006"/>
+				<mass value="0.41"/>
+				<inertia ixx="0.00142201" ixy="0.0" ixz="0.0" iyy="0.00132398" iyz="0.00023940999999999999" izz="0.00156199"/>
+			</inertial>
+		</link>
+		<joint name="leg_end_effector_mount_joint" type="fixed">
+			<origin rpy="${PI/2} 0 0"/>
+			<parent link="leg_link4"/>
+			<child link="leg_end_effector_mount_link"/>
+		</joint>
+	</xacro:unless>
 	<joint name="torso_joint" type="fixed">
 		<parent link="leg_end_effector_mount_link"/>
@@ -140,79 +164,3 @@
 		</collision>
 	</link>
-	<!-- Head Mount -->
-	<link name="torso_head_mount_link"/>
-	<joint name="torso_head_mount_joint" type="fixed">
-		<origin rpy="-1.5707963267948966 -1.5707963267948966 0" xyz="0 0.36211 0"/>
-		<parent link="torso_base_link"/>
-		<child link="torso_head_mount_link"/>
-		<axis/>
-	</joint>
-	<joint name="head_joint" type="fixed">
-		<parent link="torso_head_mount_link"/>
-		<child link="head_base_link"/>
-	</joint>
-	<link name="head_base_link">
-		<inertial>
-			<origin xyz="0.023809999999999998 0.00032 0.01966"/>
-			<mass value="0.48"/>
-			<inertia ixx="0.0032910599999999997" ixy="8.32e-06" ixz="0.00044358" iyy="0.00375998" iyz="7.18e-06"
-							 izz="0.00221683"/>
-		</inertial>
-	</link>
-	<link name="head_link1">
-		<inertial>
-			<origin xyz="-2e-05 0.00709 -0.0559"/>
-			<mass value="0.08"/>
-			<inertia ixx="0.0003544" ixy="0.0" ixz="1.6e-07" iyy="0.00034029000000000004" iyz="-1.041e-05" izz="6.652e-05"/>
-		</inertial>
-	</link>
-	<joint name="head_joint1" type="revolute">
-		<parent link="head_base_link"/>
-		<child link="head_link1"/>
-		<axis xyz="0 0 1"/>
-		<limit effort="4" lower="-1.5208" upper="1.5208" velocity="1.5"/>
-	</joint>
-	<link name="head_link2">
-		<inertial>
-			<origin xyz="0.01835 -0.033479999999999996 0.00642"/>
-			<mass value="0.08"/>
-			<inertia ixx="0.00019294" ixy="-6.442e-05" ixz="1.0900000000000002e-06" iyy="0.00015263999999999998"
-							 iyz="-4.09e-06" izz="0.00018457"/>
-		</inertial>
-		<visual>
-			<geometry>
-				<mesh filename="file://$(find galbot_foxtrot_description)/meshes/visual/head/head.glb"/>
-			</geometry>
-		</visual>
-		<collision>
-			<geometry>
-				<mesh filename="file://$(find galbot_foxtrot_description)/meshes/collision/head.stl"/>
-			</geometry>
-		</collision>
-	</link>
-	<joint name="head_joint2" type="revolute">
-		<origin rpy="-1.5707963267948966 0 0"/>
-		<parent link="head_link1"/>
-		<child link="head_link2"/>
-		<axis xyz="0 0 1"/>
-		<limit effort="4" lower="-0.321147949" upper="0.321147949" velocity="1.5"/>
-	</joint>
-	<link name="head_end_effector_mount_link"/>
-	<joint name="head_end_effector_mount_joint" type="fixed">
-		<parent link="head_link2"/>
-		<child link="head_end_effector_mount_link"/>
-		<axis/>
-	</joint>
-	<link name="head_front_camera">
-		<visual>
-			<geometry>
-				<mesh filename="file://$(find sensor_models)/meshes/realsense/d435.glb"/>
-			</geometry>
-		</visual>
-	</link>
-	<joint name="head_front_camera_joint" type="fixed">
-		<origin rpy="-${PI*29/180} ${PI/2} 0" xyz="0.088405 -0.05399 0"/>
-		<parent link="head_link2"/>
-		<child link="head_front_camera"/>
-	</joint>
 </robot>

File: galbot_foxtrot_description/xacro/robot.xacro (robot description, xacro)
@@ -6,26 +6,20 @@
 	<xacro:include filename="$(find galbot_foxtrot_description)/xacro/components/galbot_gripper.xacro"/>
 	<xacro:include filename="$(find galbot_foxtrot_description)/xacro/components/body.xacro"/>
+	<xacro:include filename="$(find galbot_foxtrot_description)/xacro/components/head.xacro"/>
 	<xacro:include filename="$(find galbot_foxtrot_description)/xacro/components/arm.xacro"/>
 	<xacro:include filename="$(find galbot_foxtrot_description)/xacro/components/chassis.xacro"/>
 	<xacro:GalbotChassisV2 enable_wheel_joints="$(arg enable_wheel_joints)"/>
-	<!-- Left Arm Mount -->
-	<link name="torso_left_mount_link"/>
+	<xacro:galbot_foxtrot_head parent_link="torso_base_link"/>
 	<joint name="torso_left_mount_joint" type="fixed">
 		<origin rpy="0 1.5707963267948966 0" xyz="0.20843 0.172 0"/>
 		<parent link="torso_base_link"/>
-		<child link="torso_left_mount_link"/>
+		<child link="left_base_link"/>
 		<axis/>
 	</joint>
-	<!-- Right Arm Mount -->
-	<link name="torso_right_mount_link"/>
 	<joint name="torso_right_mount_joint" type="fixed">
 		<origin rpy="3.141592653589793 1.5707963267948966 0" xyz="-0.20843 0.172 0"/>
 		<parent link="torso_base_link"/>
-		<child link="torso_right_mount_link"/>
+		<child link="right_base_link"/>
 		<axis/>
-	</joint>
-	<joint name="right_joint" type="fixed">
-		<parent link="torso_right_mount_link"/>
-		<child link="right_base_link"/>
 	</joint>
 	<xacro:Arm name="right" direction="-1" camera="$(arg arm_camera)"/>
@@ -37,8 +31,4 @@
 	</joint>
 	<xacro:Gripper name="right"/>
-	<joint name="left_joint" type="fixed">
-		<parent link="torso_left_mount_link"/>
-		<child link="left_base_link"/>
-	</joint>
 	<xacro:Arm name="left" camera="$(arg arm_camera)"/>
 	<joint name="left_end_effector_mount_joint" type="fixed">
