Commit message: add ros2 control support for golf

File: galbot_golf_description/urdf/galbot_golf.urdf (robot description, URDF)
Before this commit: robot galbot_one_golf, 55 links, 54 joints
Links:
- removed link left_arm_base_link
- removed link left_arm_link1
- removed link left_arm_link2
- removed link left_arm_link3
- removed link left_arm_link4
- removed link left_arm_link5
- removed link left_arm_link6
- removed link left_arm_link7
- removed link left_wrist_camera_link
- removed link right_arm_base_link
- removed link right_arm_link1
- removed link right_arm_link2
- removed link right_arm_link3
- removed link right_arm_link4
- removed link right_arm_link5
- removed link right_arm_link6
- removed link right_arm_link7
- removed link right_wrist_camera_link
- removed link torso_center_link
- added link chassis_lidar; visual mesh filename=package://sensor_models/meshes/mid360/mid360.obj
- added link left_base_link, mass 0.92
- added link left_link1, mass 1.6; collision mesh filename=package://galbot_foxtrot_description/meshes/collision/arm/l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 scale=1 1 1; visual mesh filename=package://galbot_foxtrot_description/meshes/visual/arm/link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 scale=1 1 1
- added link left_link2, mass 1.43; collision mesh filename=package://galbot_foxtrot_description/meshes/collision/arm/l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 scale=1 1 1; visual mesh filename=package://galbot_foxtrot_description/meshes/visual/arm/link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
- added link left_link3, mass 1.43; collision mesh filename=package://galbot_foxtrot_description/meshes/collision/arm/l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 scale=1 1 1; visual mesh filename=package://galbot_foxtrot_description/meshes/visual/arm/link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 scale=1 1 1
- added link left_link4, mass 1.1; collision mesh filename=package://galbot_foxtrot_description/meshes/collision/arm/l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 scale=1 1 1; visual mesh filename=package://galbot_foxtrot_description/meshes/visual/arm/link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 scale=1 1 1
- added link left_link5, mass 1.15; collision mesh filename=package://galbot_foxtrot_description/meshes/collision/arm/l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; visual mesh filename=package://galbot_foxtrot_description/meshes/visual/arm/link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
- added link left_link6, mass 0.47; collision mesh filename=package://galbot_foxtrot_description/meshes/collision/arm/l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 scale=1 1 1; visual mesh filename=package://galbot_foxtrot_description/meshes/visual/arm/link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 scale=1 1 1
- added link left_link7, mass 0.8; collision mesh filename=package://galbot_foxtrot_description/meshes/collision/arm/l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 scale=1 1 1; visual mesh filename=package://galbot_foxtrot_description/meshes/visual/arm/link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 scale=1 1 1
- added link left_wrist_camera; visual mesh filename=package://sensor_models/meshes/realsense/d405.glb
- added link left_wrist_camera_stand, mass 0.0492751941348016; visual mesh filename=package://galbot_foxtrot_description/meshes/visual/arm/d405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
- added link right_base_link, mass 0.92
- added link right_link1, mass 1.6; collision mesh filename=package://galbot_foxtrot_description/meshes/collision/arm/l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 scale=1 -1 1; visual mesh filename=package://galbot_foxtrot_description/meshes/visual/arm/link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 scale=1 -1 1
- added link right_link2, mass 1.43; collision mesh filename=package://galbot_foxtrot_description/meshes/collision/arm/l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 scale=1 -1 1; visual mesh filename=package://galbot_foxtrot_description/meshes/visual/arm/link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
- added link right_link3, mass 1.43; collision mesh filename=package://galbot_foxtrot_description/meshes/collision/arm/l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 scale=1 -1 1; visual mesh filename=package://galbot_foxtrot_description/meshes/visual/arm/link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 scale=1 -1 1
- added link right_link4, mass 1.1; collision mesh filename=package://galbot_foxtrot_description/meshes/collision/arm/l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 scale=1 -1 1; visual mesh filename=package://galbot_foxtrot_description/meshes/visual/arm/link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 scale=1 -1 1
- added link right_link5, mass 1.15; collision mesh filename=package://galbot_foxtrot_description/meshes/collision/arm/l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; visual mesh filename=package://galbot_foxtrot_description/meshes/visual/arm/link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
- added link right_link6, mass 0.47; collision mesh filename=package://galbot_foxtrot_description/meshes/collision/arm/l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 scale=1 -1 1; visual mesh filename=package://galbot_foxtrot_description/meshes/visual/arm/link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 scale=1 -1 1
- added link right_link7, mass 0.8; collision mesh filename=package://galbot_foxtrot_description/meshes/collision/arm/l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 scale=1 -1 1; visual mesh filename=package://galbot_foxtrot_description/meshes/visual/arm/link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 scale=1 -1 1
- added link right_wrist_camera; visual mesh filename=package://sensor_models/meshes/realsense/d405.glb
- added link right_wrist_camera_stand, mass 0.0492751941348016; visual mesh filename=package://galbot_foxtrot_description/meshes/visual/arm/d405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
- added link wheel_1, mass 4.24803000494366; visual mesh filename=package://component_models/meshes/omniwheel_10.glb
- added link wheel_2, mass 4.24803000494366; visual mesh filename=package://component_models/meshes/omniwheel_10.glb
- added link wheel_3, mass 4.24803000494366; visual mesh filename=package://component_models/meshes/omniwheel_10.glb
- added link wheel_4, mass 4.24803000494366; visual mesh filename=package://component_models/meshes/omniwheel_10.glb
- link head_link2: geometry collision mesh filename=package://galbot_golf_description/meshes/collision/head.stl; visual mesh filename=package://galbot_golf_description/meshes/visual/head/head.g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
- link left_gripper_base: geometry collision mesh filename=package://galbot_foxtrot_description/meshes/collision/gripp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; visual mesh filename=package://galbot_foxtrot_description/meshes/visual/gripper/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
- link left_gripper_flange: geometry visual mesh filename=package://galbot_foxtrot_description/meshes/visual/gripper/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
- link left_gripper_l_finger_link: geometry collision mesh filename=package://galbot_foxtrot_description/meshes/collision/gripp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; visual mesh filename=package://galbot_foxtrot_description/meshes/visual/gripper/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
- link left_gripper_l_inner_knuckle_link: geometry collision mesh filename=package://galbot_foxtrot_description/meshes/collision/gripp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; visual mesh filename=package://galbot_foxtrot_description/meshes/visual/gripper/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
- link left_gripper_l_knuckle_link: geometry collision mesh filename=package://galbot_foxtrot_description/meshes/collision/gripp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; visual mesh filename=package://galbot_foxtrot_description/meshes/visual/gripper/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
- link left_gripper_r_finger_link: geometry collision mesh filename=package://galbot_foxtrot_description/meshes/collision/gripp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 scale=1 -1 1; visual mesh filename=package://galbot_foxtrot_description/meshes/visual/gripper/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 scale=1 -1 1
- link left_gripper_r_inner_knuckle_link: geometry collision mesh filename=package://galbot_foxtrot_description/meshes/collision/gripp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; visual mesh filename=package://galbot_foxtrot_description/meshes/visual/gripper/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
- link left_gripper_r_knuckle_link: geometry collision mesh filename=package://galbot_foxtrot_description/meshes/collision/gripp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; visual mesh filename=package://galbot_foxtrot_description/meshes/visual/gripper/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
- link leg_link1: geometry collision mesh filename=package://galbot_foxtrot_description/meshes/collision/leg/l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; visual mesh filename=package://galbot_foxtrot_description/meshes/visual/leg/leg1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
- link leg_link2: geometry collision mesh filename=package://galbot_foxtrot_description/meshes/collision/leg/l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; visual mesh filename=package://galbot_foxtrot_description/meshes/visual/leg/leg2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
- link leg_link3: geometry collision mesh filename=package://galbot_foxtrot_description/meshes/collision/leg/l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; visual mesh filename=package://galbot_foxtrot_description/meshes/visual/leg/leg3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
- link leg_link4: geometry visual mesh filename=package://galbot_foxtrot_description/meshes/visual/leg/leg4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
- link leg_link5: geometry 
- link omni_chassis_base_link: mass 8.04 -> 8.7914; geometry collision cylinder length=0.2 radius=0.3; visual mesh filename=package://galbot_foxtrot_description/meshes/visual/chassis/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
- link right_gripper_base: geometry collision mesh filename=package://galbot_foxtrot_description/meshes/collision/gripp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; visual mesh filename=package://galbot_foxtrot_description/meshes/visual/gripper/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
- link right_gripper_flange: geometry visual mesh filename=package://galbot_foxtrot_description/meshes/visual/gripper/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
- link right_gripper_l_finger_link: geometry collision mesh filename=package://galbot_foxtrot_description/meshes/collision/gripp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; visual mesh filename=package://galbot_foxtrot_description/meshes/visual/gripper/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
- link right_gripper_l_inner_knuckle_link: geometry collision mesh filename=package://galbot_foxtrot_description/meshes/collision/gripp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; visual mesh filename=package://galbot_foxtrot_description/meshes/visual/gripper/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
- link right_gripper_l_knuckle_link: geometry collision mesh filename=package://galbot_foxtrot_description/meshes/collision/gripp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; visual mesh filename=package://galbot_foxtrot_description/meshes/visual/gripper/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
- link right_gripper_r_finger_link: geometry collision mesh filename=package://galbot_foxtrot_description/meshes/collision/gripp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 scale=1 -1 1; visual mesh filename=package://galbot_foxtrot_description/meshes/visual/gripper/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 scale=1 -1 1
- link right_gripper_r_inner_knuckle_link: geometry collision mesh filename=package://galbot_foxtrot_description/meshes/collision/gripp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; visual mesh filename=package://galbot_foxtrot_description/meshes/visual/gripper/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
- link right_gripper_r_knuckle_link: geometry collision mesh filename=package://galbot_foxtrot_description/meshes/collision/gripp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; visual mesh filename=package://galbot_foxtrot_description/meshes/visual/gripper/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
- link torso_base_link: geometry collision mesh filename=package://galbot_foxtrot_description/meshes/collision/torso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; visual mesh filename=package://galbot_foxtrot_description/meshes/visual/torso/to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
Joints:
- removed joint left_arm_joint1
- removed joint left_arm_joint2
- removed joint left_arm_joint3
- removed joint left_arm_joint4
- removed joint left_arm_joint5
- removed joint left_arm_joint6
- removed joint left_arm_joint7
- removed joint leg_joint1
- removed joint leg_joint2
- removed joint leg_joint3
- removed joint leg_joint4
- removed joint leg_joint5
- removed joint right_arm_joint1
- removed joint right_arm_joint2
- removed joint right_arm_joint3
- removed joint right_arm_joint4
- removed joint right_arm_joint5
- removed joint right_arm_joint6
- removed joint right_arm_joint7
- removed joint torso_center_joint
- added joint body_joint1: type revolute, parent leg_base_link, child leg_link1, origin rpy=1.5707963267948966 -0.385 3.141592653589793, axis 0 0 1, limit lower=0.0 upper=0.9374 effort=169 velocity=1
- added joint body_joint2: type revolute, parent leg_link1, child leg_link2, origin xyz=0.45 0 0 rpy=3.141592653589793 0 2.7566, axis 0 0 1, limit lower=0.0 upper=2.5847 effort=169 velocity=1
- added joint body_joint3: type revolute, parent leg_link2, child leg_link3, origin xyz=0.39 0 0 rpy=3.141592653589793 0 3.141592653589793, axis 0 0 1, limit lower=0.0 upper=2.3262 effort=84 velocity=1
- added joint body_joint4: type revolute, parent leg_link3, child leg_link4, origin xyz=0 0.224 0 rpy=-1.5707963267948966 -1.5707963267948966 0, axis 0 0 1, limit lower=-1.5906 upper=1.5906 effort=30 velocity=1
- added joint body_joint5: type revolute, parent leg_link4, child leg_link5, origin rpy=1.5707963267948966 0 0, axis 0 0 1, limit lower=-0.1645 upper=0.1645 effort=30 velocity=1
- added joint chassis_lidar_joint: type fixed, parent omni_chassis_base_link, child chassis_lidar, origin xyz=0.235 0 0.2144
- added joint left_camera_stand_joint: type fixed, parent left_link7, child left_wrist_camera_stand
- added joint left_joint1: type revolute, parent left_base_link, child left_link1, origin rpy=0 0 0.523598775598286, axis 0 0 1, limit lower=-3.0043 upper=3.0043 effort=60 velocity=1.5
- added joint left_joint2: type revolute, parent left_link1, child left_link2, origin rpy=1.5707963267949 0 3.14159265358979, axis 0 0 1, limit lower=-1.6081 upper=1.6081 effort=60 velocity=1.5
- added joint left_joint3: type revolute, parent left_link2, child left_link3, origin xyz=0 0.35 0 rpy=1.5707963267949 1.04719755119629 -3.14159265358979, axis 0 0 1, limit lower=-2.91697 upper=2.91697 effort=30 velocity=1.5
- added joint left_joint4: type revolute, parent left_link3, child left_link4, origin rpy=1.57079632679459 0 3.14159265358979, axis 0 0 -1, limit lower=-1.86986 upper=2.56799 effort=30 velocity=1.5
- added joint left_joint5: type revolute, parent left_link4, child left_link5, origin xyz=0 0.36 0 rpy=-1.5707963267949 0 0.0, axis 0 0 1, limit lower=-2.91697 upper=2.91697 effort=10 velocity=1.5
- added joint left_joint6: type revolute, parent left_link5, child left_link6, origin rpy=1.5707963267949 1.5707963267949 0, axis 0 0 1, limit lower=-0.7354 upper=0.8227 effort=10 velocity=1.5
- added joint left_joint7: type revolute, parent left_link6, child left_link7, origin rpy=1.5707963267949 0 0, axis 0 0 1, limit lower=-1.5382 upper=1.5382 effort=10 velocity=1.5
- added joint right_camera_stand_joint: type fixed, parent right_link7, child right_wrist_camera_stand
- added joint right_joint1: type revolute, parent right_base_link, child right_link1, origin rpy=0 0 -0.523598775598286, axis 0 0 -1, limit lower=-3.0043 upper=3.0043 effort=60 velocity=1.5
- added joint right_joint2: type revolute, parent right_link1, child right_link2, origin rpy=-1.5707963267949 0 3.14159265358979, axis 0 0 -1, limit lower=-1.6081 upper=1.6081 effort=60 velocity=1.5
- added joint right_joint3: type revolute, parent right_link2, child right_link3, origin xyz=0 -0.35 0 rpy=-1.5707963267949 1.04719755119629 -3.14159265358979, axis 0 0 -1, limit lower=-2.91697 upper=2.91697 effort=30 velocity=1.5
- added joint right_joint4: type revolute, parent right_link3, child right_link4, origin rpy=-1.57079632679459 0 3.14159265358979, axis 0 0 1, limit lower=-1.86986 upper=2.56799 effort=30 velocity=1.5
- added joint right_joint5: type revolute, parent right_link4, child right_link5, origin xyz=0 -0.36 0 rpy=-1.5707963267949 0 3.1415926535898, axis 0 0 -1, limit lower=-2.91697 upper=2.91697 effort=10 velocity=1.5
- added joint right_joint6: type revolute, parent right_link5, child right_link6, origin rpy=1.5707963267949 1.5707963267949 0, axis 0 0 -1, limit lower=-0.7354 upper=0.8227 effort=10 velocity=1.5
- added joint right_joint7: type revolute, parent right_link6, child right_link7, origin rpy=-1.5707963267949 0 0, axis 0 0 -1, limit lower=-1.5382 upper=1.5382 effort=10 velocity=1.5
- added joint wheel1_joint: type fixed, parent omni_chassis_base_link, child wheel_1, origin xyz=0.176493 0.176493 0.071834 rpy=0 0 -2.356194490192345
- added joint wheel2_joint: type fixed, parent omni_chassis_base_link, child wheel_2, origin xyz=-0.176493 0.176493 0.071834 rpy=0 0 -0.7853981633974483
- added joint wheel3_joint: type fixed, parent omni_chassis_base_link, child wheel_3, origin xyz=-0.176493 -0.176493 0.071834 rpy=0 0 0.7853981633974483
- added joint wheel4_joint: type fixed, parent omni_chassis_base_link, child wheel_4, origin xyz=0.176493 -0.176493 0.071834 rpy=0 0 2.356194490192345
- joint left_arm_end_effector_mount_joint: parent left_arm_link7 -> left_link7
- joint left_arm_joint: child left_arm_base_link -> left_base_link
- joint left_camera_joint: child left_wrist_camera_link -> left_wrist_camera; origin (none) -> xyz=-0.0822 0 -0.06842 rpy=0 1.4807963267948965 3.141592653589793; parent left_arm_link7 -> left_wrist_camera_stand
- joint right_arm_end_effector_mount_joint: parent right_arm_link7 -> right_link7
- joint right_arm_joint: child right_arm_base_link -> right_base_link
- joint right_camera_joint: child right_wrist_camera_link -> right_wrist_camera; origin (none) -> xyz=-0.0822 0 -0.06842 rpy=0 1.4807963267948965 3.141592653589793; parent right_arm_link7 -> right_wrist_camera_stand

File: galbot_golf_description/xacro/component.xacro (robot description, xacro)
@@ -1,8 +1,9 @@
 <?xml version="1.0" ?>
-<robot name="Hitbot Gripper" xmlns:xacro="http://www.ros.org/wiki/xacro">
+<robot name="Head Golf" xmlns:xacro="http://www.ros.org/wiki/xacro">
   <xacro:property name="PI" value="3.141592653589793"/>
   <xacro:arg name="type" default="body"/>
   <xacro:arg name="enable_wheel_joints" default="true"/>
   <xacro:arg name="collider" default="simple"/>
+  <xacro:arg name="enable_joint5" default="true"/>
   <xacro:if value="${'$(arg type)' == 'body'}">
     <link name="base_link"/>
@@ -12,5 +13,10 @@
     </joint>
     <link name="omni_chassis_leg_mount_link"/>
-    <xacro:include filename="$(find galbot_golf_description)/xacro/components/body.xacro"/>
+    <xacro:include filename="$(find galbot_foxtrot_description)/xacro/components/body.xacro"/>
+  </xacro:if>
+  <xacro:if value="${'$(arg type)' == 'head'}">
+    <link name="base_link"/>
+    <xacro:include filename="$(find galbot_golf_description)/xacro/components/head.xacro"/>
+    <xacro:galbot_golf_head parent_link="base_link"/>
   </xacro:if>
 </robot>

File: galbot_golf_description/xacro/robot.xacro (robot description, xacro)
@@ -3,10 +3,13 @@
 	<xacro:arg name="enable_wheel_joints" default="false"/>
 	<xacro:arg name="arm_camera" default="d405"/>
+	<xacro:arg name="enable_joint5" default="true"/>
 	<xacro:property name="PI" value="3.141592653589793"/>
 	<xacro:include filename="$(find galbot_foxtrot_description)/xacro/components/galbot_gripper.xacro"/>
-	<xacro:include filename="$(find galbot_golf_description)/xacro/components/body.xacro"/>
+	<xacro:include filename="$(find galbot_foxtrot_description)/xacro/components/body.xacro"/>
+	<xacro:include filename="$(find galbot_golf_description)/xacro/components/head.xacro"/>
 	<xacro:include filename="$(find galbot_foxtrot_description)/xacro/components/arm.xacro"/>
 	<xacro:include filename="$(find galbot_foxtrot_description)/xacro/components/chassis.xacro"/>
 	<xacro:GalbotChassisV2 enable_wheel_joints="$(arg enable_wheel_joints)"/>
+	<xacro:galbot_golf_head parent_link="torso_base_link"/>
 	<!-- Left Arm Mount -->
 	<link name="torso_left_arm_mount_link"/>
