Commit message: add d415 camera option

File: galbot_foxtrot_description/xacro/components/arm.xacro (robot description, xacro)
@@ -1,5 +1,6 @@
 <?xml version="1.0" ?>
 <robot xmlns:xacro="http://www.ros.org/wiki/xacro">
-	<xacro:macro name="Arm" params="name direction:=1">
+	<xacro:include filename="$(find galbot_foxtrot_description)/xacro/components/camera.xacro"/>
+	<xacro:macro name="Arm" params="name direction:=1 camera:=d405">
 		<xacro:property name="prefix" value="${name + '_' if name else ''}"/>
 		<link name="${prefix}base_link">
@@ -48,7 +49,12 @@
 			<visual>
 				<geometry>
-					<mesh
-							filename="file://$(find galbot_foxtrot_description)/meshes/visual/arm/link2.glb"
-							scale="1 ${direction} 1"/>
+					<xacro:if value="${float(direction) == -1.0}">
+						<mesh
+								filename="file://$(find galbot_foxtrot_description)/meshes/visual/arm/link2_right.glb"/>
+					</xacro:if>
+					<xacro:unless value="${float(direction) == -1.0}">
+						<mesh
+								filename="file://$(find galbot_foxtrot_description)/meshes/visual/arm/link2.glb"/>
+					</xacro:unless>
 				</geometry>
 			</visual>
@@ -202,38 +208,5 @@
 			<limit acceleration="2" effort="10" jerk="12" lower="-1.5382" upper="1.5382" velocity="1.5"/>
 		</joint>
-		<joint name="${prefix}camera_stand_joint" type="fixed">
-			<parent link="${prefix}link7"/>
-			<child link="${prefix}wrist_camera_stand"/>
-		</joint>
-		<link name="${prefix}wrist_camera_stand">
-			<inertial>
-				<origin xyz="-0.0621229724155358 -0.0628379837355285 -0.00140310958315455"/>
-				<mass value="0.0492751941348016"/>
-				<inertia ixx="3.66069470547417E-05" ixy="-3.55284385731841E-07" ixz="3.8533182318026E-07"
-								 iyy="3.08593710158624E-05" iyz="-3.07292981503681E-07" izz="8.80145863410975E-06"/>
-			</inertial>
-			<visual>
-				<geometry>
-					<mesh filename="file://$(find galbot_foxtrot_description)/meshes/visual/arm/d405_stand.glb"/>
-				</geometry>
-			</visual>
-			<collision>
-				<geometry>
-					<mesh filename="file://$(find galbot_foxtrot_description)/meshes/collision/d405.stl"/>
-				</geometry>
-			</collision>
-		</link>
-		<joint name="${prefix}camera_joint" type="fixed">
-			<origin xyz="-0.0822 0 -0.06842" rpy="0 ${PI/2 - 0.09} ${PI}"/>
-			<parent link="${prefix}wrist_camera_stand"/>
-			<child link="${prefix}wrist_camera"/>
-		</joint>
-		<link name="${prefix}wrist_camera">
-			<visual>
-				<geometry>
-					<mesh filename="file://$(find sensor_models)/meshes/realsense/d405.glb"/>
-				</geometry>
-			</visual>
-		</link>
+		<xacro:ArmCamera prefix="${prefix}" camera="${camera}"/>
 	</xacro:macro>
 </robot>

File: galbot_foxtrot_description/xacro/gripper.xacro (robot description, xacro)
@@ -1,5 +1,5 @@
 <?xml version="1.0"?>
 <robot name="Galbot Gripper" xmlns:xacro="http://www.ros.org/wiki/xacro">
-  <xacro:include filename="$(find galbot_foxtrot_description)/xacro/galbot_gripper.xacro"/>
+  <xacro:include filename="$(find galbot_foxtrot_description)/xacro/components/galbot_gripper.xacro"/>
   <xacro:Gripper name=""/>
 </robot>

File: galbot_foxtrot_description/xacro/robot.xacro (robot description, xacro)
@@ -2,8 +2,9 @@
 <robot name="galbot_one_foxtrot" xmlns:xacro="http://www.ros.org/wiki/xacro">
 	<xacro:arg name="enable_wheel_joints" default="false"/>
+	<xacro:arg name="arm_camera" default="d415"/>
 	<xacro:property name="PI" value="3.141592653589793"/>
-	<xacro:include filename="$(find galbot_foxtrot_description)/xacro/galbot_gripper.xacro"/>
+	<xacro:include filename="$(find galbot_foxtrot_description)/xacro/components/galbot_gripper.xacro"/>
 	<xacro:include filename="$(find galbot_foxtrot_description)/xacro/components/body.xacro"/>
-	<xacro:include filename="$(find galbot_foxtrot_description)/xacro/arm.xacro"/>
+	<xacro:include filename="$(find galbot_foxtrot_description)/xacro/components/arm.xacro"/>
 	<xacro:include filename="$(find galbot_foxtrot_description)/xacro/components/chassis.xacro"/>
 	<xacro:GalbotChassisV2 enable_wheel_joints="$(arg enable_wheel_joints)"/>
@@ -28,5 +29,5 @@
 		<child link="right_base_link"/>
 	</joint>
-	<xacro:Arm name="right" direction="-1"/>
+	<xacro:Arm name="right" direction="-1" camera="$(arg arm_camera)"/>
 	<joint name="right_end_effector_mount_joint" type="fixed">
 		<origin rpy="-1.5708 0 3.14159265358948" xyz="-0.10926 0 0"/>
@@ -40,5 +41,5 @@
 		<child link="left_base_link"/>
 	</joint>
-	<xacro:Arm name="left"/>
+	<xacro:Arm name="left" camera="$(arg arm_camera)"/>
 	<joint name="left_end_effector_mount_joint" type="fixed">
 		<origin rpy="-1.5708 0 3.14159265358979" xyz="-0.10926 0 0"/>

File: galbot_golf_description/xacro/robot.xacro (robot description, xacro)
@@ -2,8 +2,9 @@
 <robot name="galbot_one_golf" xmlns:xacro="http://www.ros.org/wiki/xacro">
 	<xacro:arg name="enable_wheel_joints" default="false"/>
+	<xacro:arg name="arm_camera" default="d405"/>
 	<xacro:property name="PI" value="3.141592653589793"/>
-	<xacro:include filename="$(find galbot_foxtrot_description)/xacro/galbot_gripper.xacro"/>
+	<xacro:include filename="$(find galbot_foxtrot_description)/xacro/components/galbot_gripper.xacro"/>
 	<xacro:include filename="$(find galbot_golf_description)/xacro/components/body.xacro"/>
-	<xacro:include filename="$(find galbot_foxtrot_description)/xacro/arm.xacro"/>
+	<xacro:include filename="$(find galbot_foxtrot_description)/xacro/components/arm.xacro"/>
 	<xacro:include filename="$(find galbot_foxtrot_description)/xacro/components/chassis.xacro"/>
 	<xacro:GalbotChassisV2 enable_wheel_joints="$(arg enable_wheel_joints)"/>
@@ -28,5 +29,5 @@
 		<child link="right_base_link"/>
 	</joint>
-	<xacro:Arm name="right" direction="-1"/>
+	<xacro:Arm name="right" direction="-1" camera="$(arg arm_camera)"/>
 	<joint name="right_arm_end_effector_mount_joint" type="fixed">
 		<origin rpy="-1.5708 0 3.14159265358948" xyz="-0.10926 0 0"/>
@@ -40,5 +41,5 @@
 		<child link="left_base_link"/>
 	</joint>
-	<xacro:Arm name="left"/>
+	<xacro:Arm name="left" camera="$(arg arm_camera)"/>
 	<joint name="left_arm_end_effector_mount_joint" type="fixed">
 		<origin rpy="-1.5708 0 3.14159265358979" xyz="-0.10926 0 0"/>
