Commit message: add galbot s1 robot

File: galbot_foxtrot_description/xacro/components/head.xacro (robot description, xacro)
@@ -68,9 +68,9 @@
 		</joint>
 		<link name="head_front_camera">
-<!--			<visual>-->
-<!--				<geometry>-->
-<!--					<mesh filename="file://$(find sensor_models)/meshes/realsense/d435.glb"/>-->
-<!--				</geometry>-->
-<!--			</visual>-->
+			<visual>
+				<geometry>
+					<mesh filename="file://$(find sensor_models)/meshes/realsense/d435.glb"/>
+				</geometry>
+			</visual>
 		</link>
 		<joint name="head_front_camera_joint" type="fixed">
