Commit message: add foxtrot ros2 control config

File: galbot_foxtrot_description/urdf/galbot_foxtrot.urdf (robot description, URDF)
Before this commit: robot galbot_one_foxtrot, 53 links, 52 joints
Links:
- removed link left_arm_base_link
- removed link left_arm_link1
- removed link left_arm_link2
- removed link left_arm_link3
- removed link left_arm_link4
- removed link left_arm_link5
- removed link left_arm_link6
- removed link left_arm_link7
- removed link right_arm_base_link
- removed link right_arm_link1
- removed link right_arm_link2
- removed link right_arm_link3
- removed link right_arm_link4
- removed link right_arm_link5
- removed link right_arm_link6
- removed link right_arm_link7
- removed link torso_left_arm_mount_link
- removed link torso_right_arm_mount_link
- added link left_base_link, mass 0.92
- added link left_link1, mass 1.6; collision mesh filename=file:///home/biao/ros2_ws/install/galbot_foxtrot_descriptio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 scale=1 1 1; visual mesh filename=file:///home/biao/ros2_ws/install/galbot_foxtrot_descriptio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 scale=1 1 1
- added link left_link2, mass 1.43; collision mesh filename=file:///home/biao/ros2_ws/install/galbot_foxtrot_descriptio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 scale=1 1 1; visual mesh filename=file:///home/biao/ros2_ws/install/galbot_foxtrot_descriptio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 scale=1 1 1
- added link left_link3, mass 1.43; collision mesh filename=file:///home/biao/ros2_ws/install/galbot_foxtrot_descriptio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 scale=1 1 1; visual mesh filename=file:///home/biao/ros2_ws/install/galbot_foxtrot_descriptio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 scale=1 1 1
- added link left_link4, mass 1.1; collision mesh filename=file:///home/biao/ros2_ws/install/galbot_foxtrot_descriptio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 scale=1 1 1; visual mesh filename=file:///home/biao/ros2_ws/install/galbot_foxtrot_descriptio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 scale=1 1 1
- added link left_link5, mass 1.15; collision mesh filename=file:///home/biao/ros2_ws/install/galbot_foxtrot_descriptio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; visual mesh filename=file:///home/biao/ros2_ws/install/galbot_foxtrot_descriptio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
- added link left_link6, mass 0.47; collision mesh filename=file:///home/biao/ros2_ws/install/galbot_foxtrot_descriptio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 scale=1 1 1; visual mesh filename=file:///home/biao/ros2_ws/install/galbot_foxtrot_descriptio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 scale=1 1 1
- added link left_link7, mass 0.8; collision mesh filename=file:///home/biao/ros2_ws/install/galbot_foxtrot_descriptio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 scale=1 1 1; visual mesh filename=file:///home/biao/ros2_ws/install/galbot_foxtrot_descriptio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 scale=1 1 1
- added link right_base_link, mass 0.92
- added link right_link1, mass 1.6; collision mesh filename=file:///home/biao/ros2_ws/install/galbot_foxtrot_descriptio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 scale=1 -1 1; visual mesh filename=file:///home/biao/ros2_ws/install/galbot_foxtrot_descriptio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 scale=1 -1 1
- added link right_link2, mass 1.43; collision mesh filename=file:///home/biao/ros2_ws/install/galbot_foxtrot_descriptio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 scale=1 -1 1; visual mesh filename=file:///home/biao/ros2_ws/install/galbot_foxtrot_descriptio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 scale=1 -1 1
- added link right_link3, mass 1.43; collision mesh filename=file:///home/biao/ros2_ws/install/galbot_foxtrot_descriptio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 scale=1 -1 1; visual mesh filename=file:///home/biao/ros2_ws/install/galbot_foxtrot_descriptio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 scale=1 -1 1
- added link right_link4, mass 1.1; collision mesh filename=file:///home/biao/ros2_ws/install/galbot_foxtrot_descriptio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 scale=1 -1 1; visual mesh filename=file:///home/biao/ros2_ws/install/galbot_foxtrot_descriptio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 scale=1 -1 1
- added link right_link5, mass 1.15; collision mesh filename=file:///home/biao/ros2_ws/install/galbot_foxtrot_descriptio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; visual mesh filename=file:///home/biao/ros2_ws/install/galbot_foxtrot_descriptio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
- added link right_link6, mass 0.47; collision mesh filename=file:///home/biao/ros2_ws/install/galbot_foxtrot_descriptio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 scale=1 -1 1; visual mesh filename=file:///home/biao/ros2_ws/install/galbot_foxtrot_descriptio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 scale=1 -1 1
- added link right_link7, mass 0.8; collision mesh filename=file:///home/biao/ros2_ws/install/galbot_foxtrot_descriptio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 scale=1 -1 1; visual mesh filename=file:///home/biao/ros2_ws/install/galbot_foxtrot_descriptio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 scale=1 -1 1
- added link torso_left_mount_link
- added link torso_right_mount_link
- link head_link2: geometry collision mesh filename=file:///home/biao/ros2_ws/install/galbot_foxtrot_descriptio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; visual mesh filename=file:///home/biao/ros2_ws/install/galbot_foxtrot_descriptio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
- link left_gripper_base: geometry collision mesh filename=file:///home/biao/ros2_ws/install/galbot_foxtrot_descriptio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; visual mesh filename=file:///home/biao/ros2_ws/install/galbot_foxtrot_descriptio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
- link left_gripper_flange: geometry visual mesh filename=file:///home/biao/ros2_ws/install/galbot_foxtrot_descriptio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
- link left_gripper_l_finger_link: geometry collision mesh filename=file:///home/biao/ros2_ws/install/galbot_foxtrot_descriptio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; visual mesh filename=file:///home/biao/ros2_ws/install/galbot_foxtrot_descriptio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
- link left_gripper_l_inner_knuckle_link: geometry collision mesh filename=file:///home/biao/ros2_ws/install/galbot_foxtrot_descriptio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; visual mesh filename=file:///home/biao/ros2_ws/install/galbot_foxtrot_descriptio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
- link left_gripper_l_knuckle_link: geometry collision mesh filename=file:///home/biao/ros2_ws/install/galbot_foxtrot_descriptio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; visual mesh filename=file:///home/biao/ros2_ws/install/galbot_foxtrot_descriptio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
- link left_gripper_r_finger_link: geometry collision mesh filename=file:///home/biao/ros2_ws/install/galbot_foxtrot_descriptio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 scale=1 -1 1; visual mesh filename=file:///home/biao/ros2_ws/install/galbot_foxtrot_descriptio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 scale=1 -1 1
- link left_gripper_r_inner_knuckle_link: geometry collision mesh filename=file:///home/biao/ros2_ws/install/galbot_foxtrot_descriptio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; visual mesh filename=file:///home/biao/ros2_ws/install/galbot_foxtrot_descriptio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
- link left_gripper_r_knuckle_link: geometry collision mesh filename=file:///home/biao/ros2_ws/install/galbot_foxtrot_descriptio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; visual mesh filename=file:///home/biao/ros2_ws/install/galbot_foxtrot_descriptio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
- link left_wrist_camera_link: geometry collision mesh filename=file:///home/biao/ros2_ws/install/galbot_foxtrot_descriptio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; visual mesh filename=file:///home/biao/ros2_ws/install/galbot_foxtrot_descriptio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
- link leg_end_effector_mount_link: geometry visual mesh filename=file:///home/biao/ros2_ws/install/galbot_foxtrot_descriptio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
- link leg_link1: geometry collision mesh filename=file:///home/biao/ros2_ws/install/galbot_foxtrot_descriptio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; visual mesh filename=file:///home/biao/ros2_ws/install/galbot_foxtrot_descriptio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
- link leg_link2: geometry collision mesh filename=file:///home/biao/ros2_ws/install/galbot_foxtrot_descriptio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; visual mesh filename=file:///home/biao/ros2_ws/install/galbot_foxtrot_descriptio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
- link leg_link3: geometry collision mesh filename=file:///home/biao/ros2_ws/install/galbot_foxtrot_descriptio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; visual mesh filename=file:///home/biao/ros2_ws/install/galbot_foxtrot_descriptio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
- link leg_link4: geometry visual mesh filename=file:///home/biao/ros2_ws/install/galbot_foxtrot_descriptio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
- link omni_chassis_base_link: geometry collision mesh filename=file:///home/biao/ros2_ws/install/galbot_foxtrot_descriptio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; visual mesh filename=file:///home/biao/ros2_ws/install/galbot_foxtrot_descriptio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
- link right_gripper_base: geometry collision mesh filename=file:///home/biao/ros2_ws/install/galbot_foxtrot_descriptio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; visual mesh filename=file:///home/biao/ros2_ws/install/galbot_foxtrot_descriptio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
- link right_gripper_flange: geometry visual mesh filename=file:///home/biao/ros2_ws/install/galbot_foxtrot_descriptio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
- link right_gripper_l_finger_link: geometry collision mesh filename=file:///home/biao/ros2_ws/install/galbot_foxtrot_descriptio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; visual mesh filename=file:///home/biao/ros2_ws/install/galbot_foxtrot_descriptio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
- link right_gripper_l_inner_knuckle_link: geometry collision mesh filename=file:///home/biao/ros2_ws/install/galbot_foxtrot_descriptio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; visual mesh filename=file:///home/biao/ros2_ws/install/galbot_foxtrot_descriptio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
- link right_gripper_l_knuckle_link: geometry collision mesh filename=file:///home/biao/ros2_ws/install/galbot_foxtrot_descriptio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; visual mesh filename=file:///home/biao/ros2_ws/install/galbot_foxtrot_descriptio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
- link right_gripper_r_finger_link: geometry collision mesh filename=file:///home/biao/ros2_ws/install/galbot_foxtrot_descriptio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 scale=1 -1 1; visual mesh filename=file:///home/biao/ros2_ws/install/galbot_foxtrot_descriptio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 scale=1 -1 1
- link right_gripper_r_inner_knuckle_link: geometry collision mesh filename=file:///home/biao/ros2_ws/install/galbot_foxtrot_descriptio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; visual mesh filename=file:///home/biao/ros2_ws/install/galbot_foxtrot_descriptio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
- link right_gripper_r_knuckle_link: geometry collision mesh filename=file:///home/biao/ros2_ws/install/galbot_foxtrot_descriptio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; visual mesh filename=file:///home/biao/ros2_ws/install/galbot_foxtrot_descriptio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
- link right_wrist_camera_link: geometry collision mesh filename=file:///home/biao/ros2_ws/install/galbot_foxtrot_descriptio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; visual mesh filename=file:///home/biao/ros2_ws/install/galbot_foxtrot_descriptio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
- link torso_base_link: geometry collision mesh filename=file:///home/biao/ros2_ws/install/galbot_foxtrot_descriptio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; visual mesh filename=file:///home/biao/ros2_ws/install/galbot_foxtrot_descriptio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
Joints:
- removed joint left_arm_end_effector_mount_joint
- removed joint left_arm_joint
- removed joint left_arm_joint1
- removed joint left_arm_joint2
- removed joint left_arm_joint3
- removed joint left_arm_joint4
- removed joint left_arm_joint5
- removed joint left_arm_joint6
- removed joint left_arm_joint7
- removed joint leg_joint1
- removed joint leg_joint2
- removed joint leg_joint3
- removed joint leg_joint4
- removed joint right_arm_end_effector_mount_joint
- removed joint right_arm_joint
- removed joint right_arm_joint1
- removed joint right_arm_joint2
- removed joint right_arm_joint3
- removed joint right_arm_joint4
- removed joint right_arm_joint5
- removed joint right_arm_joint6
- removed joint right_arm_joint7
- removed joint torso_left_arm_mount_joint
- removed joint torso_right_arm_mount_joint
- added joint body_joint1: type revolute, parent leg_base_link, child leg_link1, origin rpy=1.5707963267948966 -0.385 3.141592653589793, axis 0 0 1, limit lower=0.0 upper=0.9374 effort=169 velocity=1
- added joint body_joint2: type revolute, parent leg_link1, child leg_link2, origin xyz=0.45 0 0 rpy=3.141592653589793 0 2.7566, axis 0 0 1, limit lower=0.0 upper=2.5847 effort=169 velocity=1
- added joint body_joint3: type revolute, parent leg_link2, child leg_link3, origin xyz=0.39 0 0 rpy=3.141592653589793 0 3.141592653589793, axis 0 0 1, limit lower=0.0 upper=2.3262 effort=84 velocity=1
- added joint body_joint4: type revolute, parent leg_link3, child leg_link4, origin xyz=0 0.224 0 rpy=-1.5707963267948966 -1.5707963267948966 0, axis 0 0 1, limit lower=-1.5906 upper=1.5906 effort=30 velocity=1
- added joint left_end_effector_mount_joint: type fixed, parent left_link7, child left_gripper_flange, origin xyz=-0.10926 0 0 rpy=-1.5708 0 3.14159265358979
- added joint left_joint: type fixed, parent torso_left_mount_link, child left_base_link
- added joint left_joint1: type revolute, parent left_base_link, child left_link1, origin rpy=0 0 0.523598775598286, axis 0 0 1, limit lower=-3.0043 upper=3.0043 effort=60 velocity=1.5
- added joint left_joint2: type revolute, parent left_link1, child left_link2, origin rpy=1.5707963267949 0 3.14159265358979, axis 0 0 1, limit lower=-1.6081 upper=1.6081 effort=60 velocity=1.5
- added joint left_joint3: type revolute, parent left_link2, child left_link3, origin xyz=0 0.35 0 rpy=1.5707963267949 1.04719755119629 -3.14159265358979, axis 0 0 1, limit lower=-2.91697 upper=2.91697 effort=30 velocity=1.5
- added joint left_joint4: type revolute, parent left_link3, child left_link4, origin rpy=1.57079632679459 0 3.14159265358979, axis 0 0 -1, limit lower=-1.86986 upper=2.56799 effort=30 velocity=1.5
- added joint left_joint5: type revolute, parent left_link4, child left_link5, origin xyz=0 0.36 0 rpy=-1.5707963267949 0 0.0, axis 0 0 1, limit lower=-2.91697 upper=2.91697 effort=10 velocity=1.5
- added joint left_joint6: type revolute, parent left_link5, child left_link6, origin rpy=1.5707963267949 1.5707963267949 0, axis 0 0 1, limit lower=-0.7354 upper=0.8227 effort=10 velocity=1.5
- added joint left_joint7: type revolute, parent left_link6, child left_link7, origin rpy=1.5707963267949 0 0, axis 0 0 1, limit lower=-1.5382 upper=1.5382 effort=10 velocity=1.5
- added joint right_end_effector_mount_joint: type fixed, parent right_link7, child right_gripper_flange, origin xyz=-0.10926 0 0 rpy=-1.5708 0 3.14159265358948, axis 
- added joint right_joint: type fixed, parent torso_right_mount_link, child right_base_link
- added joint right_joint1: type revolute, parent right_base_link, child right_link1, origin rpy=0 0 -0.523598775598286, axis 0 0 -1, limit lower=-3.0043 upper=3.0043 effort=60 velocity=1.5
- added joint right_joint2: type revolute, parent right_link1, child right_link2, origin rpy=-1.5707963267949 0 3.14159265358979, axis 0 0 -1, limit lower=-1.6081 upper=1.6081 effort=60 velocity=1.5
- added joint right_joint3: type revolute, parent right_link2, child right_link3, origin xyz=0 -0.35 0 rpy=-1.5707963267949 1.04719755119629 -3.14159265358979, axis 0 0 -1, limit lower=-2.91697 upper=2.91697 effort=30 velocity=1.5
- added joint right_joint4: type revolute, parent right_link3, child right_link4, origin rpy=-1.57079632679459 0 3.14159265358979, axis 0 0 1, limit lower=-1.86986 upper=2.56799 effort=30 velocity=1.5
- added joint right_joint5: type revolute, parent right_link4, child right_link5, origin xyz=0 -0.36 0 rpy=-1.5707963267949 0 3.1415926535898, axis 0 0 -1, limit lower=-2.91697 upper=2.91697 effort=10 velocity=1.5
- added joint right_joint6: type revolute, parent right_link5, child right_link6, origin rpy=1.5707963267949 1.5707963267949 0, axis 0 0 -1, limit lower=-0.7354 upper=0.8227 effort=10 velocity=1.5
- added joint right_joint7: type revolute, parent right_link6, child right_link7, origin rpy=-1.5707963267949 0 0, axis 0 0 -1, limit lower=-1.5382 upper=1.5382 effort=10 velocity=1.5
- added joint torso_left_mount_joint: type fixed, parent torso_base_link, child torso_left_mount_link, origin xyz=0.20843 0.172 0 rpy=0 1.5707963267948966 0, axis 
- added joint torso_right_mount_joint: type fixed, parent torso_base_link, child torso_right_mount_link, origin xyz=-0.20843 0.172 0 rpy=3.141592653589793 1.5707963267948966 0, axis 
- joint left_camera_joint: parent left_arm_link7 -> left_link7
- joint right_camera_joint: parent right_arm_link7 -> right_link7

File: galbot_foxtrot_description/xacro/arm.xacro (robot description, xacro)
@@ -3,5 +3,5 @@
 	<xacro:macro name="Arm" params="name direction:=1">
 		<xacro:property name="prefix" value="${name + '_' if name else ''}"/>
-		<link name="${prefix}arm_base_link">
+		<link name="${prefix}base_link">
 			<inertial>
 				<origin xyz="0.0 0.0 -0.10506"/>
@@ -11,5 +11,5 @@
 			</inertial>
 		</link>
-		<link name="${prefix}arm_link1">
+		<link name="${prefix}link1">
 			<inertial>
 				<origin xyz="0.0 ${direction*0.0009699999999999999} -0.015390000000000001"/>
@@ -31,12 +31,12 @@
 			</collision>
 		</link>
-		<joint name="${prefix}arm_joint1" type="revolute">
+		<joint name="${prefix}joint1" type="revolute">
 			<origin rpy="0 0 ${direction*0.523598775598286}"/>
-			<parent link="${prefix}arm_base_link"/>
-			<child link="${prefix}arm_link1"/>
+			<parent link="${prefix}base_link"/>
+			<child link="${prefix}link1"/>
 			<axis xyz="0 0 ${direction}"/>
 			<limit acceleration="2" effort="60" jerk="12" lower="-3.0043" upper="3.0043" velocity="1.5"/>
 		</joint>
-		<link name="${prefix}arm_link2">
+		<link name="${prefix}link2">
 			<inertial>
 				<origin xyz="0.0 ${direction*0.09558} 0.010150000000000001"/>
@@ -61,12 +61,12 @@
 			</collision>
 		</link>
-		<joint name="${prefix}arm_joint2" type="revolute">
+		<joint name="${prefix}joint2" type="revolute">
 			<origin rpy="${direction*1.5707963267949} 0 3.14159265358979"/>
-			<parent link="${prefix}arm_link1"/>
-			<child link="${prefix}arm_link2"/>
+			<parent link="${prefix}link1"/>
+			<child link="${prefix}link2"/>
 			<axis xyz="0 0 ${direction}"/>
 			<limit acceleration="2" effort="60" jerk="12" lower="-1.6081" upper="1.6081" velocity="1.5"/>
 		</joint>
-		<link name="${prefix}arm_link3">
+		<link name="${prefix}link3">
 			<inertial>
 				<origin xyz="0.0 ${direction*0.00088} -0.04936"/>
@@ -87,12 +87,12 @@
 			</collision>
 		</link>
-		<joint name="${prefix}arm_joint3" type="revolute">
+		<joint name="${prefix}joint3" type="revolute">
 			<origin rpy="${direction*1.5707963267949} 1.04719755119629 -3.14159265358979" xyz="0 ${direction*0.35} 0"/>
-			<parent link="${prefix}arm_link2"/>
-			<child link="${prefix}arm_link3"/>
+			<parent link="${prefix}link2"/>
+			<child link="${prefix}link3"/>
 			<axis xyz="0 0 ${direction}"/>
 			<limit acceleration="2" effort="30" jerk="12" lower="-2.91697" upper="2.91697" velocity="1.5"/>
 		</joint>
-		<link name="${prefix}arm_link4">
+		<link name="${prefix}link4">
 			<inertial>
 				<origin xyz="0.0 ${direction*0.05614} 0.019170000000000003"/>
@@ -114,12 +114,12 @@
 			</collision>
 		</link>
-		<joint name="${prefix}arm_joint4" type="revolute">
+		<joint name="${prefix}joint4" type="revolute">
 			<origin rpy="${direction*1.57079632679459} 0 3.14159265358979"/>
-			<parent link="${prefix}arm_link3"/>
-			<child link="${prefix}arm_link4"/>
-			<axis xyz="0 0 ${direction}"/>
+			<parent link="${prefix}link3"/>
+			<child link="${prefix}link4"/>
+			<axis xyz="0 0 ${-direction}"/>
 			<limit acceleration="2" effort="30" jerk="12" lower="-1.86986" upper="2.56799" velocity="1.5"/>
 		</joint>
-		<link name="${prefix}arm_link5">
+		<link name="${prefix}link5">
 			<inertial>
 				<origin xyz="0.00044 0.0016899999999999999 -0.13306"/>
@@ -141,12 +141,12 @@
 			</collision>
 		</link>
-		<joint name="${prefix}arm_joint5" type="revolute">
+		<joint name="${prefix}joint5" type="revolute">
 			<origin rpy="-1.5707963267949 0 ${direction*-1.5707963267949 + 1.5707963267949}" xyz="0 ${direction*0.36} 0"/>
-			<parent link="${prefix}arm_link4"/>
-			<child link="${prefix}arm_link5"/>
+			<parent link="${prefix}link4"/>
+			<child link="${prefix}link5"/>
 			<axis xyz="0 0 ${direction}"/>
 			<limit acceleration="2" effort="10" jerk="12" lower="-2.91697" upper="2.91697" velocity="1.5"/>
 		</joint>
-		<link name="${prefix}arm_link6">
+		<link name="${prefix}link6">
 			<inertial>
 				<origin xyz="-0.00088 ${direction*-0.0072699999999999996} -0.00011999999999999999"/>
@@ -168,12 +168,12 @@
 			</collision>
 		</link>
-		<joint name="${prefix}arm_joint6" type="revolute">
+		<joint name="${prefix}joint6" type="revolute">
 			<origin rpy="1.5707963267949 1.5707963267949 0"/>
-			<parent link="${prefix}arm_link5"/>
-			<child link="${prefix}arm_link6"/>
+			<parent link="${prefix}link5"/>
+			<child link="${prefix}link6"/>
 			<axis xyz="0 0 ${direction}"/>
 			<limit acceleration="2" effort="10" jerk="12" lower="-0.7354" upper="0.8227" velocity="1.5"/>
 		</joint>
-		<link name="${prefix}arm_link7">
+		<link name="${prefix}link7">
 			<inertial>
 				<origin xyz="-0.05751 ${direction*-0.00684} 0.011869999999999999"/>
@@ -195,13 +195,13 @@
 			</collision>
 		</link>
-		<joint name="${prefix}arm_joint7" type="revolute">
+		<joint name="${prefix}joint7" type="revolute">
 			<origin rpy="${direction*1.5707963267949} 0 0"/>
-			<parent link="${prefix}arm_link6"/>
-			<child link="${prefix}arm_link7"/>
+			<parent link="${prefix}link6"/>
+			<child link="${prefix}link7"/>
 			<axis xyz="0 0 ${direction}"/>
 			<limit acceleration="2" effort="10" jerk="12" lower="-1.5382" upper="1.5382" velocity="1.5"/>
 		</joint>
 		<joint name="${prefix}camera_joint" type="fixed">
-			<parent link="${prefix}arm_link7"/>
+			<parent link="${prefix}link7"/>
 			<child link="${prefix}wrist_camera_link"/>
 		</joint>

File: galbot_foxtrot_description/xacro/robot.xacro (robot description, xacro)
@@ -62,5 +62,5 @@
 		</collision>
 	</link>
-	<joint name="leg_joint1" type="revolute">
+	<joint name="body_joint1" type="revolute">
 		<origin rpy="1.5707963267948966 -0.385 3.141592653589793"/>
 		<parent link="leg_base_link"/>
@@ -87,5 +87,5 @@
 		</collision>
 	</link>
-	<joint name="leg_joint2" type="revolute">
+	<joint name="body_joint2" type="revolute">
 		<origin rpy="3.141592653589793 0 2.7566" xyz="0.45 0 0"/>
 		<parent link="leg_link1"/>
@@ -111,5 +111,5 @@
 		</collision>
 	</link>
-	<joint name="leg_joint3" type="revolute">
+	<joint name="body_joint3" type="revolute">
 		<origin rpy="3.141592653589793 0 3.141592653589793" xyz="0.39 0 0"/>
 		<parent link="leg_link2"/>
@@ -130,5 +130,5 @@
 		</visual>
 	</link>
-	<joint name="leg_joint4" type="revolute">
+	<joint name="body_joint4" type="revolute">
 		<origin rpy="-1.5707963267948966 -1.5707963267948966 0" xyz="0 0.224 0"/>
 		<parent link="leg_link3"/>
@@ -177,17 +177,17 @@
 	</link>
 	<!-- Left Arm Mount -->
-	<link name="torso_left_arm_mount_link"/>
-	<joint name="torso_left_arm_mount_joint" type="fixed">
+	<link name="torso_left_mount_link"/>
+	<joint name="torso_left_mount_joint" type="fixed">
 		<origin rpy="0 1.5707963267948966 0" xyz="0.20843 0.172 0"/>
 		<parent link="torso_base_link"/>
-		<child link="torso_left_arm_mount_link"/>
+		<child link="torso_left_mount_link"/>
 		<axis/>
 	</joint>
 	<!-- Right Arm Mount -->
-	<link name="torso_right_arm_mount_link"/>
-	<joint name="torso_right_arm_mount_joint" type="fixed">
+	<link name="torso_right_mount_link"/>
+	<joint name="torso_right_mount_joint" type="fixed">
 		<origin rpy="3.141592653589793 1.5707963267948966 0" xyz="-0.20843 0.172 0"/>
 		<parent link="torso_base_link"/>
-		<child link="torso_right_arm_mount_link"/>
+		<child link="torso_right_mount_link"/>
 		<axis/>
 	</joint>
@@ -256,24 +256,24 @@
 		<axis/>
 	</joint>
-	<joint name="right_arm_joint" type="fixed">
-		<parent link="torso_right_arm_mount_link"/>
-		<child link="right_arm_base_link"/>
+	<joint name="right_joint" type="fixed">
+		<parent link="torso_right_mount_link"/>
+		<child link="right_base_link"/>
 	</joint>
 	<xacro:Arm name="right" direction="-1"/>
-	<joint name="right_arm_end_effector_mount_joint" type="fixed">
+	<joint name="right_end_effector_mount_joint" type="fixed">
 		<origin rpy="-1.5708 0 3.14159265358948" xyz="-0.10926 0 0"/>
-		<parent link="right_arm_link7"/>
+		<parent link="right_link7"/>
 		<child link="right_gripper_flange"/>
 		<axis/>
 	</joint>
 	<xacro:Gripper name="right"/>
-	<joint name="left_arm_joint" type="fixed">
-		<parent link="torso_left_arm_mount_link"/>
-		<child link="left_arm_base_link"/>
+	<joint name="left_joint" type="fixed">
+		<parent link="torso_left_mount_link"/>
+		<child link="left_base_link"/>
 	</joint>
 	<xacro:Arm name="left"/>
-	<joint name="left_arm_end_effector_mount_joint" type="fixed">
+	<joint name="left_end_effector_mount_joint" type="fixed">
 		<origin rpy="-1.5708 0 3.14159265358979" xyz="-0.10926 0 0"/>
-		<parent link="left_arm_link7"/>
+		<parent link="left_link7"/>
 		<child link="left_gripper_flange"/>
 	</joint>
