Commit message: add galbot zero base_footprint

File: galbot_zero_description/urdf/galbot_zero.urdf (robot description, URDF)
Before this commit: robot galbot_zero, 62 links, 61 joints
Links:
- added link base_footprint
Joints:
- added joint base_footprint_joint: type fixed, parent base_footprint, child base_link, origin xyz=0 0 0 rpy=0 0 0

File: galbot_zero_description/xacro/robot.xacro (robot description, xacro)
@@ -9,4 +9,11 @@
   <!-- ===== Camera Component ===== -->
   <xacro:include filename="$(find galbot_zero_description)/xacro/components/camera.xacro"/>
+  <!-- Robot Base Link -->
+  <link name="base_footprint"/>
+  <joint name="base_footprint_joint" type="fixed">
+    <origin rpy="0 0 0" xyz="0 0 0"/>
+    <parent link="base_footprint"/>
+    <child link="base_link"/>
+  </joint>
   <!-- ===== Assembly ===== -->
   <xacro:GalbotZeroChassis enable_wheel_joints="$(arg enable_wheel_joints)"/>
@@ -27,5 +34,5 @@
   <!-- ===== RM75 Arm ===== -->
   <xacro:include filename="$(find rm75_description)/xacro/arm.xacro"/>
-  <xacro:rm75 name="left" ee_type="f" use_simple_collision="true"/>
+  <xacro:rm75 name="left" ee_type="f" />
   <joint name="left_body_mount_joint" type="fixed">
     <origin rpy="${PI/2} -${PI/2} 0" xyz="-0.05 -0.05 0.269"/>
@@ -34,5 +41,5 @@
   </joint>
   <xacro:GalbotZeroCameraD415 prefix="left_" parent_link="left_ee"/>
-  <xacro:rm75 name="right" ee_type="f" use_simple_collision="true"/>
+  <xacro:rm75 name="right" ee_type="f" />
   <joint name="right_body_mount_joint" type="fixed">
     <origin rpy="-${PI/2} -${PI/2} 0" xyz="-0.05 0.05 0.269"/>
