Commit message: update camera.xacro

File: galbot_charlie_description/xacro/component.xacro (robot description, xacro)
@@ -40,9 +40,21 @@
     </joint>
     <xacro:include filename="$(find galbot_charlie_description)/xacro/components/arm.xacro"/>
-    <xacro:include filename="$(find galbot_charlie_description)/xacro/components/camera.xacro"/>
+    <xacro:include filename="$(find galbot_one_description)/xacro/components/camera.xacro"/>
     <xacro:galbot_charlie_arm name="left" direction="1"/>
     <xacro:galbot_charlie_arm name="right" direction="-1"/>
-    <xacro:galbot_charlie_arm_camera name="left" direction="1"/>
-    <xacro:galbot_charlie_arm_camera name="right" direction="-1"/>
+    <link name="left_camera_mount_link"/>
+    <joint name="left_camera_mount_joint" type="fixed">
+      <origin xyz="0.03 0 0" rpy="0 -1.57 0"/>
+      <parent link="left_link7"/>
+      <child link="left_camera_mount_link"/>
+    </joint>
+    <link name="right_camera_mount_link"/>
+    <joint name="right_camera_mount_joint" type="fixed">
+      <origin xyz="0 0 0" rpy="0 -1.57 0"/>
+      <parent link="right_link7"/>
+      <child link="right_camera_mount_link"/>
+    </joint>
+    <xacro:GalbotOneArmCamera name="left" direction="1" parent="left_link7" flange_parent="left_camera_mount_link"/>
+    <xacro:GalbotOneArmCamera name="right" direction="-1" parent="right_link7" flange_parent="right_camera_mount_link"/>
   </xacro:if>
 </robot>

File: galbot_charlie_description/xacro/robot.xacro (robot description, xacro)
@@ -33,10 +33,22 @@
   <xacro:include filename="$(find galbot_one_description)/xacro/components/body.xacro"/>
   <xacro:include filename="$(find galbot_charlie_description)/xacro/components/arm.xacro"/>
-  <xacro:include filename="$(find galbot_charlie_description)/xacro/components/camera.xacro"/>
+  <xacro:include filename="$(find galbot_one_description)/xacro/components/camera.xacro"/>
   <xacro:GalbotOneChassis enable_wheel_joints="$(arg enable_wheel_joints)"/>
   <xacro:galbot_charlie_arm name="left" direction="1"/>
   <xacro:galbot_charlie_arm name="right" direction="-1"/>
-  <xacro:galbot_charlie_arm_camera name="left" direction="1"/>
-  <xacro:galbot_charlie_arm_camera name="right" direction="-1"/>
+  <link name="left_camera_mount_link"/>
+  <joint name="left_camera_mount_joint" type="fixed">
+    <origin xyz="0.03 0 0" rpy="0 -1.57 0"/>
+    <parent link="left_link7"/>
+    <child link="left_camera_mount_link"/>
+  </joint>
+  <link name="right_camera_mount_link"/>
+  <joint name="right_camera_mount_joint" type="fixed">
+    <origin xyz="0 0 0" rpy="0 -1.57 0"/>
+    <parent link="right_link7"/>
+    <child link="right_camera_mount_link"/>
+  </joint>
+  <xacro:GalbotOneArmCamera name="left" direction="1" parent="left_link7" flange_parent="left_camera_mount_link"/>
+  <xacro:GalbotOneArmCamera name="right" direction="-1" parent="right_link7" flange_parent="right_camera_mount_link"/>
   <joint name="left_arm_mount_joint" type="fixed">
     <origin rpy="0 ${PI} 0" xyz="0 0 -0.13"/>
@@ -52,8 +64,8 @@
     <xacro:include filename="$(find galbot_one_description)/xacro/components/galbot_hitbot_gripper.xacro"/>
     <xacro:hitbot_gripper name="right_gripper" parent="right_arm_end_effector_mount_link">
-      <origin xyz="0 0 0" rpy="0 0 0 "/>
+      <origin xyz="0.083 0 0" rpy="0 0 0"/>
     </xacro:hitbot_gripper>
     <xacro:hitbot_gripper name="left_gripper" parent="left_arm_end_effector_mount_link">
-      <origin xyz="0 0 0" rpy="0 0 0"/>
+      <origin xyz="0.083 0 0" rpy="0 0 0"/>
     </xacro:hitbot_gripper>
   </xacro:if>
@@ -63,10 +75,10 @@
     <xacro:Gripper name="left"/>
     <joint name="left_gripper_mount_joint" type="fixed">
-      <origin xyz="0 0 0.005" rpy="1.57 0 0"/>
+      <origin xyz="0.088 0 0" rpy="1.57 0  0 "/>
       <parent link="left_arm_end_effector_mount_link"/>
       <child link="left_gripper_flange"/>
     </joint>
     <joint name="right_gripper_mount_joint" type="fixed">
-      <origin xyz="0 0 0.005" rpy="1.57 0 0"/>
+      <origin xyz="0.088 0 0" rpy="-1.57 0  0 "/>
       <parent link="right_arm_end_effector_mount_link"/>
       <child link="right_gripper_flange"/>

File: galbot_one_description/xacro/components/camera.xacro (robot description, xacro)
@@ -2,70 +2,38 @@
 <robot xmlns:xacro="http://www.ros.org/wiki/xacro">
 	<xacro:property name="PI" value="3.141592653589793"/>
-	<!-- One arm flange + wrist camera assembly -->
-	<xacro:macro name="GalbotOneArmCamera" params="name direction:=1 parent camera:=d415 collider_type:=simple">
+	<!-- Wrist camera assembly; gripper mount is kept separate from the camera support. -->
+	<xacro:macro name="GalbotOneArmCamera" params="name direction:=1 parent camera:=d415 collider_type:=simple profile:=one flange_parent:=''">
 		<xacro:property name="prefix" value="${name}_"/>
-		<link name="${prefix}end_effector_mount_link"/>
-		<joint name="${prefix}end_effector_mount_joint" type="fixed">
-			<origin xyz="0 0 0.0845"/>
+		<xacro:property name="resolved_flange_parent" value="${flange_parent if flange_parent else parent}"/>
+		<link name="${prefix}arm_end_effector_mount_link">
+			<inertial>
+				<origin rpy="0 0 0" xyz="0 0 0"/>
+				<mass value="0"/>
+				<inertia ixx="0" ixy="0" ixz="0" iyy="0" iyz="0" izz="0"/>
+			</inertial>
+		</link>
+		<joint name="${prefix}arm_end_effector_mount_joint" type="fixed">
+			<origin rpy="${-PI/2 * direction} 0 ${PI}" xyz="0 0 0"/>
 			<parent link="${parent}"/>
-			<child link="${prefix}end_effector_mount_link"/>
+			<child link="${prefix}arm_end_effector_mount_link"/>
 		</joint>
-		<joint name="${prefix}flange_joint" type="fixed">
-			<origin rpy="0 0 ${(1 + direction) * PI/2}"/>
-			<parent link="${prefix}end_effector_mount_link"/>
-			<child link="${prefix}flange_base_link"/>
-		</joint>
-		<link name="${prefix}flange_base_link">
+		<link name="${prefix}flange_link">
 			<inertial>
-				<origin xyz="0.052829 -0.00096484 0.013285"/>
+				<origin rpy="0 0 0" xyz="0.052829 -0.00096484 0.013285"/>
 				<mass value="0.25733"/>
-				<inertia ixx="0.0002175" ixy="-2.5433E-06" ixz="4.0586E-06" iyy="5.3894E-05" iyz="-1.8533E-06"
-								 izz="0.00025319"/>
+				<inertia ixx="0.0002175" ixy="-2.5433E-06" ixz="4.0586E-06" iyy="5.3894E-05" iyz="-1.8533E-06" izz="0.00025319"/>
 			</inertial>
 			<visual>
 				<geometry>
-					<mesh filename="file://$(find galbot_one_description)/meshes/flange/flange.glb"/>
+					<mesh filename="file://$(find galbot_one_description)/meshes/flange/camera_support.glb" scale="1 ${direction} 1"/>
 				</geometry>
 			</visual>
-			<xacro:if value="${collider_type == 'convex'}">
-				<collision>
-					<geometry>
-						<mesh filename="file://$(find galbot_one_description)/meshes/flange/flange.glb"/>
-					</geometry>
-				</collision>
-			</xacro:if>
 		</link>
-		<link name="${prefix}flange_mount_link"/>
-		<joint name="${prefix}flange_mount_joint" type="fixed">
-			<origin xyz="0 0 0.006"/>
-			<parent link="${prefix}flange_base_link"/>
-			<child link="${prefix}flange_mount_link"/>
+		<joint name="${prefix}joint" type="fixed">
+			<origin rpy="${PI} -1.308996939 ${PI * (1 + direction) / 2}" xyz="${-0.0526 * direction} 0.02 0.101982"/>
+			<parent link="${resolved_flange_parent}"/>
+			<child link="${prefix}flange_link"/>
 		</joint>
 		<xacro:if value="${camera == 'd415'}">
-			<joint name="${prefix}camera_flange_joint" type="fixed">
-				<origin rpy="${PI} -1.308996939 0" xyz="0.0526 -0.02 0.017482"/>
-				<parent link="${prefix}flange_base_link"/>
-				<child link="${prefix}camera_flange_link"/>
-			</joint>
-			<link name="${prefix}camera_flange_link">
-				<inertial>
-					<origin xyz="0.052829 -0.00096484 0.02054"/>##3-2
-					<mass value="0.25733"/>
-					<inertia ixx="0.0002175" ixy="-2.5433E-06" ixz="4.0586E-06" iyy="5.3894E-05" iyz="-1.8533E-06"
-									 izz="0.00025319"/>
-				</inertial>
-				<visual>
-					<geometry>
-						<mesh filename="file://$(find galbot_one_description)/meshes/flange/camera_support.glb"/>
-					</geometry>
-				</visual>
-				<xacro:if value="${collider_type == 'convex'}">
-					<collision>
-						<geometry>
-							<mesh filename="file://$(find galbot_one_description)/meshes/flange/camera_support.glb"/>
-						</geometry>
-					</collision>
-				</xacro:if>
-			</link>
 			<link name="${prefix}camera_link">
 				<visual>
@@ -76,6 +44,6 @@
 			</link>
 			<joint name="${prefix}camera_joint" type="fixed">
-				<origin rpy="-${PI/2} 0 -${PI/2}" xyz="0.0095 -0.02 0"/>
-				<parent link="${prefix}camera_flange_link"/>
+				<origin rpy="-${PI/2} 0 -${PI/2}" xyz="0.0095 ${-0.02 * direction} 0"/>
+				<parent link="${prefix}flange_link"/>
 				<child link="${prefix}camera_link"/>
 			</joint>

File: galbot_one_description/xacro/robot.xacro (robot description, xacro)
@@ -50,9 +50,9 @@
   <xacro:if value="${selected_gripper_type == 'hitbot'}">
     <xacro:include filename="$(find galbot_one_description)/xacro/components/galbot_hitbot_gripper.xacro"/>
-    <xacro:hitbot_gripper name="right_gripper" parent="right_flange_mount_link">
-      <origin xyz="0 0 0" rpy="0 -1.5708 0"/>
+    <xacro:hitbot_gripper name="right_gripper" parent="right_arm_end_effector_mount_link">
+      <origin xyz="0 0.084525 0" rpy="${PI/2} 0 ${PI/2}"/>
     </xacro:hitbot_gripper>
-    <xacro:hitbot_gripper name="left_gripper" parent="left_flange_mount_link">
-      <origin xyz="0 0 0" rpy="0 -1.5708 0"/>
+    <xacro:hitbot_gripper name="left_gripper" parent="left_arm_end_effector_mount_link">
+      <origin xyz="0 -0.084525 0" rpy="${PI/2} 0 -${PI/2}"/>
     </xacro:hitbot_gripper>
   </xacro:if>
@@ -62,11 +62,11 @@
     <xacro:Gripper name="left"/>
     <joint name="left_gripper_mount_joint" type="fixed">
-      <origin xyz="0 0 0.005" rpy="0 -1.5708 1.5708"/>
-      <parent link="left_flange_mount_link"/>
+      <origin xyz="0 -0.089525 0" rpy="${-PI} 0 -${PI/2}"/>
+      <parent link="left_arm_end_effector_mount_link"/>
       <child link="left_gripper_flange"/>
     </joint>
     <joint name="right_gripper_mount_joint" type="fixed">
-      <origin xyz="0 0 0.005" rpy="0 -1.5708 1.5708"/>
-      <parent link="right_flange_mount_link"/>
+      <origin xyz="0 0.089525 0" rpy="${-PI} 0 ${PI/2}"/>
+      <parent link="right_arm_end_effector_mount_link"/>
       <child link="right_gripper_flange"/>
     </joint>
