Commit message: 更新galbot整体readme以及照片

File: galbot_one_description/urdf/galbot_one_galbot_gripper.urdf (robot description, URDF)
Before this commit: robot galbot_one, 64 links, 63 joints
Links:
- link left_gripper_base: geometry collision mesh filename=package://galbot_foxtrot_description/meshes/collision/gripp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; visual mesh filename=package://galbot_foxtrot_description/meshes/visual/gripper/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
- link left_gripper_flange: geometry visual mesh filename=package://galbot_foxtrot_description/meshes/visual/gripper/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
- link left_gripper_l_finger_link: geometry collision mesh filename=package://galbot_foxtrot_description/meshes/collision/gripp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; visual mesh filename=package://galbot_foxtrot_description/meshes/visual/gripper/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
- link left_gripper_l_inner_knuckle_link: geometry collision mesh filename=package://galbot_foxtrot_description/meshes/collision/gripp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; visual mesh filename=package://galbot_foxtrot_description/meshes/visual/gripper/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
- link left_gripper_l_knuckle_link: geometry collision mesh filename=package://galbot_foxtrot_description/meshes/collision/gripp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; visual mesh filename=package://galbot_foxtrot_description/meshes/visual/gripper/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
- link left_gripper_r_finger_link: geometry collision mesh filename=package://galbot_foxtrot_description/meshes/collision/gripp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 scale=1 -1 1; visual mesh filename=package://galbot_foxtrot_description/meshes/visual/gripper/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 scale=1 -1 1
- link left_gripper_r_inner_knuckle_link: geometry collision mesh filename=package://galbot_foxtrot_description/meshes/collision/gripp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; visual mesh filename=package://galbot_foxtrot_description/meshes/visual/gripper/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
- link left_gripper_r_knuckle_link: geometry collision mesh filename=package://galbot_foxtrot_description/meshes/collision/gripp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; visual mesh filename=package://galbot_foxtrot_description/meshes/visual/gripper/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
- link right_gripper_base: geometry collision mesh filename=package://galbot_foxtrot_description/meshes/collision/gripp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; visual mesh filename=package://galbot_foxtrot_description/meshes/visual/gripper/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
- link right_gripper_flange: geometry visual mesh filename=package://galbot_foxtrot_description/meshes/visual/gripper/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
- link right_gripper_l_finger_link: geometry collision mesh filename=package://galbot_foxtrot_description/meshes/collision/gripp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; visual mesh filename=package://galbot_foxtrot_description/meshes/visual/gripper/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
- link right_gripper_l_inner_knuckle_link: geometry collision mesh filename=package://galbot_foxtrot_description/meshes/collision/gripp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; visual mesh filename=package://galbot_foxtrot_description/meshes/visual/gripper/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
- link right_gripper_l_knuckle_link: geometry collision mesh filename=package://galbot_foxtrot_description/meshes/collision/gripp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; visual mesh filename=package://galbot_foxtrot_description/meshes/visual/gripper/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
- link right_gripper_r_finger_link: geometry collision mesh filename=package://galbot_foxtrot_description/meshes/collision/gripp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 scale=1 -1 1; visual mesh filename=package://galbot_foxtrot_description/meshes/visual/gripper/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 scale=1 -1 1
- link right_gripper_r_inner_knuckle_link: geometry collision mesh filename=package://galbot_foxtrot_description/meshes/collision/gripp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; visual mesh filename=package://galbot_foxtrot_description/meshes/visual/gripper/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
- link right_gripper_r_knuckle_link: geometry collision mesh filename=package://galbot_foxtrot_description/meshes/collision/gripp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; visual mesh filename=package://galbot_foxtrot_description/meshes/visual/gripper/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
- link wheel_1: geometry visual mesh filename=package://component_models/meshes/omniwheel_10.glb
- link wheel_2: geometry visual mesh filename=package://component_models/meshes/omniwheel_10.glb
- link wheel_3: geometry visual mesh filename=package://component_models/meshes/omniwheel_10.glb
- link wheel_4: geometry visual mesh filename=package://component_models/meshes/omniwheel_10.glb
