Commit message: fix body name

File: galbot_charlie_description/urdf/galbot_charlie.urdf (robot description, URDF)
Before this commit: robot galbot_charlie, 64 links, 65 joints
Links:
- link chassis_lidar: geometry visual mesh filename=file:///home/fiveages/ros2_ws/install/sensor_models/share/s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
- link head_back_camera: geometry visual mesh filename=file:///home/fiveages/ros2_ws/install/sensor_models/share/s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
- link head_base_link: geometry visual mesh filename=package://galbot_one_description/meshes/head/head_base.glb
- link head_front_camera: geometry visual mesh filename=file:///home/fiveages/ros2_ws/install/sensor_models/share/s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
- link head_link1: geometry visual mesh filename=package://galbot_one_description/meshes/head/head_link1.glb
- link head_link2: geometry visual mesh filename=package://galbot_one_description/meshes/head/head_link2.glb
- link left_base_link: geometry collision cylinder length=0.091350 radius=0.044983; visual mesh filename=package://galbot_one_description/meshes/arm/base.glb scale=1 1 1
- link left_camera_link: geometry visual mesh filename=file:///home/fiveages/ros2_ws/install/sensor_models/share/s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
- link left_ear_camera: geometry visual mesh filename=file:///home/fiveages/ros2_ws/install/sensor_models/share/s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
- link left_flange_link: geometry visual mesh filename=file:///home/fiveages/ros2_ws/install/galbot_charlie_descri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 scale=1 1 1
- link left_gripper_base_link: geometry collision mesh filename=package://galbot_one_description/meshes/gripper_hitbot/conv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; visual mesh filename=package://galbot_one_description/meshes/gripper_hitbot/visu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
- link left_gripper_link1: geometry collision mesh filename=package://galbot_one_description/meshes/gripper_hitbot/conv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; visual mesh filename=package://galbot_one_description/meshes/gripper_hitbot/visu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
- link left_gripper_link2: geometry collision mesh filename=package://galbot_one_description/meshes/gripper_hitbot/conv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; visual mesh filename=package://galbot_one_description/meshes/gripper_hitbot/visu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
- link left_gripper_link3: geometry collision mesh filename=package://galbot_one_description/meshes/gripper_hitbot/conv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; visual mesh filename=package://galbot_one_description/meshes/gripper_hitbot/visu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
- link left_gripper_link4: geometry collision mesh filename=package://galbot_one_description/meshes/gripper_hitbot/conv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; visual mesh filename=package://galbot_one_description/meshes/gripper_hitbot/visu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
- link left_gripper_link5: geometry collision mesh filename=package://galbot_one_description/meshes/gripper_hitbot/conv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; visual mesh filename=package://galbot_one_description/meshes/gripper_hitbot/visu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
- link left_gripper_link6: geometry collision mesh filename=package://galbot_one_description/meshes/gripper_hitbot/conv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; visual mesh filename=package://galbot_one_description/meshes/gripper_hitbot/visu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
- link left_link1: geometry collision cylinder length=0.068650 radius=0.044983; visual mesh filename=package://galbot_one_description/meshes/arm/link1.glb
- link left_link2: geometry collision cylinder length=0.19825 radius=0.044983; visual mesh filename=package://galbot_one_description/meshes/arm/link2.glb scale=1 1 1
- link left_link3: geometry collision cylinder length=0.223485 radius=0.044983; visual mesh filename=package://galbot_one_description/meshes/arm/link3.glb
- link left_link4: geometry collision cylinder length=0.16085 radius=0.044983; visual mesh filename=package://galbot_one_description/meshes/arm/link4.glb
- link left_link5: geometry collision mesh filename=file:///home/fiveages/ros2_ws/install/galbot_charlie_descri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; visual mesh filename=file:///home/fiveages/ros2_ws/install/galbot_charlie_descri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
- link left_link6: geometry collision mesh filename=file:///home/fiveages/ros2_ws/install/galbot_charlie_descri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; visual mesh filename=file:///home/fiveages/ros2_ws/install/galbot_charlie_descri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
- link left_link7: geometry collision mesh filename=file:///home/fiveages/ros2_ws/install/galbot_charlie_descri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; visual mesh filename=file:///home/fiveages/ros2_ws/install/galbot_charlie_descri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
- link leg_base_link: geometry visual mesh filename=package://galbot_one_description/meshes/leg/leg_base.glb
- link leg_link1: geometry visual mesh filename=package://galbot_one_description/meshes/leg/leg_link1.glb
- link leg_link2: geometry visual mesh filename=package://galbot_one_description/meshes/leg/leg_link2.glb
- link leg_link3: geometry visual mesh filename=package://galbot_one_description/meshes/leg/leg_link3.glb
- link leg_link4: geometry visual mesh filename=package://galbot_one_description/meshes/leg/leg_link4.glb
- link omni_chassis_base_link: geometry collision cylinder length=0.2 radius=0.3; visual mesh filename=package://galbot_one_description/meshes/chassis/chassis.glb
- link right_base_link: geometry collision cylinder length=0.091350 radius=0.044983; visual mesh filename=package://galbot_one_description/meshes/arm/base.glb scale=1 -1 1
- link right_camera_link: geometry visual mesh filename=file:///home/fiveages/ros2_ws/install/sensor_models/share/s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
- link right_ear_camera: geometry visual mesh filename=file:///home/fiveages/ros2_ws/install/sensor_models/share/s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
- link right_flange_link: geometry visual mesh filename=file:///home/fiveages/ros2_ws/install/galbot_charlie_descri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 scale=1 -1 1
- link right_gripper_base_link: geometry collision mesh filename=package://galbot_one_description/meshes/gripper_hitbot/conv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; visual mesh filename=package://galbot_one_description/meshes/gripper_hitbot/visu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
- link right_gripper_link1: geometry collision mesh filename=package://galbot_one_description/meshes/gripper_hitbot/conv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; visual mesh filename=package://galbot_one_description/meshes/gripper_hitbot/visu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
- link right_gripper_link2: geometry collision mesh filename=package://galbot_one_description/meshes/gripper_hitbot/conv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; visual mesh filename=package://galbot_one_description/meshes/gripper_hitbot/visu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
- link right_gripper_link3: geometry collision mesh filename=package://galbot_one_description/meshes/gripper_hitbot/conv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; visual mesh filename=package://galbot_one_description/meshes/gripper_hitbot/visu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
- link right_gripper_link4: geometry collision mesh filename=package://galbot_one_description/meshes/gripper_hitbot/conv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; visual mesh filename=package://galbot_one_description/meshes/gripper_hitbot/visu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
- link right_gripper_link5: geometry collision mesh filename=package://galbot_one_description/meshes/gripper_hitbot/conv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; visual mesh filename=package://galbot_one_description/meshes/gripper_hitbot/visu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
- link right_gripper_link6: geometry collision mesh filename=package://galbot_one_description/meshes/gripper_hitbot/conv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; visual mesh filename=package://galbot_one_description/meshes/gripper_hitbot/visu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
- link right_link1: geometry collision cylinder length=0.068650 radius=0.044983; visual mesh filename=package://galbot_one_description/meshes/arm/link1.glb
- link right_link2: geometry collision cylinder length=0.19825 radius=0.044983; visual mesh filename=package://galbot_one_description/meshes/arm/link2.glb scale=-1 1 1
- link right_link3: geometry collision cylinder length=0.223485 radius=0.044983; visual mesh filename=package://galbot_one_description/meshes/arm/link3.glb
- link right_link4: geometry collision cylinder length=0.16085 radius=0.044983; visual mesh filename=package://galbot_one_description/meshes/arm/link4.glb
- link right_link5: geometry collision mesh filename=file:///home/fiveages/ros2_ws/install/galbot_charlie_descri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; visual mesh filename=file:///home/fiveages/ros2_ws/install/galbot_charlie_descri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
- link right_link6: geometry collision mesh filename=file:///home/fiveages/ros2_ws/install/galbot_charlie_descri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; visual mesh filename=file:///home/fiveages/ros2_ws/install/galbot_charlie_descri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
- link right_link7: geometry collision mesh filename=file:///home/fiveages/ros2_ws/install/galbot_charlie_descri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; visual mesh filename=file:///home/fiveages/ros2_ws/install/galbot_charlie_descri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
- link torso_base_link: geometry collision box size=0.155192 0.181326 0.165600; collision box size=0.232789 0.271990 0.248400
- link wheel_1: geometry visual mesh filename=file:///home/fiveages/ros2_ws/install/component_models/shar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
- link wheel_2: geometry visual mesh filename=file:///home/fiveages/ros2_ws/install/component_models/shar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
- link wheel_3: geometry visual mesh filename=file:///home/fiveages/ros2_ws/install/component_models/shar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
- link wheel_4: geometry visual mesh filename=file:///home/fiveages/ros2_ws/install/component_models/shar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
Joints:
- removed joint leg_joint
- removed joint leg_joint1
- removed joint leg_joint2
- removed joint leg_joint3
- removed joint leg_joint4
- added joint body_joint: type fixed, parent omni_chassis_leg_mount_link, child leg_base_link, origin rpy=1.5707963267948966 0 0
- added joint body_joint1: type revolute, parent leg_base_link, child leg_link1, origin xyz=0 0 -0.087 rpy=-3.141592653589793 0 2.756573021, axis 0 0 1, limit lower=0 upper=0.994837674 effort=169 velocity=2.3
- added joint body_joint2: type revolute, parent leg_link1, child leg_link2, origin xyz=0.45 0 0 rpy=-3.141592653589793 0 2.756573021, axis 0 0 1, limit lower=0 upper=3.141592653589793 effort=169 velocity=2.3
- added joint body_joint3: type revolute, parent leg_link2, child leg_link3, origin xyz=0.39 0 0 rpy=-3.141592653589793 0 -3.141592653589793, axis 0 0 1, limit lower=0 upper=2.356194490192345 effort=84 velocity=2.83
- added joint body_joint4: type revolute, parent leg_link3, child leg_link4, origin rpy=1.5707963267948966 0 -3.141592653589793, axis 0 0 1, limit lower=-1.5707963267948966 upper=1.5707963267948966 effort=30 velocity=3.56
- joint left_joint: parent left_link7 -> left_arm_end_effector_mount_link
- joint right_joint: parent right_link7 -> right_arm_end_effector_mount_link
