Commit message: fix body name

File: galbot_charlie_description/xacro/components/arm.xacro (robot description, xacro)
@@ -1,247 +1,249 @@
 <?xml version="1.0" ?>
 <robot xmlns:xacro="http://www.ros.org/wiki/xacro">
-  <xacro:property name="PI" value="3.141592653589793"/>
-  <xacro:macro name="GalbotCharlieArmCamera" params="name direction:=1">
-    <xacro:property name="prefix" value="${name}_"/>
-    <link name="${prefix}arm_end_effector_mount_link">
-      <inertial>
-        <origin rpy="0 0 0" xyz="0 0 0"/>
-        <mass value="0"/>
-        <inertia ixx="0" ixy="0" ixz="0" iyy="0" iyz="0" izz="0"/>
-      </inertial>
-    </link>
-    <joint name="${prefix}arm_end_effector_mount_joint" type="fixed">
-      <origin rpy="${-PI/2 * direction} 0 ${PI}" xyz="-0.083 0 0"/>
-      <parent link="${prefix}link7"/>
-      <child link="${prefix}arm_end_effector_mount_link"/>
-    </joint>
-    <link name="${prefix}flange_link">
-      <inertial>
-        <origin rpy="0 0 0" xyz="0.052829 -0.00096484 0.013285"/>
-        <mass value="0.25733"/>
-        <inertia ixx="0.0002175" ixy="-2.5433E-06" ixz="4.0586E-06" iyy="5.3894E-05" iyz="-1.8533E-06" izz="0.00025319"/>
-      </inertial>
-      <visual>
-        <origin rpy="0 0 0" xyz="0 0 0"/>
-        <geometry>
-          <mesh filename="file://$(find galbot_charlie_description)/meshs/camera/camera_support.glb" scale="1 ${direction} 1"/>
-        </geometry>
-      </visual>
-    </link>
-    <joint name="${prefix}joint" type="fixed">
-      <origin rpy="0 0 0" xyz="0 0 0"/>
-      <parent link="${prefix}arm_end_effector_mount_link"/>
-      <child link="${prefix}flange_link"/>
-    </joint>
-    <link name="${prefix}camera_link">
-      <visual>
-        <geometry>
-          <mesh filename="file://$(find sensor_models)/meshes/realsense/d415.glb"  />
-        </geometry>
-      </visual>
-    </link>
-    <joint name="${prefix}camera_joint" type="fixed">
-      <origin rpy="-0.27 -${PI/2} 0 " xyz=" -0.072196  ${0.054731 * direction} 0 "/>(后)(右)(下)
-      <parent link="${prefix}flange_link"/>
-      <child link="${prefix}camera_link"/>
-    </joint>
-  </xacro:macro>
-  <!-- one-style macro: name + direction + prefix -->
-  <xacro:macro name="galbot_charlie_arm" params="name direction:=1 parent">
-    <xacro:property name="prefix" value="${name}_"/>
-    <link name="${prefix}base_link">
-      <inertial>
-        <origin xyz="${0.00056868 * direction} ${-5.0139e-06 * direction} -0.030184"/>
-        <mass value="1.1015"/>
-        <inertia ixx="0.00056381" ixy="${1.1123e-07 * direction}" ixz="${2.1236e-05 * direction}" iyy="0.00057439" iyz="${-1.685e-07 * direction}" izz="0.00068513"/>
-      </inertial>
-      <visual>
-        <geometry>
-          <mesh filename="file://$(find galbot_one_description)/meshes/arm/base.glb" scale="1 ${direction} 1"/>
-        </geometry>
-      </visual>
-      <collision>
-        <geometry>
-          <cylinder length="0.091350" radius="0.044983"/>
-        </geometry>
-      </collision>
-    </link>
-    <joint name="${prefix}arm_joint" type="fixed">
-      <origin xyz="0 0 0"/>
-      <parent link="${parent}"/>
-      <child link="${prefix}base_link"/>
-    </joint>
-    <link name="${prefix}link1">
-      <inertial>
-        <origin xyz="${-3.49009164621467e-05 * direction} ${-0.0108339687508697 * direction} -0.00355285779638756"/>
-        <mass value="1.503"/>
-        <inertia ixx="0.0014148" ixy="1.786E-06" ixz="${8.6353e-07 * direction}" iyy="0.001774" iyz="${-5.8604e-06 * direction}" izz="0.0011021"/>
-      </inertial>
-      <visual>
-        <geometry>
-          <mesh filename="file://$(find galbot_one_description)/meshes/arm/link1.glb"/>
-        </geometry>
-      </visual>
-      <collision>
-        <geometry>
-          <cylinder length="0.068650" radius="0.044983"/>
-        </geometry>
-      </collision>
-    </link>
-    <joint name="${prefix}joint1" type="revolute">
-      <origin xyz="0 0 0.076"/>
-      <parent link="${prefix}base_link"/>
-      <child link="${prefix}link1"/>
-      <axis xyz="0 0 1"/>
-      <limit effort="60" lower="-${PI}" upper="${PI}" velocity="1.5"/>
-    </joint>
-    <link name="${prefix}link2">
-      <inertial>
-        <origin xyz="${0.0011542937189659 * direction} ${0.125918427333295 * direction} 0.00403909337671848"/>
-        <mass value="1.45678998733303"/>
-        <inertia ixx="0.00269801896410487" ixy="4.63119567548212E-05" ixz="${1.77748665814381e-05 * direction}" iyy="0.00131692955308753" iyz="${0.000382862812261171 * direction}" izz="0.00264831680492027"/>
-      </inertial>
-      <visual>
-        <geometry>
-          <mesh filename="file://$(find galbot_one_description)/meshes/arm/link2.glb" scale="${direction} 1 1"/>
-        </geometry>
-      </visual>
-      <collision>
-        <origin rpy="${PI/2} 0 0" xyz="0 -0.074 0"/>
-        <geometry>
-          <cylinder length="0.19825" radius="0.044983"/>
-        </geometry>
-      </collision>
-    </link>
-    <joint name="${prefix}joint2" type="revolute">
-      <origin rpy="-${PI/2} 0 ${PI}"/>
-      <parent link="${prefix}link1"/>
-      <child link="${prefix}link2"/>
-      <axis xyz="0 0 ${direction}"/>
-      <limit effort="60" lower="-${PI/2}" upper="1.83" velocity="1.5"/>
-    </joint>
-    <link name="${prefix}link3">
-      <inertial>
-        <origin xyz="0.000352305768300032 -0.00726519320891149 -0.0216211172275835"/>
-        <mass value="1.19882450635199"/>
-        <inertia ixx="0.00220937810713451" ixy="-1.39043584660172E-05" ixz="1.48996603867525E-06" iyy="0.00236018741531392" iyz="4.46418780437893E-05" izz="0.000843927012398976"/>
-      </inertial>
-      <visual>
-        <geometry>
-          <mesh filename="file://$(find galbot_one_description)/meshes/arm/link3.glb"/>
-        </geometry>
-      </visual>
-      <collision>
-        <origin xyz="0 0 -0.074"/>
-        <geometry>
-          <cylinder length="0.223485" radius="0.044983"/>
-        </geometry>
-      </collision>
-    </link>
-    <joint name="${prefix}joint3" type="revolute">
-      <origin rpy="${PI/2} ${PI/2 * direction} 0" xyz="0 -0.35 0"/>
-      <parent link="${prefix}link2"/>
-      <child link="${prefix}link3"/>
-      <axis xyz="0 0 1"/>
-      <limit effort="30" lower="-${PI}" upper="${PI}" velocity="1.5"/>
-    </joint>
-    <link name="${prefix}link4">
-      <inertial>
-        <origin xyz="1.6053E-07 -0.0841 0.0032663"/>
-        <mass value="0.86736"/>
-        <inertia ixx="0.00087789" ixy="1.0686E-08" ixz="-1.4208E-07" iyy="0.00058539" iyz="-0.0001428" izz="0.00082718"/>
-      </inertial>
-      <visual>
-        <geometry>
-          <mesh filename="file://$(find galbot_one_description)/meshes/arm/link4.glb"/>
-        </geometry>
-      </visual>
-      <collision>
-        <origin rpy="${PI/2} 0 0" xyz="0 -0.14 0"/>
-        <geometry>
-          <cylinder length="0.16085" radius="0.044983"/>
-        </geometry>
-      </collision>
-    </link>
-    <joint name="${prefix}joint4" type="revolute">
-      <origin rpy="-${PI/2} 0 ${PI}"/>
-      <parent link="${prefix}link3"/>
-      <child link="${prefix}link4"/>
-      <axis xyz="0 0 1"/>
-      <limit effort="30" lower="-2.1" upper="2.1" velocity="1.5"/>
-    </joint>
-    <link name="${prefix}link5">
-      <inertial>
-        <origin xyz="${-0.00201 * direction} ${0.00042 * direction} -0.14589"/>
-        <mass value="1.22"/>
-        <inertia ixx="0.03428" ixy="0.00001" ixz="${0.000355 * direction}" iyy="0.03366" iyz="${0.000075 * direction}" izz="0.00222"/>
-      </inertial>
-      <visual>
-        <geometry>
-          <mesh filename="file://$(find galbot_charlie_description)/meshs/arm/link5.glb"/>
-        </geometry>
-      </visual>
-      <collision>
-        <geometry>
-          <mesh filename="file://$(find galbot_charlie_description)/meshs/arm/link5.glb"/>
-        </geometry>
-      </collision>
-    </link>
-    <joint name="${prefix}joint5" type="revolute">
-      <origin rpy="${PI/2} ${PI} 0" xyz="0 -0.36 0"/>
-      <parent link="${prefix}link4"/>
-      <child link="${prefix}link5"/>
-      <axis xyz="0 0 1"/>
-      <limit effort="10" lower="-2.9" upper="2.9" velocity="1.5"/>
-    </joint>
-    <link name="${prefix}link6">
-      <inertial>
-        <origin xyz="0 ${-0.01031 * direction} 0"/>
-        <mass value="0.43"/>
-        <inertia ixx="0.00051" ixy="0" ixz="0" iyy="0.00070" iyz="0" izz="0.00091"/>
-      </inertial>
-      <visual>
-        <geometry>
-          <mesh filename="file://$(find galbot_charlie_description)/meshs/arm/link6.glb"/>
-        </geometry>
-      </visual>
-      <collision>
-        <geometry>
-          <mesh filename="file://$(find galbot_charlie_description)/meshs/arm/link6.glb"/>
-        </geometry>
-      </collision>
-    </link>
-    <joint name="${prefix}joint6" type="revolute">
-      <origin rpy="-${PI/2} ${PI/2} ${PI}" xyz="0 0 0"/>
-      <parent link="${prefix}link5"/>
-      <child link="${prefix}link6"/>
-      <axis xyz="0 0 1"/>
-      <limit effort="10" lower="-0.785398163" upper="0.785398163" velocity="1.5"/>
-    </joint>
-    <link name="${prefix}link7">
-      <inertial>
-        <origin xyz="-0.03291 0.00799 -0.00131"/>
-        <mass value="0.6"/>
-        <inertia ixx="0.00124" ixy="0.00015" ixz="0.000125" iyy="0.00198" iyz="0.000055" izz="0.00164"/>
-      </inertial>
-      <visual>
-        <geometry>
-          <mesh filename="file://$(find galbot_charlie_description)/meshs/arm/link7.glb"/>
-        </geometry>
-      </visual>
-      <collision>
-        <geometry>
-          <mesh filename="file://$(find galbot_charlie_description)/meshs/arm/link7.glb"/>
-        </geometry>
-      </collision>
-    </link>
-    <joint name="${prefix}joint7" type="revolute">
-      <origin rpy="${PI/2 * direction} 0 0" xyz="0 0 0"/>
-      <parent link="${prefix}link6"/>
-      <child link="${prefix}link7"/>
-      <axis xyz="0 0 1"/>
-      <limit effort="10" lower="-1.4" upper="1.4" velocity="1.5"/>
-    </joint>
-    <xacro:GalbotCharlieArmCamera name="${name}" direction="${direction}"/>
-  </xacro:macro>
+	<xacro:property name="PI" value="3.141592653589793"/>
+	<xacro:macro name="GalbotCharlieArmCamera" params="name direction:=1">
+		<xacro:property name="prefix" value="${name}_"/>
+		<link name="${prefix}arm_end_effector_mount_link"/>
+		<joint name="${prefix}arm_end_effector_mount_joint" type="fixed">
+			<origin rpy="${-PI/2 * direction} 0 ${PI}" xyz="-0.083 0 0"/>
+			<parent link="${prefix}link7"/>
+			<child link="${prefix}arm_end_effector_mount_link"/>
+		</joint>
+		<link name="${prefix}flange_link">
+			<inertial>
+				<origin rpy="0 0 0" xyz="0.052829 -0.00096484 0.013285"/>
+				<mass value="0.25733"/>
+				<inertia ixx="0.0002175" ixy="-2.5433E-06" ixz="4.0586E-06" iyy="5.3894E-05" iyz="-1.8533E-06"
+				         izz="0.00025319"/>
+			</inertial>
+			<visual>
+				<origin rpy="0 0 0" xyz="0 0 0"/>
+				<geometry>
+					<mesh filename="file://$(find galbot_charlie_description)/meshs/camera/camera_support.glb"
+					      scale="1 ${direction} 1"/>
+				</geometry>
+			</visual>
+		</link>
+		<joint name="${prefix}joint" type="fixed">
+			<origin rpy="0 0 0" xyz="0 0 0"/>
+			<parent link="${prefix}arm_end_effector_mount_link"/>
+			<child link="${prefix}flange_link"/>
+		</joint>
+		<link name="${prefix}camera_link">
+			<visual>
+				<geometry>
+					<mesh filename="file://$(find sensor_models)/meshes/realsense/d415.glb"/>
+				</geometry>
+			</visual>
+		</link>
+		<joint name="${prefix}camera_joint" type="fixed">
+			<origin rpy="-0.27 -${PI/2} 0 " xyz=" -0.072196  ${0.054731 * direction} 0 "/>(后)(右)(下)
+			<parent link="${prefix}flange_link"/>
+			<child link="${prefix}camera_link"/>
+		</joint>
+	</xacro:macro>
+	<!-- one-style macro: name + direction + prefix -->
+	<xacro:macro name="galbot_charlie_arm" params="name direction:=1 parent">
+		<xacro:property name="prefix" value="${name}_"/>
+		<link name="${prefix}base_link">
+			<inertial>
+				<origin xyz="${0.00056868 * direction} ${-5.0139e-06 * direction} -0.030184"/>
+				<mass value="1.1015"/>
+				<inertia ixx="0.00056381" ixy="${1.1123e-07 * direction}" ixz="${2.1236e-05 * direction}" iyy="0.00057439"
+				         iyz="${-1.685e-07 * direction}" izz="0.00068513"/>
+			</inertial>
+			<visual>
+				<geometry>
+					<mesh filename="file://$(find galbot_one_description)/meshes/arm/base.glb" scale="1 ${direction} 1"/>
+				</geometry>
+			</visual>
+			<collision>
+				<geometry>
+					<cylinder length="0.091350" radius="0.044983"/>
+				</geometry>
+			</collision>
+		</link>
+		<joint name="${prefix}arm_joint" type="fixed">
+			<origin xyz="0 0 0"/>
+			<parent link="${parent}"/>
+			<child link="${prefix}base_link"/>
+		</joint>
+		<link name="${prefix}link1">
+			<inertial>
+				<origin xyz="${-3.49009164621467e-05 * direction} ${-0.0108339687508697 * direction} -0.00355285779638756"/>
+				<mass value="1.503"/>
+				<inertia ixx="0.0014148" ixy="1.786E-06" ixz="${8.6353e-07 * direction}" iyy="0.001774"
+				         iyz="${-5.8604e-06 * direction}" izz="0.0011021"/>
+			</inertial>
+			<visual>
+				<geometry>
+					<mesh filename="file://$(find galbot_one_description)/meshes/arm/link1.glb"/>
+				</geometry>
+			</visual>
+			<collision>
+				<geometry>
+					<cylinder length="0.068650" radius="0.044983"/>
+				</geometry>
+			</collision>
+		</link>
+		<joint name="${prefix}joint1" type="revolute">
+			<origin xyz="0 0 0.076"/>
+			<parent link="${prefix}base_link"/>
+			<child link="${prefix}link1"/>
+			<axis xyz="0 0 1"/>
+			<limit effort="60" lower="-${PI}" upper="${PI}" velocity="1.5"/>
+		</joint>
+		<link name="${prefix}link2">
+			<inertial>
+				<origin xyz="${0.0011542937189659 * direction} ${0.125918427333295 * direction} 0.00403909337671848"/>
+				<mass value="1.45678998733303"/>
+				<inertia ixx="0.00269801896410487" ixy="4.63119567548212E-05" ixz="${1.77748665814381e-05 * direction}"
+				         iyy="0.00131692955308753" iyz="${0.000382862812261171 * direction}" izz="0.00264831680492027"/>
+			</inertial>
+			<visual>
+				<geometry>
+					<mesh filename="file://$(find galbot_one_description)/meshes/arm/link2.glb" scale="${direction} 1 1"/>
+				</geometry>
+			</visual>
+			<collision>
+				<origin rpy="${PI/2} 0 0" xyz="0 -0.074 0"/>
+				<geometry>
+					<cylinder length="0.19825" radius="0.044983"/>
+				</geometry>
+			</collision>
+		</link>
+		<joint name="${prefix}joint2" type="revolute">
+			<origin rpy="-${PI/2} 0 ${PI}"/>
+			<parent link="${prefix}link1"/>
+			<child link="${prefix}link2"/>
+			<axis xyz="0 0 ${direction}"/>
+			<limit effort="60" lower="-${PI/2}" upper="1.83" velocity="1.5"/>
+		</joint>
+		<link name="${prefix}link3">
+			<inertial>
+				<origin xyz="0.000352305768300032 -0.00726519320891149 -0.0216211172275835"/>
+				<mass value="1.19882450635199"/>
+				<inertia ixx="0.00220937810713451" ixy="-1.39043584660172E-05" ixz="1.48996603867525E-06"
+				         iyy="0.00236018741531392" iyz="4.46418780437893E-05" izz="0.000843927012398976"/>
+			</inertial>
+			<visual>
+				<geometry>
+					<mesh filename="file://$(find galbot_one_description)/meshes/arm/link3.glb"/>
+				</geometry>
+			</visual>
+			<collision>
+				<origin xyz="0 0 -0.074"/>
+				<geometry>
+					<cylinder length="0.223485" radius="0.044983"/>
+				</geometry>
+			</collision>
+		</link>
+		<joint name="${prefix}joint3" type="revolute">
+			<origin rpy="${PI/2} ${PI/2 * direction} 0" xyz="0 -0.35 0"/>
+			<parent link="${prefix}link2"/>
+			<child link="${prefix}link3"/>
+			<axis xyz="0 0 1"/>
+			<limit effort="30" lower="-${PI}" upper="${PI}" velocity="1.5"/>
+		</joint>
+		<link name="${prefix}link4">
+			<inertial>
+				<origin xyz="1.6053E-07 -0.0841 0.0032663"/>
+				<mass value="0.86736"/>
+				<inertia ixx="0.00087789" ixy="1.0686E-08" ixz="-1.4208E-07" iyy="0.00058539" iyz="-0.0001428"
+				         izz="0.00082718"/>
+			</inertial>
+			<visual>
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
File: galbot_one_description/urdf/galbot_one.urdf (robot description, URDF)
Before this commit: robot galbot_one, 67 links, 66 joints
Joints:
- removed joint leg_joint
- removed joint leg_joint1
- removed joint leg_joint2
- removed joint leg_joint3
- removed joint leg_joint4
- added joint body_joint: type fixed, parent omni_chassis_leg_mount_link, child leg_base_link, origin rpy=1.5707963267948966 0 0
- added joint body_joint1: type revolute, parent leg_base_link, child leg_link1, origin xyz=0 0 -0.087 rpy=-3.141592653589793 0 2.756573021, axis 0 0 1, limit lower=0 upper=0.994837674 effort=169 velocity=2.3
- added joint body_joint2: type revolute, parent leg_link1, child leg_link2, origin xyz=0.45 0 0 rpy=-3.141592653589793 0 2.756573021, axis 0 0 1, limit lower=0 upper=3.141592653589793 effort=169 velocity=2.3
- added joint body_joint3: type revolute, parent leg_link2, child leg_link3, origin xyz=0.39 0 0 rpy=-3.141592653589793 0 -3.141592653589793, axis 0 0 1, limit lower=0 upper=2.356194490192345 effort=84 velocity=2.83
- added joint body_joint4: type revolute, parent leg_link3, child leg_link4, origin rpy=1.5707963267948966 0 -3.141592653589793, axis 0 0 1, limit lower=-1.5707963267948966 upper=1.5707963267948966 effort=30 velocity=3.56

File: galbot_one_description/urdf/galbot_one_galbot_gripper.urdf (robot description, URDF)
Before this commit: robot galbot_one, 69 links, 68 joints
Joints:
- removed joint leg_joint
- removed joint leg_joint1
- removed joint leg_joint2
- removed joint leg_joint3
- removed joint leg_joint4
- added joint body_joint: type fixed, parent omni_chassis_leg_mount_link, child leg_base_link, origin rpy=1.5707963267948966 0 0
- added joint body_joint1: type revolute, parent leg_base_link, child leg_link1, origin xyz=0 0 -0.087 rpy=-3.141592653589793 0 2.756573021, axis 0 0 1, limit lower=0 upper=0.994837674 effort=169 velocity=2.3
- added joint body_joint2: type revolute, parent leg_link1, child leg_link2, origin xyz=0.45 0 0 rpy=-3.141592653589793 0 2.756573021, axis 0 0 1, limit lower=0 upper=3.141592653589793 effort=169 velocity=2.3
- added joint body_joint3: type revolute, parent leg_link2, child leg_link3, origin xyz=0.39 0 0 rpy=-3.141592653589793 0 -3.141592653589793, axis 0 0 1, limit lower=0 upper=2.356194490192345 effort=84 velocity=2.83
- added joint body_joint4: type revolute, parent leg_link3, child leg_link4, origin rpy=1.5707963267948966 0 -3.141592653589793, axis 0 0 1, limit lower=-1.5707963267948966 upper=1.5707963267948966 effort=30 velocity=3.56
