Commit message: update galbot charlie

File: galbot_charlie_description/urdf/galbot_charlie.urdf (robot description, URDF)
Before this commit: robot galbot_charlie, 64 links, 65 joints
Links:
- link chassis_lidar: geometry visual mesh filename=package://sensor_models/meshes/mid360/mid360.obj
- link head_back_camera: geometry visual mesh filename=package://sensor_models/meshes/realsense/d415.glb
- link head_front_camera: geometry visual mesh filename=package://sensor_models/meshes/realsense/d435.glb
- link left_camera_link: geometry visual mesh filename=package://sensor_models/meshes/realsense/d415.glb
- link left_ear_camera: geometry visual mesh filename=package://sensor_models/meshes/usb_camera/camera_01.glb
- link left_flange_link: geometry visual mesh filename=package://galbot_charlie_description/meshs/camera/camera_su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 scale=1 1 1
- link left_link5: geometry collision mesh filename=package://galbot_charlie_description/meshs/arm/link5.glb; visual mesh filename=package://galbot_charlie_description/meshs/arm/link5.glb
- link left_link6: geometry collision mesh filename=package://galbot_charlie_description/meshs/arm/link6.glb; visual mesh filename=package://galbot_charlie_description/meshs/arm/link6.glb
- link left_link7: geometry collision mesh filename=package://galbot_charlie_description/meshs/arm/link7.glb; visual mesh filename=package://galbot_charlie_description/meshs/arm/link7.glb
- link right_camera_link: geometry visual mesh filename=package://sensor_models/meshes/realsense/d415.glb
- link right_ear_camera: geometry visual mesh filename=package://sensor_models/meshes/usb_camera/camera_01.glb
- link right_flange_link: geometry visual mesh filename=package://galbot_charlie_description/meshs/camera/camera_su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 scale=1 -1 1
- link right_link5: geometry collision mesh filename=package://galbot_charlie_description/meshs/arm/link5.glb; visual mesh filename=package://galbot_charlie_description/meshs/arm/link5.glb
- link right_link6: geometry collision mesh filename=package://galbot_charlie_description/meshs/arm/link6.glb; visual mesh filename=package://galbot_charlie_description/meshs/arm/link6.glb
- link right_link7: geometry collision mesh filename=package://galbot_charlie_description/meshs/arm/link7.glb; visual mesh filename=package://galbot_charlie_description/meshs/arm/link7.glb
- link wheel_1: geometry visual mesh filename=package://component_models/meshes/omniwheel_10.glb
- link wheel_2: geometry visual mesh filename=package://component_models/meshes/omniwheel_10.glb
- link wheel_3: geometry visual mesh filename=package://component_models/meshes/omniwheel_10.glb
- link wheel_4: geometry visual mesh filename=package://component_models/meshes/omniwheel_10.glb
Joints:
- removed joint left_arm_joint
- removed joint right_arm_joint
- joint left_camera_joint: origin xyz= -0.072196  0.054731 0  rpy=-0.27 -1.5707963267948966 0  -> xyz=-0.072196 0.054731 0 rpy=-0.27 -1.5707963267948966 0
- joint left_joint: parent left_arm_end_effector_mount_link -> left_link7
- joint right_camera_joint: origin xyz= -0.072196  -0.054731 0  rpy=-0.27 -1.5707963267948966 0  -> xyz=-0.072196 -0.054731 0 rpy=-0.27 -1.5707963267948966 0
- joint right_joint: parent right_arm_end_effector_mount_link -> right_link7

File: galbot_charlie_description/urdf/galbot_charlie_galbot_gripper.urdf (robot description, URDF)
Before this commit: robot galbot_charlie, 66 links, 67 joints
Links:
- link chassis_lidar: geometry visual mesh filename=package://sensor_models/meshes/mid360/mid360.obj
- link head_back_camera: geometry visual mesh filename=package://sensor_models/meshes/realsense/d415.glb
- link head_base_link: geometry visual mesh filename=package://galbot_one_description/meshes/head/head_base.glb
- link head_front_camera: geometry visual mesh filename=package://sensor_models/meshes/realsense/d435.glb
- link head_link1: geometry visual mesh filename=package://galbot_one_description/meshes/head/head_link1.glb
- link head_link2: geometry visual mesh filename=package://galbot_one_description/meshes/head/head_link2.glb
- link left_base_link: geometry collision cylinder length=0.091350 radius=0.044983; visual mesh filename=package://galbot_one_description/meshes/arm/base.glb scale=1 1 1
- link left_camera_link: geometry visual mesh filename=package://sensor_models/meshes/realsense/d415.glb
- link left_ear_camera: geometry visual mesh filename=package://sensor_models/meshes/usb_camera/camera_01.glb
- link left_flange_link: geometry visual mesh filename=package://galbot_charlie_description/meshs/camera/camera_su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 scale=1 1 1
- link left_gripper_base: geometry collision mesh filename=package://galbot_foxtrot_description/meshes/collision/gripp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; visual mesh filename=package://galbot_foxtrot_description/meshes/visual/gripper/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
- link left_gripper_flange: geometry visual mesh filename=package://galbot_foxtrot_description/meshes/visual/gripper/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
- link left_gripper_l_finger_link: geometry collision mesh filename=package://galbot_foxtrot_description/meshes/collision/gripp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; visual mesh filename=package://galbot_foxtrot_description/meshes/visual/gripper/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
- link left_gripper_l_inner_knuckle_link: geometry collision mesh filename=package://galbot_foxtrot_description/meshes/collision/gripp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; visual mesh filename=package://galbot_foxtrot_description/meshes/visual/gripper/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
- link left_gripper_l_knuckle_link: geometry collision mesh filename=package://galbot_foxtrot_description/meshes/collision/gripp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; visual mesh filename=package://galbot_foxtrot_description/meshes/visual/gripper/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
- link left_gripper_r_finger_link: geometry collision mesh filename=package://galbot_foxtrot_description/meshes/collision/gripp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 scale=1 -1 1; visual mesh filename=package://galbot_foxtrot_description/meshes/visual/gripper/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 scale=1 -1 1
- link left_gripper_r_inner_knuckle_link: geometry collision mesh filename=package://galbot_foxtrot_description/meshes/collision/gripp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; visual mesh filename=package://galbot_foxtrot_description/meshes/visual/gripper/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
- link left_gripper_r_knuckle_link: geometry collision mesh filename=package://galbot_foxtrot_description/meshes/collision/gripp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; visual mesh filename=package://galbot_foxtrot_description/meshes/visual/gripper/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
- link left_link1: geometry collision cylinder length=0.068650 radius=0.044983; visual mesh filename=package://galbot_one_description/meshes/arm/link1.glb
- link left_link2: geometry collision cylinder length=0.19825 radius=0.044983; visual mesh filename=package://galbot_one_description/meshes/arm/link2.glb scale=1 1 1
- link left_link3: geometry collision cylinder length=0.223485 radius=0.044983; visual mesh filename=package://galbot_one_description/meshes/arm/link3.glb
- link left_link4: geometry collision cylinder length=0.16085 radius=0.044983; visual mesh filename=package://galbot_one_description/meshes/arm/link4.glb
- link left_link5: geometry collision mesh filename=package://galbot_charlie_description/meshs/arm/link5.glb; visual mesh filename=package://galbot_charlie_description/meshs/arm/link5.glb
- link left_link6: geometry collision mesh filename=package://galbot_charlie_description/meshs/arm/link6.glb; visual mesh filename=package://galbot_charlie_description/meshs/arm/link6.glb
- link left_link7: geometry collision mesh filename=package://galbot_charlie_description/meshs/arm/link7.glb; visual mesh filename=package://galbot_charlie_description/meshs/arm/link7.glb
- link leg_base_link: geometry visual mesh filename=package://galbot_one_description/meshes/leg/leg_base.glb
- link leg_link1: geometry visual mesh filename=package://galbot_one_description/meshes/leg/leg_link1.glb
- link leg_link2: geometry visual mesh filename=package://galbot_one_description/meshes/leg/leg_link2.glb
- link leg_link3: geometry visual mesh filename=package://galbot_one_description/meshes/leg/leg_link3.glb
- link leg_link4: geometry visual mesh filename=package://galbot_one_description/meshes/leg/leg_link4.glb
- link omni_chassis_base_link: geometry collision cylinder length=0.2 radius=0.3; visual mesh filename=package://galbot_one_description/meshes/chassis/chassis.glb
- link right_base_link: geometry collision cylinder length=0.091350 radius=0.044983; visual mesh filename=package://galbot_one_description/meshes/arm/base.glb scale=1 -1 1
- link right_camera_link: geometry visual mesh filename=package://sensor_models/meshes/realsense/d415.glb
- link right_ear_camera: geometry visual mesh filename=package://sensor_models/meshes/usb_camera/camera_01.glb
- link right_flange_link: geometry visual mesh filename=package://galbot_charlie_description/meshs/camera/camera_su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 scale=1 -1 1
- link right_gripper_base: geometry collision mesh filename=package://galbot_foxtrot_description/meshes/collision/gripp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; visual mesh filename=package://galbot_foxtrot_description/meshes/visual/gripper/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
- link right_gripper_flange: geometry visual mesh filename=package://galbot_foxtrot_description/meshes/visual/gripper/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
- link right_gripper_l_finger_link: geometry collision mesh filename=package://galbot_foxtrot_description/meshes/collision/gripp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; visual mesh filename=package://galbot_foxtrot_description/meshes/visual/gripper/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
- link right_gripper_l_inner_knuckle_link: geometry collision mesh filename=package://galbot_foxtrot_description/meshes/collision/gripp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; visual mesh filename=package://galbot_foxtrot_description/meshes/visual/gripper/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
- link right_gripper_l_knuckle_link: geometry collision mesh filename=package://galbot_foxtrot_description/meshes/collision/gripp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; visual mesh filename=package://galbot_foxtrot_description/meshes/visual/gripper/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
- link right_gripper_r_finger_link: geometry collision mesh filename=package://galbot_foxtrot_description/meshes/collision/gripp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 scale=1 -1 1; visual mesh filename=package://galbot_foxtrot_description/meshes/visual/gripper/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 scale=1 -1 1
- link right_gripper_r_inner_knuckle_link: geometry collision mesh filename=package://galbot_foxtrot_description/meshes/collision/gripp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; visual mesh filename=package://galbot_foxtrot_description/meshes/visual/gripper/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
- link right_gripper_r_knuckle_link: geometry collision mesh filename=package://galbot_foxtrot_description/meshes/collision/gripp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; visual mesh filename=package://galbot_foxtrot_description/meshes/visual/gripper/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
- link right_link1: geometry collision cylinder length=0.068650 radius=0.044983; visual mesh filename=package://galbot_one_description/meshes/arm/link1.glb
- link right_link2: geometry collision cylinder length=0.19825 radius=0.044983; visual mesh filename=package://galbot_one_description/meshes/arm/link2.glb scale=-1 1 1
- link right_link3: geometry collision cylinder length=0.223485 radius=0.044983; visual mesh filename=package://galbot_one_description/meshes/arm/link3.glb
- link right_link4: geometry collision cylinder length=0.16085 radius=0.044983; visual mesh filename=package://galbot_one_description/meshes/arm/link4.glb
- link right_link5: geometry collision mesh filename=package://galbot_charlie_description/meshs/arm/link5.glb; visual mesh filename=package://galbot_charlie_description/meshs/arm/link5.glb
- link right_link6: geometry collision mesh filename=package://galbot_charlie_description/meshs/arm/link6.glb; visual mesh filename=package://galbot_charlie_description/meshs/arm/link6.glb
- link right_link7: geometry collision mesh filename=package://galbot_charlie_description/meshs/arm/link7.glb; visual mesh filename=package://galbot_charlie_description/meshs/arm/link7.glb
- link torso_base_link: geometry collision box size=0.155192 0.181326 0.165600; collision box size=0.232789 0.271990 0.248400
- link wheel_1: geometry visual mesh filename=package://component_models/meshes/omniwheel_10.glb
- link wheel_2: geometry visual mesh filename=package://component_models/meshes/omniwheel_10.glb
- link wheel_3: geometry visual mesh filename=package://component_models/meshes/omniwheel_10.glb
- link wheel_4: geometry visual mesh filename=package://component_models/meshes/omniwheel_10.glb
Joints:
- removed joint left_arm_joint
- removed joint leg_joint
- removed joint leg_joint1
- removed joint leg_joint2
- removed joint leg_joint3
- removed joint leg_joint4
- removed joint right_arm_joint
- added joint body_joint: type fixed, parent omni_chassis_leg_mount_link, child leg_base_link, origin rpy=1.5707963267948966 0 0
- added joint body_joint1: type revolute, parent leg_base_link, child leg_link1, origin xyz=0 0 -0.087 rpy=-3.141592653589793 0 2.756573021, axis 0 0 1, limit lower=0 upper=0.994837674 effort=169 velocity=2.3
- added joint body_joint2: type revolute, parent leg_link1, child leg_link2, origin xyz=0.45 0 0 rpy=-3.141592653589793 0 2.756573021, axis 0 0 1, limit lower=0 upper=3.141592653589793 effort=169 velocity=2.3
- added joint body_joint3: type revolute, parent leg_link2, child leg_link3, origin xyz=0.39 0 0 rpy=-3.141592653589793 0 -3.141592653589793, axis 0 0 1, limit lower=0 upper=2.356194490192345 effort=84 velocity=2.83
- added joint body_joint4: type revolute, parent leg_link3, child leg_link4, origin rpy=1.5707963267948966 0 -3.141592653589793, axis 0 0 1, limit lower=-1.5707963267948966 upper=1.5707963267948966 effort=30 velocity=3.56
- joint left_camera_joint: origin xyz= -0.072196  0.054731 0  rpy=-0.27 -1.5707963267948966 0  -> xyz=-0.072196 0.054731 0 rpy=-0.27 -1.5707963267948966 0
- joint right_camera_joint: origin xyz= -0.072196  -0.054731 0  rpy=-0.27 -1.5707963267948966 0  -> xyz=-0.072196 -0.054731 0 rpy=-0.27 -1.5707963267948966 0

File: galbot_charlie_description/xacro/component.xacro (robot description, xacro)
@@ -40,6 +40,9 @@
     </joint>
     <xacro:include filename="$(find galbot_charlie_description)/xacro/components/arm.xacro"/>
-    <xacro:galbot_charlie_arm name="left" direction="1" parent="arm_base"/>
-    <xacro:galbot_charlie_arm name="right" direction="-1" parent="arm_base"/>
+    <xacro:include filename="$(find galbot_charlie_description)/xacro/components/camera.xacro"/>
+    <xacro:galbot_charlie_arm name="left" direction="1"/>
+    <xacro:galbot_charlie_arm name="right" direction="-1"/>
+    <xacro:galbot_charlie_arm_camera name="left" direction="1"/>
+    <xacro:galbot_charlie_arm_camera name="right" direction="-1"/>
   </xacro:if>
 </robot>

File: galbot_charlie_description/xacro/components/arm.xacro (robot description, xacro)
@@ -2,47 +2,6 @@
 <robot xmlns:xacro="http://www.ros.org/wiki/xacro">
 	<xacro:property name="PI" value="3.141592653589793"/>
-	<xacro:macro name="GalbotCharlieArmCamera" params="name direction:=1">
-		<xacro:property name="prefix" value="${name}_"/>
-		<link name="${prefix}arm_end_effector_mount_link"/>
-		<joint name="${prefix}arm_end_effector_mount_joint" type="fixed">
-			<origin rpy="${-PI/2 * direction} 0 ${PI}" xyz="-0.083 0 0"/>
-			<parent link="${prefix}link7"/>
-			<child link="${prefix}arm_end_effector_mount_link"/>
-		</joint>
-		<link name="${prefix}flange_link">
-			<inertial>
-				<origin rpy="0 0 0" xyz="0.052829 -0.00096484 0.013285"/>
-				<mass value="0.25733"/>
-				<inertia ixx="0.0002175" ixy="-2.5433E-06" ixz="4.0586E-06" iyy="5.3894E-05" iyz="-1.8533E-06"
-				         izz="0.00025319"/>
-			</inertial>
-			<visual>
-				<origin rpy="0 0 0" xyz="0 0 0"/>
-				<geometry>
-					<mesh filename="file://$(find galbot_charlie_description)/meshs/camera/camera_support.glb"
-					      scale="1 ${direction} 1"/>
-				</geometry>
-			</visual>
-		</link>
-		<joint name="${prefix}joint" type="fixed">
-			<origin rpy="0 0 0" xyz="0 0 0"/>
-			<parent link="${prefix}arm_end_effector_mount_link"/>
-			<child link="${prefix}flange_link"/>
-		</joint>
-		<link name="${prefix}camera_link">
-			<visual>
-				<geometry>
-					<mesh filename="file://$(find sensor_models)/meshes/realsense/d415.glb"/>
-				</geometry>
-			</visual>
-		</link>
-		<joint name="${prefix}camera_joint" type="fixed">
-			<origin rpy="-0.27 -${PI/2} 0 " xyz=" -0.072196  ${0.054731 * direction} 0 "/>(后)(右)(下)
-			<parent link="${prefix}flange_link"/>
-			<child link="${prefix}camera_link"/>
-		</joint>
-	</xacro:macro>
 	<!-- one-style macro: name + direction + prefix -->
-	<xacro:macro name="galbot_charlie_arm" params="name direction:=1 parent">
+	<xacro:macro name="galbot_charlie_arm" params="name direction:=1">
 		<xacro:property name="prefix" value="${name}_"/>
 		<link name="${prefix}base_link">
@@ -64,9 +23,4 @@
 			</collision>
 		</link>
-		<joint name="${prefix}arm_joint" type="fixed">
-			<origin xyz="0 0 0"/>
-			<parent link="${parent}"/>
-			<child link="${prefix}base_link"/>
-		</joint>
 		<link name="${prefix}link1">
 			<inertial>
@@ -245,5 +199,4 @@
 			<limit effort="10" lower="-1.4" upper="1.4" velocity="1.5"/>
 		</joint>
-		<xacro:GalbotCharlieArmCamera name="${name}" direction="${direction}"/>
 	</xacro:macro>
 </robot>

File: galbot_charlie_description/xacro/robot.xacro (robot description, xacro)
@@ -33,7 +33,10 @@
   <xacro:include filename="$(find galbot_one_description)/xacro/components/body.xacro"/>
   <xacro:include filename="$(find galbot_charlie_description)/xacro/components/arm.xacro"/>
+  <xacro:include filename="$(find galbot_charlie_description)/xacro/components/camera.xacro"/>
   <xacro:GalbotOneChassis enable_wheel_joints="$(arg enable_wheel_joints)"/>
-  <xacro:galbot_charlie_arm name="left" direction="1" parent="arm_base"/>
-  <xacro:galbot_charlie_arm name="right" direction="-1" parent="arm_base"/>
+  <xacro:galbot_charlie_arm name="left" direction="1"/>
+  <xacro:galbot_charlie_arm name="right" direction="-1"/>
+  <xacro:galbot_charlie_arm_camera name="left" direction="1"/>
+  <xacro:galbot_charlie_arm_camera name="right" direction="-1"/>
   <joint name="left_arm_mount_joint" type="fixed">
     <origin rpy="0 ${PI} 0" xyz="0 0 -0.13"/>
