Commit message: update galbot one and charlie xacro and urdf

File: galbot_charlie_description/urdf/galbot_charlie.urdf (robot description, URDF)
Before this commit: robot galbot_charlie, 64 links, 63 joints
Links:
- removed link left_arm_end_effector_mount_link
- removed link right_arm_end_effector_mount_link
- added link left_camera_mount_link
- added link right_camera_mount_link
- link left_flange_link: geometry visual mesh filename=package://galbot_one_description/meshes/flange/camera_suppo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 scale=1 1 1
- link right_flange_link: geometry visual mesh filename=package://galbot_one_description/meshes/flange/camera_suppo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 scale=1 -1 1
- link wheel_1: geometry visual mesh filename=file:///home/king/ros2_ws/install/component_models/share/co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
- link wheel_2: geometry visual mesh filename=file:///home/king/ros2_ws/install/component_models/share/co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
- link wheel_3: geometry visual mesh filename=file:///home/king/ros2_ws/install/component_models/share/co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
- link wheel_4: geometry visual mesh filename=file:///home/king/ros2_ws/install/component_models/share/co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
Joints:
- removed joint left_arm_end_effector_mount_joint
- removed joint left_gripper_mount_joint
- removed joint right_arm_end_effector_mount_joint
- removed joint right_gripper_mount_joint
- added joint left_camera_mount_joint: type fixed, parent left_link7, child left_camera_mount_link, origin xyz=0.03 0 0 rpy=1.5707963267948966 0 -1.5707963267948966
- added joint left_end_effector_mount_joint: type fixed, parent left_link7, child left_gripper_base_link, origin xyz=-0.083 0 0 rpy=-1.5707963267948966 0 3.141592653589793
- added joint right_camera_mount_joint: type fixed, parent right_link7, child right_camera_mount_link, origin xyz=0.03 0 0 rpy=1.5707963267948966 0 -1.5707963267948966
- added joint right_end_effector_mount_joint: type fixed, parent right_link7, child right_gripper_base_link, origin xyz=-0.083 0 0 rpy=1.5707963267948966 0 3.141592653589793
- joint left_camera_joint: origin xyz=-0.072196 0.054731 0 rpy=-0.27 -1.5707963267948966 0 -> xyz=0.0095 -0.02 0 rpy=-1.5707963267948966 0 -1.5707963267948966
- joint left_joint: origin xyz=0 0 0 rpy=0 0 0 -> xyz=-0.0526 0.02 0.101982 rpy=3.141592653589793 -1.308996939 3.141592653589793; parent left_link7 -> left_camera_mount_link
- joint right_camera_joint: origin xyz=-0.072196 -0.054731 0 rpy=-0.27 -1.5707963267948966 0 -> xyz=0.0095 0.02 0 rpy=-1.5707963267948966 0 -1.5707963267948966
- joint right_joint: origin xyz=0 0 0 rpy=0 0 0 -> xyz=0.0526 0.02 0.101982 rpy=3.141592653589793 -1.308996939 0.0; parent right_link7 -> right_camera_mount_link

File: galbot_charlie_description/urdf/galbot_charlie_galbot_gripper.urdf (robot description, URDF)
Before this commit: robot galbot_charlie, 66 links, 65 joints
Links:
- removed link left_arm_end_effector_mount_link
- removed link right_arm_end_effector_mount_link
- added link left_camera_mount_link
- added link right_camera_mount_link
- link left_flange_link: geometry visual mesh filename=package://galbot_one_description/meshes/flange/camera_suppo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 scale=1 1 1
- link right_flange_link: geometry visual mesh filename=package://galbot_one_description/meshes/flange/camera_suppo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 scale=1 -1 1
- link wheel_1: geometry visual mesh filename=file:///home/king/ros2_ws/install/component_models/share/co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
- link wheel_2: geometry visual mesh filename=file:///home/king/ros2_ws/install/component_models/share/co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
- link wheel_3: geometry visual mesh filename=file:///home/king/ros2_ws/install/component_models/share/co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
- link wheel_4: geometry visual mesh filename=file:///home/king/ros2_ws/install/component_models/share/co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
Joints:
- removed joint left_arm_end_effector_mount_joint
- removed joint left_gripper_mount_joint
- removed joint right_arm_end_effector_mount_joint
- removed joint right_gripper_mount_joint
- added joint left_camera_mount_joint: type fixed, parent left_link7, child left_camera_mount_link, origin xyz=0.03 0 0 rpy=1.5707963267948966 0 -1.5707963267948966
- added joint left_end_effector_mount_joint: type fixed, parent left_link7, child left_gripper_flange, origin xyz=-0.088 0 0 rpy=0 0 3.141592653589793
- added joint right_camera_mount_joint: type fixed, parent right_link7, child right_camera_mount_link, origin xyz=0.03 0 0 rpy=1.5707963267948966 0 -1.5707963267948966
- added joint right_end_effector_mount_joint: type fixed, parent right_link7, child right_gripper_flange, origin xyz=-0.088 0 0 rpy=0 0 3.141592653589793
- joint left_camera_joint: origin xyz=-0.072196 0.054731 0 rpy=-0.27 -1.5707963267948966 0 -> xyz=0.0095 -0.02 0 rpy=-1.5707963267948966 0 -1.5707963267948966
- joint left_joint: origin xyz=0 0 0 rpy=0 0 0 -> xyz=-0.0526 0.02 0.101982 rpy=3.141592653589793 -1.308996939 3.141592653589793; parent left_link7 -> left_camera_mount_link
- joint right_camera_joint: origin xyz=-0.072196 -0.054731 0 rpy=-0.27 -1.5707963267948966 0 -> xyz=0.0095 0.02 0 rpy=-1.5707963267948966 0 -1.5707963267948966
- joint right_joint: origin xyz=0 0 0 rpy=0 0 0 -> xyz=0.0526 0.02 0.101982 rpy=3.141592653589793 -1.308996939 0.0; parent right_link7 -> right_camera_mount_link

File: galbot_charlie_description/xacro/component.xacro (robot description, xacro)
@@ -6,4 +6,5 @@
   <xacro:arg name="collider" default="simple"/>
   <xacro:arg name="enable_joint5" default="true"/>
+  <xacro:arg name="arm_camera" default="d415"/>
   <xacro:if value="${'$(arg type)' == 'base'}">
     <xacro:include filename="$(find galbot_one_description)/xacro/components/chassis.xacro"/>
@@ -40,21 +41,6 @@
     </joint>
     <xacro:include filename="$(find galbot_charlie_description)/xacro/components/arm.xacro"/>
-    <xacro:include filename="$(find galbot_one_description)/xacro/components/camera.xacro"/>
-    <xacro:galbot_charlie_arm name="left" direction="1"/>
-    <xacro:galbot_charlie_arm name="right" direction="-1"/>
-    <link name="left_camera_mount_link"/>
-    <joint name="left_camera_mount_joint" type="fixed">
-      <origin xyz="0.03 0 0" rpy="0 -1.57 0"/>
-      <parent link="left_link7"/>
-      <child link="left_camera_mount_link"/>
-    </joint>
-    <link name="right_camera_mount_link"/>
-    <joint name="right_camera_mount_joint" type="fixed">
-      <origin xyz="0 0 0" rpy="0 -1.57 0"/>
-      <parent link="right_link7"/>
-      <child link="right_camera_mount_link"/>
-    </joint>
-    <xacro:GalbotOneArmCamera name="left" direction="1" parent="left_link7" flange_parent="left_camera_mount_link"/>
-    <xacro:GalbotOneArmCamera name="right" direction="-1" parent="right_link7" flange_parent="right_camera_mount_link"/>
+    <xacro:Arm name="left" direction="1" camera="$(arg arm_camera)"/>
+    <xacro:Arm name="right" direction="-1" camera="$(arg arm_camera)"/>
   </xacro:if>
 </robot>

File: galbot_charlie_description/xacro/components/arm.xacro (robot description, xacro)
@@ -2,6 +2,7 @@
 <robot xmlns:xacro="http://www.ros.org/wiki/xacro">
 	<xacro:property name="PI" value="3.141592653589793"/>
+	<xacro:include filename="$(find galbot_one_description)/xacro/components/camera.xacro"/>
 	<!-- one-style macro: name + direction + prefix -->
-	<xacro:macro name="galbot_charlie_arm" params="name direction:=1">
+	<xacro:macro name="Arm" params="name direction:=1 camera:=d415">
 		<xacro:property name="prefix" value="${name}_"/>
 		<link name="${prefix}base_link">
@@ -199,4 +200,12 @@
 			<limit effort="10" lower="-1.4" upper="1.4" velocity="1.5"/>
 		</joint>
+		<link name="${prefix}camera_mount_link"/>
+		<joint name="${prefix}camera_mount_joint" type="fixed">
+			<!-- Combined from the previous align + mount joints. -->
+			<origin xyz="0.03 0 0" rpy="${PI/2} 0 ${-PI/2}"/>
+			<parent link="${prefix}link7"/>
+			<child link="${prefix}camera_mount_link"/>
+		</joint>
+		<xacro:ArmCamera name="${name}" direction="${direction}" parent="${prefix}link7" flange_parent="${prefix}camera_mount_link" camera="${camera}"/>
 	</xacro:macro>
 </robot>

File: galbot_charlie_description/xacro/robot.xacro (robot description, xacro)
@@ -2,5 +2,5 @@
 <robot name="galbot_charlie" xmlns:xacro="http://www.ros.org/wiki/xacro">
   <xacro:arg name="enable_wheel_joints" default="false"/>
-  <xacro:arg name="arm_camera" default="d405"/>
+  <xacro:arg name="arm_camera" default="d415"/>
   <xacro:arg name="enable_joint5" default="true"/>
   <xacro:arg name="collider" default="simple"/>
@@ -33,22 +33,7 @@
   <xacro:include filename="$(find galbot_one_description)/xacro/components/body.xacro"/>
   <xacro:include filename="$(find galbot_charlie_description)/xacro/components/arm.xacro"/>
-  <xacro:include filename="$(find galbot_one_description)/xacro/components/camera.xacro"/>
   <xacro:GalbotOneChassis enable_wheel_joints="$(arg enable_wheel_joints)"/>
-  <xacro:galbot_charlie_arm name="left" direction="1"/>
-  <xacro:galbot_charlie_arm name="right" direction="-1"/>
-  <link name="left_camera_mount_link"/>
-  <joint name="left_camera_mount_joint" type="fixed">
-    <origin xyz="0.03 0 0" rpy="0 -1.57 0"/>
-    <parent link="left_link7"/>
-    <child link="left_camera_mount_link"/>
-  </joint>
-  <link name="right_camera_mount_link"/>
-  <joint name="right_camera_mount_joint" type="fixed">
-    <origin xyz="0 0 0" rpy="0 -1.57 0"/>
-    <parent link="right_link7"/>
-    <child link="right_camera_mount_link"/>
-  </joint>
-  <xacro:GalbotOneArmCamera name="left" direction="1" parent="left_link7" flange_parent="left_camera_mount_link"/>
-  <xacro:GalbotOneArmCamera name="right" direction="-1" parent="right_link7" flange_parent="right_camera_mount_link"/>
+  <xacro:Arm name="left" direction="1" camera="$(arg arm_camera)"/>
+  <xacro:Arm name="right" direction="-1" camera="$(arg arm_camera)"/>
   <joint name="left_arm_mount_joint" type="fixed">
     <origin rpy="0 ${PI} 0" xyz="0 0 -0.13"/>
@@ -63,9 +48,9 @@
   <xacro:if value="${selected_gripper_type == 'hitbot'}">
     <xacro:include filename="$(find galbot_one_description)/xacro/components/galbot_hitbot_gripper.xacro"/>
-    <xacro:hitbot_gripper name="right_gripper" parent="right_arm_end_effector_mount_link">
-      <origin xyz="0.083 0 0" rpy="0 0 0"/>
+    <xacro:hitbot_gripper name="right_gripper" parent="right_link7" mount_joint_name="right_end_effector_mount_joint">
+      <origin xyz="-0.083 0 0" rpy="${PI/2} 0 ${PI}"/>
     </xacro:hitbot_gripper>
-    <xacro:hitbot_gripper name="left_gripper" parent="left_arm_end_effector_mount_link">
-      <origin xyz="0.083 0 0" rpy="0 0 0"/>
+    <xacro:hitbot_gripper name="left_gripper" parent="left_link7" mount_joint_name="left_end_effector_mount_joint">
+      <origin xyz="-0.083 0 0" rpy="${-PI/2} 0 ${PI}"/>
     </xacro:hitbot_gripper>
   </xacro:if>
@@ -74,12 +59,12 @@
     <xacro:Gripper name="right"/>
     <xacro:Gripper name="left"/>
-    <joint name="left_gripper_mount_joint" type="fixed">
-      <origin xyz="0.088 0 0" rpy="1.57 0  0 "/>
-      <parent link="left_arm_end_effector_mount_link"/>
+    <joint name="left_end_effector_mount_joint" type="fixed">
+      <origin xyz="-0.088 0 0" rpy="0 0 ${PI}"/>
+      <parent link="left_link7"/>
       <child link="left_gripper_flange"/>
     </joint>
-    <joint name="right_gripper_mount_joint" type="fixed">
-      <origin xyz="0.088 0 0" rpy="-1.57 0  0 "/>
-      <parent link="right_arm_end_effector_mount_link"/>
+    <joint name="right_end_effector_mount_joint" type="fixed">
+      <origin xyz="-0.088 0 0" rpy="0 0 ${PI}"/>
+      <parent link="right_link7"/>
       <child link="right_gripper_flange"/>
     </joint>

File: galbot_one_description/urdf/galbot_one.urdf (robot description, URDF)
Before this commit: robot galbot_one, 67 links, 66 joints
Links:
- removed link left_camera_flange_link
- removed link left_end_effector_mount_link
- removed link left_flange_base_link
- removed link left_flange_mount_link
- removed link right_camera_flange_link
- removed link right_end_effector_mount_link
- removed link right_flange_base_link
- removed link right_flange_mount_link
- added link chassis_lidar_frame
- added link left_flange_link, mass 0.25733; visual mesh filename=package://galbot_one_description/meshes/flange/camera_suppo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 scale=1 1 1
- added link right_flange_link, mass 0.25733; visual mesh filename=package://galbot_one_description/meshes/flange/camera_suppo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 scale=1 -1 1
- link wheel_1: geometry visual mesh filename=file:///home/king/ros2_ws/install/component_models/share/co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
- link wheel_2: geometry visual mesh filename=file:///home/king/ros2_ws/install/component_models/share/co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
- link wheel_3: geometry visual mesh filename=file:///home/king/ros2_ws/install/component_models/share/co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
- link wheel_4: geometry visual mesh filename=file:///home/king/ros2_ws/install/component_models/share/co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
Joints:
- removed joint left_camera_flange_joint
- removed joint left_end_effector_mount_joint
- removed joint left_flange_joint
- removed joint left_flange_mount_joint
- removed joint right_camera_flange_joint
- removed joint right_end_effector_mount_joint
- removed joint right_flange_joint
- removed joint right_flange_mount_joint
- added joint chassis_lidar_frame_joint: type fixed, parent chassis_lidar, child chassis_lidar_frame, origin xyz=0 0 0.012
- added joint left_joint: type fixed, parent left_link7, child left_flange_link, origin xyz=-0.0526 0.02 0.101982 rpy=3.141592653589793 -1.308996939 3.141592653589793
- added joint right_joint: type fixed, parent right_link7, child right_flange_link, origin xyz=0.0526 0.02 0.101982 rpy=3.141592653589793 -1.308996939 0.0
- joint base_footprint_joint: origin (none) -> xyz=0 0 0
- joint left_camera_joint: parent left_camera_flange_link -> left_flange_link
- joint left_gripper_mount_joint: origin xyz=0 0 0 rpy=0 -1.5708 0 -> xyz=0 0 0.084525 rpy=0 -1.5707963267948966 3.141592653589793; parent left_flange_mount_link -> left_link7
- joint right_camera_joint: origin xyz=0.0095 -0.02 0 rpy=-1.5707963267948966 0 -1.5707963267948966 -> xyz=0.0095 0.02 0 rpy=-1.5707963267948966 0 -1.5707963267948966; parent right_camera_flange_link -> right_flange_link
- joint right_gripper_mount_joint: origin xyz=0 0 0 rpy=0 -1.5708 0 -> xyz=0 0 0.084525 rpy=0 -1.5707963267948966 0; parent right_flange_mount_link -> right_link7

File: galbot_one_description/urdf/galbot_one_galbot_gripper.urdf (robot description, URDF)
Before this commit: robot galbot_one, 69 links, 68 joints
Links:
- removed link left_camera_flange_link
- removed link left_end_effector_mount_link
- removed link left_flange_base_link
- removed link left_flange_mount_link
- removed link right_camera_flange_link
- removed link right_end_effector_mount_link
- removed link right_flange_base_link
- removed link right_flange_mount_link
- added link chassis_lidar_frame
- added link left_flange_link, mass 0.25733; visual mesh filename=package://galbot_one_description/meshes/flange/camera_suppo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 scale=1 1 1
- added link right_flange_link, mass 0.25733; visual mesh filename=package://galbot_one_description/meshes/flange/camera_suppo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 scale=1 -1 1
- link left_gripper_base: geometry collision mesh filename=file:///home/king/ros2_ws/install/galbot_foxtrot_descriptio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; visual mesh filename=file:///home/king/ros2_ws/install/galbot_foxtrot_descriptio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
- link left_gripper_flange: geometry visual mesh filename=file:///home/king/ros2_ws/install/galbot_foxtrot_descriptio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
- link left_gripper_l_finger_link: geometry collision mesh filename=file:///home/king/ros2_ws/install/galbot_foxtrot_descriptio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; visual mesh filename=file:///home/king/ros2_ws/install/galbot_foxtrot_descriptio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
- link left_gripper_l_inner_knuckle_link: geometry collision mesh filename=file:///home/king/ros2_ws/install/galbot_foxtrot_descriptio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; visual mesh filename=file:///home/king/ros2_ws/install/galbot_foxtrot_descriptio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
- link left_gripper_l_knuckle_link: geometry collision mesh filename=file:///home/king/ros2_ws/install/galbot_foxtrot_descriptio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; visual mesh filename=file:///home/king/ros2_ws/install/galbot_foxtrot_descriptio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
- link left_gripper_r_finger_link: geometry collision mesh filename=file:///home/king/ros2_ws/install/galbot_foxtrot_descriptio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 scale=1 -1 1; visual mesh filename=file:///home/king/ros2_ws/install/galbot_foxtrot_descriptio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 scale=1 -1 1
- link left_gripper_r_inner_knuckle_link: geometry collision mesh filename=file:///home/king/ros2_ws/install/galbot_foxtrot_descriptio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; visual mesh filename=file:///home/king/ros2_ws/install/galbot_foxtrot_descriptio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
- link left_gripper_r_knuckle_link: geometry collision mesh filename=file:///home/king/ros2_ws/install/galbot_foxtrot_descriptio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; visual mesh filename=file:///home/king/ros2_ws/install/galbot_foxtrot_descriptio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
- link right_gripper_base: geometry collision mesh filename=file:///home/king/ros2_ws/install/galbot_foxtrot_descriptio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; visual mesh filename=file:///home/king/ros2_ws/install/galbot_foxtrot_descriptio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
- link right_gripper_flange: geometry visual mesh filename=file:///home/king/ros2_ws/install/galbot_foxtrot_descriptio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
- link right_gripper_l_finger_link: geometry collision mesh filename=file:///home/king/ros2_ws/install/galbot_foxtrot_descriptio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; visual mesh filename=file:///home/king/ros2_ws/install/galbot_foxtrot_descriptio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
- link right_gripper_l_inner_knuckle_link: geometry collision mesh filename=file:///home/king/ros2_ws/install/galbot_foxtrot_descriptio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; visual mesh filename=file:///home/king/ros2_ws/install/galbot_foxtrot_descriptio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
- link right_gripper_l_knuckle_link: geometry collision mesh filename=file:///home/king/ros2_ws/install/galbot_foxtrot_descriptio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; visual mesh filename=file:///home/king/ros2_ws/install/galbot_foxtrot_descriptio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
- link right_gripper_r_finger_link: geometry collision mesh filename=file:///home/king/ros2_ws/install/galbot_foxtrot_descriptio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 scale=1 -1 1; visual mesh filename=file:///home/king/ros2_ws/install/galbot_foxtrot_descriptio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 scale=1 -1 1
- link right_gripper_r_inner_knuckle_link: geometry collision mesh filename=file:///home/king/ros2_ws/install/galbot_foxtrot_descriptio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; visual mesh filename=file:///home/king/ros2_ws/install/galbot_foxtrot_descriptio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
- link right_gripper_r_knuckle_link: geometry collision mesh filename=file:///home/king/ros2_ws/install/galbot_foxtrot_descriptio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; visual mesh filename=file:///home/king/ros2_ws/install/galbot_foxtrot_descriptio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
- link wheel_1: geometry visual mesh filename=file:///home/king/ros2_ws/install/component_models/share/co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
- link wheel_2: geometry visual mesh filename=file:///home/king/ros2_ws/install/component_models/share/co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
- link wheel_3: geometry visual mesh filename=file:///home/king/ros2_ws/install/component_models/share/co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
- link wheel_4: geometry visual mesh filename=file:///home/king/ros2_ws/install/component_models/share/co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
Joints:
- removed joint left_camera_flange_joint
- removed joint left_flange_joint
- removed joint left_flange_mount_joint
- removed joint left_gripper_mount_joint
- removed joint right_camera_flange_joint
- removed joint right_flange_joint
- removed joint right_flange_mount_joint
- removed joint right_gripper_mount_joint
- added joint chassis_lidar_frame_joint: type fixed, parent chassis_lidar, child chassis_lidar_frame, origin xyz=0 0 0.012
- added joint left_joint: type fixed, parent left_link7, child left_flange_link, origin xyz=-0.0526 0.02 0.101982 rpy=3.141592653589793 -1.308996939 3.141592653589793
- added joint right_joint: type fixed, parent right_link7, child right_flange_link, origin xyz=0.0526 0.02 0.101982 rpy=3.141592653589793 -1.308996939 0.0
- joint base_footprint_joint: origin (none) -> xyz=0 0 0
- joint left_camera_joint: parent left_camera_flange_link -> left_flange_link
- joint left_end_effector_mount_joint: child left_end_effector_mount_link -> left_gripper_flange; origin xyz=0 0 0.0845 -> xyz=0 0 0.089525 rpy=0 -1.5707963267948966 -1.5707963267948966
- joint right_camera_joint: origin xyz=0.0095 -0.02 0 rpy=-1.5707963267948966 0 -1.5707963267948966 -> xyz=0.0095 0.02 0 rpy=-1.5707963267948966 0 -1.5707963267948966; parent right_camera_flange_link -> right_flange_link
- joint right_end_effector_mount_joint: child right_end_effector_mount_link -> right_gripper_flange; origin xyz=0 0 0.0845 -> xyz=0 0 0.089525 rpy=0 -1.5707963267948966 1.5707963267948966

File: galbot_one_description/xacro/component.xacro (robot description, xacro)
@@ -5,4 +5,5 @@
   <xacro:arg name="enable_wheel_joints" default="true"/>
   <xacro:arg name="collider" default="simple"/>
+  <xacro:arg name="arm_camera" default="d415"/>
   <xacro:if value="${'$(arg type)' == 'base'}">
     <xacro:include filename="$(find galbot_one_description)/xacro/components/chassis.xacro"/>
@@ -48,9 +49,6 @@
     </joint>
     <xacro:include filename="$(find galbot_one_description)/xacro/components/arm.xacro"/>
-    <xacro:include filename="$(find galbot_one_description)/xacro/components/camera.xacro"/>
-    <xacro:galbot_one_arm name="left" direction="1"/>
-    <xacro:galbot_one_arm name="right" direction="-1"/>
-    <xacro:GalbotOneArmCamera name="left" direction="1" parent="left_link7" collider_type="$(arg collider)"/>
-    <xacro:GalbotOneArmCamera name="right" direction="-1" parent="right_link7" collider_type="$(arg collider)"/>
+    <xacro:Arm name="left" direction="1" camera="$(arg arm_camera)"/>
+    <xacro:Arm name="right" direction="-1" camera="$(arg arm_camera)"/>
   </xacro:if>
 </robot>

File: galbot_one_description/xacro/components/arm.xacro (robot description, xacro)
@@ -4,10 +4,6 @@
 	<!-- collider: simple (primitives) | convex (visual mesh as collision); set on entry xacro e.g. robot.xacro -->
 	<xacro:property name="collider_type" value="$(arg collider)"/>
-	<!--
-	  Parametric arm (same idea as Ai2Bot2Arm): name = link/joint prefix, direction = 1 (left) / -1 (right).
-	  Usage: <xacro:galbot_one_arm name="left" direction="1"/>
-	         <xacro:galbot_one_arm name="right" direction="-1"/>
-	-->
-	<xacro:macro name="galbot_one_arm" params="name direction:=1">
+	<xacro:include filename="$(find galbot_one_description)/xacro/components/camera.xacro"/>
+	<xacro:macro name="Arm" params="name direction:=1 camera:=d415">
 		<xacro:property name="prefix" value="${name}_"/>
 		<link name="${prefix}base_link">
@@ -276,4 +272,5 @@
 			<limit effort="10" lower="-${PI}" upper="${PI}" velocity="1.5"/>
 		</joint>
+		<xacro:ArmCamera name="${name}" direction="${direction}" parent="${prefix}link7" camera="${camera}" collider_type="${collider_type}"/>
 	</xacro:macro>
 </robot>
