Commit message: update galbot one and charlie xacro and urdf

File: galbot_one_description/xacro/components/camera.xacro (robot description, xacro)
@@ -2,20 +2,8 @@
 <robot xmlns:xacro="http://www.ros.org/wiki/xacro">
 	<xacro:property name="PI" value="3.141592653589793"/>
-	<!-- Wrist camera assembly; gripper mount is kept separate from the camera support. -->
-	<xacro:macro name="GalbotOneArmCamera" params="name direction:=1 parent camera:=d415 collider_type:=simple profile:=one flange_parent:=''">
+	<!-- Wrist camera assembly. The end-effector mount is owned by the arm macro. -->
+	<xacro:macro name="ArmCamera" params="name direction:=1 parent camera:=d415 collider_type:=simple profile:=one flange_parent:=''">
 		<xacro:property name="prefix" value="${name}_"/>
 		<xacro:property name="resolved_flange_parent" value="${flange_parent if flange_parent else parent}"/>
-		<link name="${prefix}arm_end_effector_mount_link">
-			<inertial>
-				<origin rpy="0 0 0" xyz="0 0 0"/>
-				<mass value="0"/>
-				<inertia ixx="0" ixy="0" ixz="0" iyy="0" iyz="0" izz="0"/>
-			</inertial>
-		</link>
-		<joint name="${prefix}arm_end_effector_mount_joint" type="fixed">
-			<origin rpy="${-PI/2 * direction} 0 ${PI}" xyz="0 0 0"/>
-			<parent link="${parent}"/>
-			<child link="${prefix}arm_end_effector_mount_link"/>
-		</joint>
 		<link name="${prefix}flange_link">
 			<inertial>

File: galbot_one_description/xacro/components/galbot_hitbot_gripper.xacro (robot description, xacro)
@@ -23,7 +23,7 @@
 <robot xmlns:xacro="http://ros.org/wiki/xacro" name="hitbot_gripper">
   <xacro:macro name="hitbot_gripper"
-    params="parent *origin name:=hitbot_gripper collider_type:=simple">
+    params="parent *origin name:=hitbot_gripper collider_type:=simple mount_joint_name:=''">
     <xacro:property name="M_PI" value="3.1415926535897931" />
-    <joint name="${name}_mount_joint" type="fixed">
+    <joint name="${mount_joint_name if mount_joint_name else name + '_mount_joint'}" type="fixed">
       <xacro:insert_block name="origin" />
       <parent link="${parent}" />

File: galbot_one_description/xacro/robot.xacro (robot description, xacro)
@@ -2,4 +2,5 @@
 <robot name="galbot_one" xmlns:xacro="http://www.ros.org/wiki/xacro">
   <xacro:arg name="enable_wheel_joints" default="false"/>
+  <xacro:arg name="arm_camera" default="d415"/>
   <xacro:property name="PI" value="3.141592653589793"/>
   <!-- type options:
@@ -32,9 +33,6 @@
   <xacro:include filename="$(find galbot_one_description)/xacro/components/body.xacro"/>
   <xacro:include filename="$(find galbot_one_description)/xacro/components/arm.xacro"/>
-  <xacro:include filename="$(find galbot_one_description)/xacro/components/camera.xacro"/>
-  <xacro:galbot_one_arm name="left" direction="1"/>
-  <xacro:galbot_one_arm name="right" direction="-1"/>
-  <xacro:GalbotOneArmCamera name="left" direction="1" parent="left_link7" collider_type="$(arg collider)"/>
-  <xacro:GalbotOneArmCamera name="right" direction="-1" parent="right_link7" collider_type="$(arg collider)"/>
+  <xacro:Arm name="left" direction="1" camera="$(arg arm_camera)"/>
+  <xacro:Arm name="right" direction="-1" camera="$(arg arm_camera)"/>
   <xacro:GalbotOneChassis enable_wheel_joints="$(arg enable_wheel_joints)"/>
   <joint name="left_arm_mount_joint" type="fixed">
@@ -50,9 +48,9 @@
   <xacro:if value="${selected_gripper_type == 'hitbot'}">
     <xacro:include filename="$(find galbot_one_description)/xacro/components/galbot_hitbot_gripper.xacro"/>
-    <xacro:hitbot_gripper name="right_gripper" parent="right_arm_end_effector_mount_link">
-      <origin xyz="0 0.084525 0" rpy="${PI/2} 0 ${PI/2}"/>
+    <xacro:hitbot_gripper name="right_gripper" parent="right_link7">
+      <origin xyz="0 0 0.084525" rpy="0 ${-PI/2} 0"/>
     </xacro:hitbot_gripper>
-    <xacro:hitbot_gripper name="left_gripper" parent="left_arm_end_effector_mount_link">
-      <origin xyz="0 -0.084525 0" rpy="${PI/2} 0 -${PI/2}"/>
+    <xacro:hitbot_gripper name="left_gripper" parent="left_link7">
+      <origin xyz="0 0 0.084525" rpy="0 ${-PI/2} ${PI}"/>
     </xacro:hitbot_gripper>
   </xacro:if>
@@ -61,12 +59,12 @@
     <xacro:Gripper name="right"/>
     <xacro:Gripper name="left"/>
-    <joint name="left_gripper_mount_joint" type="fixed">
-      <origin xyz="0 -0.089525 0" rpy="${-PI} 0 -${PI/2}"/>
-      <parent link="left_arm_end_effector_mount_link"/>
+    <joint name="left_end_effector_mount_joint" type="fixed">
+      <origin xyz="0 0 0.089525" rpy="0 ${-PI/2} ${-PI/2}"/>
+      <parent link="left_link7"/>
       <child link="left_gripper_flange"/>
     </joint>
-    <joint name="right_gripper_mount_joint" type="fixed">
-      <origin xyz="0 0.089525 0" rpy="${-PI} 0 ${PI/2}"/>
-      <parent link="right_arm_end_effector_mount_link"/>
+    <joint name="right_end_effector_mount_joint" type="fixed">
+      <origin xyz="0 0 0.089525" rpy="0 ${-PI/2} ${PI/2}"/>
+      <parent link="right_link7"/>
       <child link="right_gripper_flange"/>
     </joint>
