Commit message: 更新galbot机器人对hitbot夹爪的include路径

File: galbot_charlie_description/urdf/galbot_charlie.urdf (robot description, URDF)
Before this commit: robot galbot_charlie, 64 links, 63 joints
Links:
- removed link left_gripper_base_link
- removed link right_gripper_base_link
- added link left_gripper_base, mass 0.878; collision mesh filename=package://hitbot_description/meshes/Z-EFG-100/convex/base_l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; visual mesh filename=package://hitbot_description/meshes/Z-EFG-100/visual/base.g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
- added link right_gripper_base, mass 0.878; collision mesh filename=package://hitbot_description/meshes/Z-EFG-100/convex/base_l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; visual mesh filename=package://hitbot_description/meshes/Z-EFG-100/visual/base.g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
- link left_gripper_link1: geometry collision mesh filename=package://hitbot_description/meshes/Z-EFG-100/convex/grippe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; visual mesh filename=package://hitbot_description/meshes/Z-EFG-100/visual/link1.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
- link left_gripper_link2: geometry collision mesh filename=package://hitbot_description/meshes/Z-EFG-100/convex/grippe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; visual mesh filename=package://hitbot_description/meshes/Z-EFG-100/visual/link2.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
- link left_gripper_link3: geometry collision mesh filename=package://hitbot_description/meshes/Z-EFG-100/convex/grippe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; visual mesh filename=package://hitbot_description/meshes/Z-EFG-100/visual/link3.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
- link left_gripper_link4: geometry collision mesh filename=package://hitbot_description/meshes/Z-EFG-100/convex/grippe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; visual mesh filename=package://hitbot_description/meshes/Z-EFG-100/visual/link4.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
- link left_gripper_link5: geometry collision mesh filename=package://hitbot_description/meshes/Z-EFG-100/convex/grippe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; visual mesh filename=package://hitbot_description/meshes/Z-EFG-100/visual/link5.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
- link left_gripper_link6: geometry collision mesh filename=package://hitbot_description/meshes/Z-EFG-100/convex/grippe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; visual mesh filename=package://hitbot_description/meshes/Z-EFG-100/visual/link6.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
- link right_gripper_link1: geometry collision mesh filename=package://hitbot_description/meshes/Z-EFG-100/convex/grippe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; visual mesh filename=package://hitbot_description/meshes/Z-EFG-100/visual/link1.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
- link right_gripper_link2: geometry collision mesh filename=package://hitbot_description/meshes/Z-EFG-100/convex/grippe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; visual mesh filename=package://hitbot_description/meshes/Z-EFG-100/visual/link2.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
- link right_gripper_link3: geometry collision mesh filename=package://hitbot_description/meshes/Z-EFG-100/convex/grippe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; visual mesh filename=package://hitbot_description/meshes/Z-EFG-100/visual/link3.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
- link right_gripper_link4: geometry collision mesh filename=package://hitbot_description/meshes/Z-EFG-100/convex/grippe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; visual mesh filename=package://hitbot_description/meshes/Z-EFG-100/visual/link4.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
- link right_gripper_link5: geometry collision mesh filename=package://hitbot_description/meshes/Z-EFG-100/convex/grippe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; visual mesh filename=package://hitbot_description/meshes/Z-EFG-100/visual/link5.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
- link right_gripper_link6: geometry collision mesh filename=package://hitbot_description/meshes/Z-EFG-100/convex/grippe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; visual mesh filename=package://hitbot_description/meshes/Z-EFG-100/visual/link6.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
- link wheel_1: geometry visual mesh filename=package://component_models/meshes/omniwheel_10.glb
- link wheel_2: geometry visual mesh filename=package://component_models/meshes/omniwheel_10.glb
- link wheel_3: geometry visual mesh filename=package://component_models/meshes/omniwheel_10.glb
- link wheel_4: geometry visual mesh filename=package://component_models/meshes/omniwheel_10.glb
Joints:
- joint left_end_effector_mount_joint: child left_gripper_base_link -> left_gripper_base
- joint left_gripper_joint: parent left_gripper_base_link -> left_gripper_base
- joint left_gripper_joint2: parent left_gripper_base_link -> left_gripper_base
- joint left_gripper_joint4: parent left_gripper_base_link -> left_gripper_base
- joint left_gripper_joint5: parent left_gripper_base_link -> left_gripper_base
- joint left_gripper_tcp_joint: parent left_gripper_base_link -> left_gripper_base
- joint right_end_effector_mount_joint: child right_gripper_base_link -> right_gripper_base
- joint right_gripper_joint: parent right_gripper_base_link -> right_gripper_base
- joint right_gripper_joint2: parent right_gripper_base_link -> right_gripper_base
- joint right_gripper_joint4: parent right_gripper_base_link -> right_gripper_base
- joint right_gripper_joint5: parent right_gripper_base_link -> right_gripper_base
- joint right_gripper_tcp_joint: parent right_gripper_base_link -> right_gripper_base

File: galbot_charlie_description/xacro/robot.xacro (robot description, xacro)
@@ -47,11 +47,17 @@
   </joint>
   <xacro:if value="${selected_gripper_type == 'hitbot'}">
-    <xacro:include filename="$(find galbot_one_description)/xacro/components/galbot_hitbot_gripper.xacro"/>
-    <xacro:hitbot_gripper name="right_gripper" parent="right_link7" mount_joint_name="right_end_effector_mount_joint">
+    <xacro:include filename="$(find hitbot_description)/xacro/Z-EFG-100.xacro"/>
+    <joint name="right_end_effector_mount_joint" type="fixed">
       <origin xyz="-0.083 0 0" rpy="${PI/2} 0 ${PI}"/>
-    </xacro:hitbot_gripper>
-    <xacro:hitbot_gripper name="left_gripper" parent="left_link7" mount_joint_name="left_end_effector_mount_joint">
+      <parent link="right_link7"/>
+      <child link="right_gripper_base"/>
+    </joint>
+    <xacro:Gripper name="right_gripper" collider_type="$(arg collider)"/>
+    <joint name="left_end_effector_mount_joint" type="fixed">
       <origin xyz="-0.083 0 0" rpy="${-PI/2} 0 ${PI}"/>
-    </xacro:hitbot_gripper>
+      <parent link="left_link7"/>
+      <child link="left_gripper_base"/>
+    </joint>
+    <xacro:Gripper name="left_gripper" collider_type="$(arg collider)"/>
   </xacro:if>
   <xacro:if value="${selected_gripper_type == 'galbot_gripper'}">

File: galbot_foxtrot_description/urdf/galbot_foxtrot_hitbot.urdf (robot description, URDF)
Before this commit: robot galbot_one_foxtrot, 58 links, 57 joints
Links:
- removed link left_gripper_base_link
- removed link right_gripper_base_link
- added link left_gripper_base, mass 0.878; collision mesh filename=package://hitbot_description/meshes/Z-EFG-100/convex/base_l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; visual mesh filename=package://hitbot_description/meshes/Z-EFG-100/visual/base.g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
- added link right_gripper_base, mass 0.878; collision mesh filename=package://hitbot_description/meshes/Z-EFG-100/convex/base_l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; visual mesh filename=package://hitbot_description/meshes/Z-EFG-100/visual/base.g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
- link left_gripper_link1: geometry collision mesh filename=package://hitbot_description/meshes/Z-EFG-100/convex/grippe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; visual mesh filename=package://hitbot_description/meshes/Z-EFG-100/visual/link1.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
- link left_gripper_link2: geometry collision mesh filename=package://hitbot_description/meshes/Z-EFG-100/convex/grippe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; visual mesh filename=package://hitbot_description/meshes/Z-EFG-100/visual/link2.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
- link left_gripper_link3: geometry collision mesh filename=package://hitbot_description/meshes/Z-EFG-100/convex/grippe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; visual mesh filename=package://hitbot_description/meshes/Z-EFG-100/visual/link3.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
- link left_gripper_link4: geometry collision mesh filename=package://hitbot_description/meshes/Z-EFG-100/convex/grippe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; visual mesh filename=package://hitbot_description/meshes/Z-EFG-100/visual/link4.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
- link left_gripper_link5: geometry collision mesh filename=package://hitbot_description/meshes/Z-EFG-100/convex/grippe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; visual mesh filename=package://hitbot_description/meshes/Z-EFG-100/visual/link5.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
- link left_gripper_link6: geometry collision mesh filename=package://hitbot_description/meshes/Z-EFG-100/convex/grippe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; visual mesh filename=package://hitbot_description/meshes/Z-EFG-100/visual/link6.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
- link right_gripper_link1: geometry collision mesh filename=package://hitbot_description/meshes/Z-EFG-100/convex/grippe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; visual mesh filename=package://hitbot_description/meshes/Z-EFG-100/visual/link1.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
- link right_gripper_link2: geometry collision mesh filename=package://hitbot_description/meshes/Z-EFG-100/convex/grippe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; visual mesh filename=package://hitbot_description/meshes/Z-EFG-100/visual/link2.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
- link right_gripper_link3: geometry collision mesh filename=package://hitbot_description/meshes/Z-EFG-100/convex/grippe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; visual mesh filename=package://hitbot_description/meshes/Z-EFG-100/visual/link3.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
- link right_gripper_link4: geometry collision mesh filename=package://hitbot_description/meshes/Z-EFG-100/convex/grippe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; visual mesh filename=package://hitbot_description/meshes/Z-EFG-100/visual/link4.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
- link right_gripper_link5: geometry collision mesh filename=package://hitbot_description/meshes/Z-EFG-100/convex/grippe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; visual mesh filename=package://hitbot_description/meshes/Z-EFG-100/visual/link5.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
- link right_gripper_link6: geometry collision mesh filename=package://hitbot_description/meshes/Z-EFG-100/convex/grippe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; visual mesh filename=package://hitbot_description/meshes/Z-EFG-100/visual/link6.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
Joints:
- removed joint left_gripper_mount_joint
- removed joint right_gripper_mount_joint
- added joint left_end_effector_mount_joint: type fixed, parent left_link7, child left_gripper_base, origin xyz=-0.10926 0 0 rpy=0 0 3.14159265358979
- added joint right_end_effector_mount_joint: type fixed, parent right_link7, child right_gripper_base, origin xyz=-0.10926 0 0 rpy=0 0 3.14159265358948
- joint left_gripper_joint: parent left_gripper_base_link -> left_gripper_base
- joint left_gripper_joint2: parent left_gripper_base_link -> left_gripper_base
- joint left_gripper_joint4: parent left_gripper_base_link -> left_gripper_base
- joint left_gripper_joint5: parent left_gripper_base_link -> left_gripper_base
- joint left_gripper_tcp_joint: parent left_gripper_base_link -> left_gripper_base
- joint right_gripper_joint: parent right_gripper_base_link -> right_gripper_base
- joint right_gripper_joint2: parent right_gripper_base_link -> right_gripper_base
- joint right_gripper_joint4: parent right_gripper_base_link -> right_gripper_base
- joint right_gripper_joint5: parent right_gripper_base_link -> right_gripper_base
- joint right_gripper_tcp_joint: parent right_gripper_base_link -> right_gripper_base

File: galbot_foxtrot_description/xacro/gripper.xacro (robot description, xacro)
@@ -15,9 +15,6 @@
   </xacro:if>
   <xacro:if value="${selected_gripper_type == 'hitbot'}">
-    <xacro:include filename="$(find galbot_one_description)/xacro/components/galbot_hitbot_gripper.xacro"/>
-    <link name="gripper_base"/>
-    <xacro:hitbot_gripper name="gripper" parent="gripper_base">
-      <origin xyz="0 0 0" rpy="0 0 0"/>
-    </xacro:hitbot_gripper>
+    <xacro:include filename="$(find hitbot_description)/xacro/Z-EFG-100.xacro"/>
+    <xacro:Gripper name=""/>
   </xacro:if>
 </robot>

File: galbot_foxtrot_description/xacro/robot.xacro (robot description, xacro)
@@ -43,8 +43,11 @@
 	</xacro:if>
 	<xacro:if value="${selected_gripper_type == 'hitbot'}">
-		<xacro:include filename="$(find galbot_one_description)/xacro/components/galbot_hitbot_gripper.xacro"/>
-		<xacro:hitbot_gripper name="right_gripper" parent="right_link7">
-			<origin rpy="0 0 3.14159265358948" xyz="-0.10926 0 0"/>
-		</xacro:hitbot_gripper>
+		<xacro:include filename="$(find hitbot_description)/xacro/Z-EFG-100.xacro"/>
+		<joint name="right_end_effector_mount_joint" type="fixed">
+			<origin xyz="-0.10926 0 0" rpy="0 0 3.14159265358948"/>
+			<parent link="right_link7"/>
+			<child link="right_gripper_base"/>
+		</joint>
+		<xacro:Gripper name="right_gripper"/>
 	</xacro:if>
 	<xacro:Arm name="left" camera="$(arg arm_camera)"/>
@@ -58,7 +61,10 @@
 	</xacro:if>
 	<xacro:if value="${selected_gripper_type == 'hitbot'}">
-		<xacro:hitbot_gripper name="left_gripper" parent="left_link7">
-			<origin rpy="0 0 3.14159265358979" xyz="-0.10926 0 0"/>
-		</xacro:hitbot_gripper>
+		<joint name="left_end_effector_mount_joint" type="fixed">
+			<origin xyz="-0.10926 0 0" rpy="0 0 3.14159265358979"/>
+			<parent link="left_link7"/>
+			<child link="left_gripper_base"/>
+		</joint>
+		<xacro:Gripper name="left_gripper"/>
 	</xacro:if>
 </robot>

File: galbot_golf_description/urdf/galbot_golf_hitbot.urdf (robot description, URDF)
Before this commit: robot galbot_one_golf, 60 links, 59 joints
Links:
- removed link left_gripper_base_link
- removed link right_gripper_base_link
- added link left_gripper_base, mass 0.878; collision mesh filename=package://hitbot_description/meshes/Z-EFG-100/convex/base_l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; visual mesh filename=package://hitbot_description/meshes/Z-EFG-100/visual/base.g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
- added link right_gripper_base, mass 0.878; collision mesh filename=package://hitbot_description/meshes/Z-EFG-100/convex/base_l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; visual mesh filename=package://hitbot_description/meshes/Z-EFG-100/visual/base.g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
- link left_gripper_link1: geometry collision mesh filename=package://hitbot_description/meshes/Z-EFG-100/convex/grippe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; visual mesh filename=package://hitbot_description/meshes/Z-EFG-100/visual/link1.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
- link left_gripper_link2: geometry collision mesh filename=package://hitbot_description/meshes/Z-EFG-100/convex/grippe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; visual mesh filename=package://hitbot_description/meshes/Z-EFG-100/visual/link2.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
- link left_gripper_link3: geometry collision mesh filename=package://hitbot_description/meshes/Z-EFG-100/convex/grippe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; visual mesh filename=package://hitbot_description/meshes/Z-EFG-100/visual/link3.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
- link left_gripper_link4: geometry collision mesh filename=package://hitbot_description/meshes/Z-EFG-100/convex/grippe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; visual mesh filename=package://hitbot_description/meshes/Z-EFG-100/visual/link4.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
- link left_gripper_link5: geometry collision mesh filename=package://hitbot_description/meshes/Z-EFG-100/convex/grippe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; visual mesh filename=package://hitbot_description/meshes/Z-EFG-100/visual/link5.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
- link left_gripper_link6: geometry collision mesh filename=package://hitbot_description/meshes/Z-EFG-100/convex/grippe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; visual mesh filename=package://hitbot_description/meshes/Z-EFG-100/visual/link6.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
- link right_gripper_link1: geometry collision mesh filename=package://hitbot_description/meshes/Z-EFG-100/convex/grippe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; visual mesh filename=package://hitbot_description/meshes/Z-EFG-100/visual/link1.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
- link right_gripper_link2: geometry collision mesh filename=package://hitbot_description/meshes/Z-EFG-100/convex/grippe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; visual mesh filename=package://hitbot_description/meshes/Z-EFG-100/visual/link2.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
- link right_gripper_link3: geometry collision mesh filename=package://hitbot_description/meshes/Z-EFG-100/convex/grippe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; visual mesh filename=package://hitbot_description/meshes/Z-EFG-100/visual/link3.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
- link right_gripper_link4: geometry collision mesh filename=package://hitbot_description/meshes/Z-EFG-100/convex/grippe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; visual mesh filename=package://hitbot_description/meshes/Z-EFG-100/visual/link4.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
- link right_gripper_link5: geometry collision mesh filename=package://hitbot_description/meshes/Z-EFG-100/convex/grippe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; visual mesh filename=package://hitbot_description/meshes/Z-EFG-100/visual/link5.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
- link right_gripper_link6: geometry collision mesh filename=package://hitbot_description/meshes/Z-EFG-100/convex/grippe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; visual mesh filename=package://hitbot_description/meshes/Z-EFG-100/visual/link6.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
Joints:
- removed joint left_gripper_mount_joint
- removed joint right_gripper_mount_joint
- added joint left_end_effector_mount_joint: type fixed, parent left_link7, child left_gripper_base, origin xyz=-0.10926 0 0 rpy=0 0 3.14159265358979
- added joint right_end_effector_mount_joint: type fixed, parent right_link7, child right_gripper_base, origin xyz=-0.10926 0 0 rpy=0 0 3.14159265358948
- joint left_gripper_joint: parent left_gripper_base_link -> left_gripper_base
- joint left_gripper_joint2: parent left_gripper_base_link -> left_gripper_base
- joint left_gripper_joint4: parent left_gripper_base_link -> left_gripper_base
- joint left_gripper_joint5: parent left_gripper_base_link -> left_gripper_base
- joint left_gripper_tcp_joint: parent left_gripper_base_link -> left_gripper_base
- joint right_gripper_joint: parent right_gripper_base_link -> right_gripper_base
- joint right_gripper_joint2: parent right_gripper_base_link -> right_gripper_base
- joint right_gripper_joint4: parent right_gripper_base_link -> right_gripper_base
- joint right_gripper_joint5: parent right_gripper_base_link -> right_gripper_base
- joint right_gripper_tcp_joint: parent right_gripper_base_link -> right_gripper_base

File: galbot_golf_description/xacro/gripper.xacro (robot description, xacro)
@@ -16,8 +16,6 @@
   </xacro:if>
   <xacro:if value="${selected_gripper_type == 'hitbot'}">
-    <xacro:include filename="$(find galbot_one_description)/xacro/components/galbot_hitbot_gripper.xacro"/>
-    <link name="gripper_base"/>
-    <xacro:hitbot_gripper name="gripper" parent="gripper_base" collider_type="$(arg collider)">
-    </xacro:hitbot_gripper>
+    <xacro:include filename="$(find hitbot_description)/xacro/Z-EFG-100.xacro"/>
+    <xacro:Gripper name="" collider_type="$(arg collider)"/>
   </xacro:if>
 </robot>

File: galbot_golf_description/xacro/robot.xacro (robot description, xacro)
@@ -53,8 +53,11 @@
 	</xacro:if>
 	<xacro:if value="${selected_gripper_type == 'hitbot'}">
-		<xacro:include filename="$(find galbot_one_description)/xacro/components/galbot_hitbot_gripper.xacro"/>
-		<xacro:hitbot_gripper name="right_gripper" parent="right_link7" collider_type="$(arg collider)">
-			<origin rpy="0 0 3.14159265358948" xyz="-0.10926 0 0"/>
-		</xacro:hitbot_gripper>
+		<xacro:include filename="$(find hitbot_description)/xacro/Z-EFG-100.xacro"/>
+		<joint name="right_end_effector_mount_joint" type="fixed">
+			<origin xyz="-0.10926 0 0" rpy="0 0 3.14159265358948"/>
+			<parent link="right_link7"/>
+			<child link="right_gripper_base"/>
+		</joint>
+		<xacro:Gripper name="right_gripper" collider_type="$(arg collider)"/>
 	</xacro:if>
 	<joint name="left_arm_joint" type="fixed">
@@ -72,7 +75,10 @@
 	</xacro:if>
 	<xacro:if value="${selected_gripper_type == 'hitbot'}">
-		<xacro:hitbot_gripper name="left_gripper" parent="left_link7" collider_type="$(arg collider)">
-			<origin rpy="0 0 3.14159265358979" xyz="-0.10926 0 0"/>
-		</xacro:hitbot_gripper>
+		<joint name="left_end_effector_mount_joint" type="fixed">
+			<origin xyz="-0.10926 0 0" rpy="0 0 3.14159265358979"/>
+			<parent link="left_link7"/>
+			<child link="left_gripper_base"/>
+		</joint>
+		<xacro:Gripper name="left_gripper" collider_type="$(arg collider)"/>
 	</xacro:if>
 </robot>
