Commit message: 更新galbot机器人对hitbot夹爪的include路径

File: galbot_one_description/urdf/galbot_one.urdf (robot description, URDF)
Before this commit: robot galbot_one, 62 links, 61 joints
Links:
- removed link left_gripper_base_link
- removed link right_gripper_base_link
- added link left_gripper_base, mass 0.878; collision mesh filename=package://hitbot_description/meshes/Z-EFG-100/convex/base_l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; visual mesh filename=package://hitbot_description/meshes/Z-EFG-100/visual/base.g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
- added link right_gripper_base, mass 0.878; collision mesh filename=package://hitbot_description/meshes/Z-EFG-100/convex/base_l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; visual mesh filename=package://hitbot_description/meshes/Z-EFG-100/visual/base.g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
- link left_gripper_link1: geometry collision mesh filename=package://hitbot_description/meshes/Z-EFG-100/convex/grippe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; visual mesh filename=package://hitbot_description/meshes/Z-EFG-100/visual/link1.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
- link left_gripper_link2: geometry collision mesh filename=package://hitbot_description/meshes/Z-EFG-100/convex/grippe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; visual mesh filename=package://hitbot_description/meshes/Z-EFG-100/visual/link2.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
- link left_gripper_link3: geometry collision mesh filename=package://hitbot_description/meshes/Z-EFG-100/convex/grippe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; visual mesh filename=package://hitbot_description/meshes/Z-EFG-100/visual/link3.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
- link left_gripper_link4: geometry collision mesh filename=package://hitbot_description/meshes/Z-EFG-100/convex/grippe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; visual mesh filename=package://hitbot_description/meshes/Z-EFG-100/visual/link4.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
- link left_gripper_link5: geometry collision mesh filename=package://hitbot_description/meshes/Z-EFG-100/convex/grippe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; visual mesh filename=package://hitbot_description/meshes/Z-EFG-100/visual/link5.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
- link left_gripper_link6: geometry collision mesh filename=package://hitbot_description/meshes/Z-EFG-100/convex/grippe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; visual mesh filename=package://hitbot_description/meshes/Z-EFG-100/visual/link6.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
- link right_gripper_link1: geometry collision mesh filename=package://hitbot_description/meshes/Z-EFG-100/convex/grippe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; visual mesh filename=package://hitbot_description/meshes/Z-EFG-100/visual/link1.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
- link right_gripper_link2: geometry collision mesh filename=package://hitbot_description/meshes/Z-EFG-100/convex/grippe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; visual mesh filename=package://hitbot_description/meshes/Z-EFG-100/visual/link2.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
- link right_gripper_link3: geometry collision mesh filename=package://hitbot_description/meshes/Z-EFG-100/convex/grippe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; visual mesh filename=package://hitbot_description/meshes/Z-EFG-100/visual/link3.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
- link right_gripper_link4: geometry collision mesh filename=package://hitbot_description/meshes/Z-EFG-100/convex/grippe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; visual mesh filename=package://hitbot_description/meshes/Z-EFG-100/visual/link4.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
- link right_gripper_link5: geometry collision mesh filename=package://hitbot_description/meshes/Z-EFG-100/convex/grippe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; visual mesh filename=package://hitbot_description/meshes/Z-EFG-100/visual/link5.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
- link right_gripper_link6: geometry collision mesh filename=package://hitbot_description/meshes/Z-EFG-100/convex/grippe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; visual mesh filename=package://hitbot_description/meshes/Z-EFG-100/visual/link6.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
- link wheel_1: geometry visual mesh filename=package://component_models/meshes/omniwheel_10.glb
- link wheel_2: geometry visual mesh filename=package://component_models/meshes/omniwheel_10.glb
- link wheel_3: geometry visual mesh filename=package://component_models/meshes/omniwheel_10.glb
- link wheel_4: geometry visual mesh filename=package://component_models/meshes/omniwheel_10.glb
Joints:
- removed joint left_gripper_mount_joint
- removed joint right_gripper_mount_joint
- added joint left_end_effector_mount_joint: type fixed, parent left_link7, child left_gripper_base, origin xyz=0 0 0.084525 rpy=0 -1.5707963267948966 3.141592653589793
- added joint right_end_effector_mount_joint: type fixed, parent right_link7, child right_gripper_base, origin xyz=0 0 0.084525 rpy=0 -1.5707963267948966 0
- joint left_gripper_joint: parent left_gripper_base_link -> left_gripper_base
- joint left_gripper_joint2: parent left_gripper_base_link -> left_gripper_base
- joint left_gripper_joint4: parent left_gripper_base_link -> left_gripper_base
- joint left_gripper_joint5: parent left_gripper_base_link -> left_gripper_base
- joint left_gripper_tcp_joint: parent left_gripper_base_link -> left_gripper_base
- joint right_gripper_joint: parent right_gripper_base_link -> right_gripper_base
- joint right_gripper_joint2: parent right_gripper_base_link -> right_gripper_base
- joint right_gripper_joint4: parent right_gripper_base_link -> right_gripper_base
- joint right_gripper_joint5: parent right_gripper_base_link -> right_gripper_base
- joint right_gripper_tcp_joint: parent right_gripper_base_link -> right_gripper_base

File: galbot_one_description/xacro/gripper.xacro (robot description, xacro)
@@ -12,9 +12,6 @@
   </xacro:if>
   <xacro:if value="${selected_gripper_type == 'hitbot'}">
-    <xacro:include filename="$(find galbot_one_description)/xacro/components/galbot_hitbot_gripper.xacro"/>
-    <link name="gripper_base"/>
-    <xacro:hitbot_gripper name="gripper" parent="gripper_base" collider_type="$(arg collider)">
-      <origin xyz="0 0 0" rpy="0 0 0"/>
-    </xacro:hitbot_gripper>
+    <xacro:include filename="$(find hitbot_description)/xacro/Z-EFG-100.xacro"/>
+    <xacro:Gripper name="" collider_type="$(arg collider)"/>
   </xacro:if>
   <xacro:if value="${selected_gripper_type == 'galbot_gripper'}">

File: galbot_one_description/xacro/robot.xacro (robot description, xacro)
@@ -47,11 +47,17 @@
   </joint>
   <xacro:if value="${selected_gripper_type == 'hitbot'}">
-    <xacro:include filename="$(find galbot_one_description)/xacro/components/galbot_hitbot_gripper.xacro"/>
-    <xacro:hitbot_gripper name="right_gripper" parent="right_link7">
+    <xacro:include filename="$(find hitbot_description)/xacro/Z-EFG-100.xacro"/>
+    <joint name="right_end_effector_mount_joint" type="fixed">
       <origin xyz="0 0 0.084525" rpy="0 ${-PI/2} 0"/>
-    </xacro:hitbot_gripper>
-    <xacro:hitbot_gripper name="left_gripper" parent="left_link7">
+      <parent link="right_link7"/>
+      <child link="right_gripper_base"/>
+    </joint>
+    <xacro:Gripper name="right_gripper" collider_type="$(arg collider)"/>
+    <joint name="left_end_effector_mount_joint" type="fixed">
       <origin xyz="0 0 0.084525" rpy="0 ${-PI/2} ${PI}"/>
-    </xacro:hitbot_gripper>
+      <parent link="left_link7"/>
+      <child link="left_gripper_base"/>
+    </joint>
+    <xacro:Gripper name="left_gripper" collider_type="$(arg collider)"/>
   </xacro:if>
   <xacro:if value="${selected_gripper_type == 'galbot_gripper'}">
