Commit message: 加galbot整体readme,加charlie碰撞体，规范写法

File: galbot_charlie_description/urdf/galbot_charlie.urdf (robot description, URDF)
Before this commit: robot galbot_charlie, 64 links, 63 joints
Links:
- link left_gripper_base: geometry collision mesh filename=package://hitbot_description/meshes/Z-EFG-100/collision/bas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; visual mesh filename=package://hitbot_description/meshes/Z-EFG-100/visual/base.g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
- link left_gripper_link1: geometry collision mesh filename=package://hitbot_description/meshes/Z-EFG-100/collision/gri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; visual mesh filename=package://hitbot_description/meshes/Z-EFG-100/visual/link1.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
- link left_gripper_link2: geometry collision mesh filename=package://hitbot_description/meshes/Z-EFG-100/collision/gri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; visual mesh filename=package://hitbot_description/meshes/Z-EFG-100/visual/link2.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
- link left_gripper_link3: geometry collision mesh filename=package://hitbot_description/meshes/Z-EFG-100/collision/gri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; visual mesh filename=package://hitbot_description/meshes/Z-EFG-100/visual/link3.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
- link left_gripper_link4: geometry collision mesh filename=package://hitbot_description/meshes/Z-EFG-100/collision/gri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; visual mesh filename=package://hitbot_description/meshes/Z-EFG-100/visual/link4.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
- link left_gripper_link5: geometry collision mesh filename=package://hitbot_description/meshes/Z-EFG-100/collision/gri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; visual mesh filename=package://hitbot_description/meshes/Z-EFG-100/visual/link5.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
- link left_gripper_link6: geometry collision mesh filename=package://hitbot_description/meshes/Z-EFG-100/collision/gri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; visual mesh filename=package://hitbot_description/meshes/Z-EFG-100/visual/link6.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
- link left_link4: geometry collision cylinder length=0.10085 radius=0.044983; visual mesh filename=package://galbot_one_description/meshes/arm/link4.glb
- link left_link5: geometry collision box size=0.07466 0.093966 0.16955; visual mesh filename=package://galbot_charlie_description/meshs/arm/link5.glb
- link left_link6: geometry collision sphere radius=0.05987; visual mesh filename=package://galbot_charlie_description/meshs/arm/link6.glb
- link left_link7: geometry collision cylinder length=0.16 radius=0.007; visual mesh filename=package://galbot_charlie_description/meshs/arm/link7.glb
- link right_gripper_base: geometry collision mesh filename=package://hitbot_description/meshes/Z-EFG-100/collision/bas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; visual mesh filename=package://hitbot_description/meshes/Z-EFG-100/visual/base.g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
- link right_gripper_link1: geometry collision mesh filename=package://hitbot_description/meshes/Z-EFG-100/collision/gri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; visual mesh filename=package://hitbot_description/meshes/Z-EFG-100/visual/link1.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
- link right_gripper_link2: geometry collision mesh filename=package://hitbot_description/meshes/Z-EFG-100/collision/gri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; visual mesh filename=package://hitbot_description/meshes/Z-EFG-100/visual/link2.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
- link right_gripper_link3: geometry collision mesh filename=package://hitbot_description/meshes/Z-EFG-100/collision/gri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; visual mesh filename=package://hitbot_description/meshes/Z-EFG-100/visual/link3.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
- link right_gripper_link4: geometry collision mesh filename=package://hitbot_description/meshes/Z-EFG-100/collision/gri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; visual mesh filename=package://hitbot_description/meshes/Z-EFG-100/visual/link4.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
- link right_gripper_link5: geometry collision mesh filename=package://hitbot_description/meshes/Z-EFG-100/collision/gri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; visual mesh filename=package://hitbot_description/meshes/Z-EFG-100/visual/link5.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
- link right_gripper_link6: geometry collision mesh filename=package://hitbot_description/meshes/Z-EFG-100/collision/gri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; visual mesh filename=package://hitbot_description/meshes/Z-EFG-100/visual/link6.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
- link right_link4: geometry collision cylinder length=0.10085 radius=0.044983; visual mesh filename=package://galbot_one_description/meshes/arm/link4.glb
- link right_link5: geometry collision box size=0.07466 0.093966 0.16955; visual mesh filename=package://galbot_charlie_description/meshs/arm/link5.glb
- link right_link6: geometry collision sphere radius=0.05987; visual mesh filename=package://galbot_charlie_description/meshs/arm/link6.glb
- link right_link7: geometry collision cylinder length=0.16 radius=0.007; visual mesh filename=package://galbot_charlie_description/meshs/arm/link7.glb

File: galbot_charlie_description/urdf/galbot_charlie_galbot_gripper.urdf (robot description, URDF)
Before this commit: robot galbot_charlie, 66 links, 65 joints
Links:
- link left_link4: geometry collision cylinder length=0.10085 radius=0.044983; visual mesh filename=package://galbot_one_description/meshes/arm/link4.glb
- link left_link5: geometry collision box size=0.07466 0.093966 0.16955; visual mesh filename=package://galbot_charlie_description/meshs/arm/link5.glb
- link left_link6: geometry collision sphere radius=0.05987; visual mesh filename=package://galbot_charlie_description/meshs/arm/link6.glb
- link left_link7: geometry collision cylinder length=0.16 radius=0.007; visual mesh filename=package://galbot_charlie_description/meshs/arm/link7.glb
- link right_link4: geometry collision cylinder length=0.10085 radius=0.044983; visual mesh filename=package://galbot_one_description/meshes/arm/link4.glb
- link right_link5: geometry collision box size=0.07466 0.093966 0.16955; visual mesh filename=package://galbot_charlie_description/meshs/arm/link5.glb
- link right_link6: geometry collision sphere radius=0.05987; visual mesh filename=package://galbot_charlie_description/meshs/arm/link6.glb
- link right_link7: geometry collision cylinder length=0.16 radius=0.007; visual mesh filename=package://galbot_charlie_description/meshs/arm/link7.glb
- link wheel_1: geometry visual mesh filename=package://component_models/meshes/omniwheel_10.glb
- link wheel_2: geometry visual mesh filename=package://component_models/meshes/omniwheel_10.glb
- link wheel_3: geometry visual mesh filename=package://component_models/meshes/omniwheel_10.glb
- link wheel_4: geometry visual mesh filename=package://component_models/meshes/omniwheel_10.glb

File: galbot_charlie_description/xacro/component.xacro (robot description, xacro)
@@ -1,4 +1,4 @@
 <?xml version="1.0" ?>
-<robot name="galbot_charlie_component" xmlns:xacro="http://www.ros.org/wiki/xacro">
+<robot name="Galbot Charlie Arms" xmlns:xacro="http://www.ros.org/wiki/xacro">
   <xacro:property name="PI" value="3.141592653589793"/>
   <xacro:arg name="type" default="base"/>

File: galbot_charlie_description/xacro/components/arm.xacro (robot description, xacro)
@@ -116,5 +116,5 @@
 				<origin rpy="${PI/2} 0 0" xyz="0 -0.14 0"/>
 				<geometry>
-					<cylinder length="0.16085" radius="0.044983"/>
+					<cylinder length="0.10085" radius="0.044983"/>
 				</geometry>
 			</collision>
@@ -140,6 +140,7 @@
 			</visual>
 			<collision>
-				<geometry>
-					<mesh filename="file://$(find galbot_charlie_description)/meshs/arm/link5.glb"/>
+				<origin xyz="0 0 -0.12"/>
+				<geometry>
+					<box size="0.07466 0.093966 0.16955"/>
 				</geometry>
 			</collision>
@@ -165,5 +166,5 @@
 			<collision>
 				<geometry>
-					<mesh filename="file://$(find galbot_charlie_description)/meshs/arm/link6.glb"/>
+					<sphere radius="0.05987"/>
 				</geometry>
 			</collision>
@@ -188,6 +189,7 @@
 			</visual>
 			<collision>
-				<geometry>
-					<mesh filename="file://$(find galbot_charlie_description)/meshs/arm/link7.glb"/>
+				<origin xyz="0 0 -0.015"/>
+				<geometry>
+					<cylinder length="0.16" radius="0.007"/>
 				</geometry>
 			</collision>

File: galbot_charlie_description/xacro/robot.xacro (robot description, xacro)
@@ -53,5 +53,5 @@
       <child link="right_gripper_base"/>
     </joint>
-    <xacro:Gripper name="right_gripper" collider_type="$(arg collider)"/>
+    <xacro:Gripper name="right" collider_type="$(arg collider)"/>
     <joint name="left_end_effector_mount_joint" type="fixed">
       <origin xyz="-0.083 0 0" rpy="${-PI/2} 0 ${PI}"/>
@@ -59,5 +59,5 @@
       <child link="left_gripper_base"/>
     </joint>
-    <xacro:Gripper name="left_gripper" collider_type="$(arg collider)"/>
+    <xacro:Gripper name="left" collider_type="$(arg collider)"/>
   </xacro:if>
   <xacro:if value="${selected_gripper_type == 'galbot_gripper'}">

File: galbot_foxtrot_description/urdf/galbot_foxtrot_hitbot.urdf (robot description, URDF)
Before this commit: robot galbot_one_foxtrot, 58 links, 57 joints
Links:
- link left_gripper_base: geometry collision mesh filename=package://hitbot_description/meshes/Z-EFG-100/collision/bas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; visual mesh filename=package://hitbot_description/meshes/Z-EFG-100/visual/base.g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
- link left_gripper_link1: geometry collision mesh filename=package://hitbot_description/meshes/Z-EFG-100/collision/gri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; visual mesh filename=package://hitbot_description/meshes/Z-EFG-100/visual/link1.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
- link left_gripper_link2: geometry collision mesh filename=package://hitbot_description/meshes/Z-EFG-100/collision/gri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; visual mesh filename=package://hitbot_description/meshes/Z-EFG-100/visual/link2.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
- link left_gripper_link3: geometry collision mesh filename=package://hitbot_description/meshes/Z-EFG-100/collision/gri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; visual mesh filename=package://hitbot_description/meshes/Z-EFG-100/visual/link3.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
- link left_gripper_link4: geometry collision mesh filename=package://hitbot_description/meshes/Z-EFG-100/collision/gri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; visual mesh filename=package://hitbot_description/meshes/Z-EFG-100/visual/link4.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
- link left_gripper_link5: geometry collision mesh filename=package://hitbot_description/meshes/Z-EFG-100/collision/gri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; visual mesh filename=package://hitbot_description/meshes/Z-EFG-100/visual/link5.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
- link left_gripper_link6: geometry collision mesh filename=package://hitbot_description/meshes/Z-EFG-100/collision/gri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; visual mesh filename=package://hitbot_description/meshes/Z-EFG-100/visual/link6.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
- link right_gripper_base: geometry collision mesh filename=package://hitbot_description/meshes/Z-EFG-100/collision/bas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; visual mesh filename=package://hitbot_description/meshes/Z-EFG-100/visual/base.g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
- link right_gripper_link1: geometry collision mesh filename=package://hitbot_description/meshes/Z-EFG-100/collision/gri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; visual mesh filename=package://hitbot_description/meshes/Z-EFG-100/visual/link1.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
- link right_gripper_link2: geometry collision mesh filename=package://hitbot_description/meshes/Z-EFG-100/collision/gri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; visual mesh filename=package://hitbot_description/meshes/Z-EFG-100/visual/link2.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
- link right_gripper_link3: geometry collision mesh filename=package://hitbot_description/meshes/Z-EFG-100/collision/gri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; visual mesh filename=package://hitbot_description/meshes/Z-EFG-100/visual/link3.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
- link right_gripper_link4: geometry collision mesh filename=package://hitbot_description/meshes/Z-EFG-100/collision/gri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; visual mesh filename=package://hitbot_description/meshes/Z-EFG-100/visual/link4.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
- link right_gripper_link5: geometry collision mesh filename=package://hitbot_description/meshes/Z-EFG-100/collision/gri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; visual mesh filename=package://hitbot_description/meshes/Z-EFG-100/visual/link5.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
- link right_gripper_link6: geometry collision mesh filename=package://hitbot_description/meshes/Z-EFG-100/collision/gri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; visual mesh filename=package://hitbot_description/meshes/Z-EFG-100/visual/link6.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

File: galbot_foxtrot_description/xacro/robot.xacro (robot description, xacro)
@@ -49,5 +49,5 @@
 			<child link="right_gripper_base"/>
 		</joint>
-		<xacro:Gripper name="right_gripper"/>
+		<xacro:Gripper name="right"/>
 	</xacro:if>
 	<xacro:Arm name="left" camera="$(arg arm_camera)"/>
@@ -66,5 +66,5 @@
 			<child link="left_gripper_base"/>
 		</joint>
-		<xacro:Gripper name="left_gripper"/>
+		<xacro:Gripper name="left"/>
 	</xacro:if>
 </robot>

File: galbot_golf_description/urdf/galbot_golf_hitbot.urdf (robot description, URDF)
Before this commit: robot galbot_one_golf, 60 links, 59 joints
Links:
- link left_gripper_base: geometry collision mesh filename=package://hitbot_description/meshes/Z-EFG-100/collision/bas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; visual mesh filename=package://hitbot_description/meshes/Z-EFG-100/visual/base.g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
- link left_gripper_link1: geometry collision mesh filename=package://hitbot_description/meshes/Z-EFG-100/collision/gri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; visual mesh filename=package://hitbot_description/meshes/Z-EFG-100/visual/link1.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
- link left_gripper_link2: geometry collision mesh filename=package://hitbot_description/meshes/Z-EFG-100/collision/gri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; visual mesh filename=package://hitbot_description/meshes/Z-EFG-100/visual/link2.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
- link left_gripper_link3: geometry collision mesh filename=package://hitbot_description/meshes/Z-EFG-100/collision/gri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; visual mesh filename=package://hitbot_description/meshes/Z-EFG-100/visual/link3.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
- link left_gripper_link4: geometry collision mesh filename=package://hitbot_description/meshes/Z-EFG-100/collision/gri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; visual mesh filename=package://hitbot_description/meshes/Z-EFG-100/visual/link4.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
- link left_gripper_link5: geometry collision mesh filename=package://hitbot_description/meshes/Z-EFG-100/collision/gri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; visual mesh filename=package://hitbot_description/meshes/Z-EFG-100/visual/link5.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
- link left_gripper_link6: geometry collision mesh filename=package://hitbot_description/meshes/Z-EFG-100/collision/gri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; visual mesh filename=package://hitbot_description/meshes/Z-EFG-100/visual/link6.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
- link right_gripper_base: geometry collision mesh filename=package://hitbot_description/meshes/Z-EFG-100/collision/bas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; visual mesh filename=package://hitbot_description/meshes/Z-EFG-100/visual/base.g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
- link right_gripper_link1: geometry collision mesh filename=package://hitbot_description/meshes/Z-EFG-100/collision/gri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; visual mesh filename=package://hitbot_description/meshes/Z-EFG-100/visual/link1.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
- link right_gripper_link2: geometry collision mesh filename=package://hitbot_description/meshes/Z-EFG-100/collision/gri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; visual mesh filename=package://hitbot_description/meshes/Z-EFG-100/visual/link2.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
- link right_gripper_link3: geometry collision mesh filename=package://hitbot_description/meshes/Z-EFG-100/collision/gri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; visual mesh filename=package://hitbot_description/meshes/Z-EFG-100/visual/link3.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
- link right_gripper_link4: geometry collision mesh filename=package://hitbot_description/meshes/Z-EFG-100/collision/gri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; visual mesh filename=package://hitbot_description/meshes/Z-EFG-100/visual/link4.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
- link right_gripper_link5: geometry collision mesh filename=package://hitbot_description/meshes/Z-EFG-100/collision/gri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; visual mesh filename=package://hitbot_description/meshes/Z-EFG-100/visual/link5.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
- link right_gripper_link6: geometry collision mesh filename=package://hitbot_description/meshes/Z-EFG-100/collision/gri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; visual mesh filename=package://hitbot_description/meshes/Z-EFG-100/visual/link6.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

File: galbot_golf_description/xacro/robot.xacro (robot description, xacro)
@@ -59,5 +59,5 @@
 			<child link="right_gripper_base"/>
 		</joint>
-		<xacro:Gripper name="right_gripper" collider_type="$(arg collider)"/>
+		<xacro:Gripper name="right" collider_type="$(arg collider)"/>
 	</xacro:if>
 	<joint name="left_arm_joint" type="fixed">
@@ -80,5 +80,5 @@
 			<child link="left_gripper_base"/>
 		</joint>
-		<xacro:Gripper name="left_gripper" collider_type="$(arg collider)"/>
+		<xacro:Gripper name="left" collider_type="$(arg collider)"/>
 	</xacro:if>
 </robot>

File: galbot_one_description/urdf/galbot_one.urdf (robot description, URDF)
Before this commit: robot galbot_one, 62 links, 61 joints
Links:
- link left_gripper_base: geometry collision mesh filename=package://hitbot_description/meshes/Z-EFG-100/collision/bas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; visual mesh filename=package://hitbot_description/meshes/Z-EFG-100/visual/base.g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
- link left_gripper_link1: geometry collision mesh filename=package://hitbot_description/meshes/Z-EFG-100/collision/gri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; visual mesh filename=package://hitbot_description/meshes/Z-EFG-100/visual/link1.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
- link left_gripper_link2: geometry collision mesh filename=package://hitbot_description/meshes/Z-EFG-100/collision/gri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; visual mesh filename=package://hitbot_description/meshes/Z-EFG-100/visual/link2.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
- link left_gripper_link3: geometry collision mesh filename=package://hitbot_description/meshes/Z-EFG-100/collision/gri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; visual mesh filename=package://hitbot_description/meshes/Z-EFG-100/visual/link3.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
- link left_gripper_link4: geometry collision mesh filename=package://hitbot_description/meshes/Z-EFG-100/collision/gri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; visual mesh filename=package://hitbot_description/meshes/Z-EFG-100/visual/link4.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
- link left_gripper_link5: geometry collision mesh filename=package://hitbot_description/meshes/Z-EFG-100/collision/gri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; visual mesh filename=package://hitbot_description/meshes/Z-EFG-100/visual/link5.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
- link left_gripper_link6: geometry collision mesh filename=package://hitbot_description/meshes/Z-EFG-100/collision/gri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; visual mesh filename=package://hitbot_description/meshes/Z-EFG-100/visual/link6.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
- link right_gripper_base: geometry collision mesh filename=package://hitbot_description/meshes/Z-EFG-100/collision/bas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; visual mesh filename=package://hitbot_description/meshes/Z-EFG-100/visual/base.g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
- link right_gripper_link1: geometry collision mesh filename=package://hitbot_description/meshes/Z-EFG-100/collision/gri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; visual mesh filename=package://hitbot_description/meshes/Z-EFG-100/visual/link1.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
- link right_gripper_link2: geometry collision mesh filename=package://hitbot_description/meshes/Z-EFG-100/collision/gri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; visual mesh filename=package://hitbot_description/meshes/Z-EFG-100/visual/link2.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
- link right_gripper_link3: geometry collision mesh filename=package://hitbot_description/meshes/Z-EFG-100/collision/gri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; visual mesh filename=package://hitbot_description/meshes/Z-EFG-100/visual/link3.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
- link right_gripper_link4: geometry collision mesh filename=package://hitbot_description/meshes/Z-EFG-100/collision/gri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; visual mesh filename=package://hitbot_description/meshes/Z-EFG-100/visual/link4.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
- link right_gripper_link5: geometry collision mesh filename=package://hitbot_description/meshes/Z-EFG-100/collision/gri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; visual mesh filename=package://hitbot_description/meshes/Z-EFG-100/visual/link5.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
- link right_gripper_link6: geometry collision mesh filename=package://hitbot_description/meshes/Z-EFG-100/collision/gri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; visual mesh filename=package://hitbot_description/meshes/Z-EFG-100/visual/link6.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

File: galbot_one_description/xacro/robot.xacro (robot description, xacro)
@@ -53,5 +53,5 @@
       <child link="right_gripper_base"/>
     </joint>
-    <xacro:Gripper name="right_gripper" collider_type="$(arg collider)"/>
+    <xacro:Gripper name="right" collider_type="$(arg collider)"/>
     <joint name="left_end_effector_mount_joint" type="fixed">
       <origin xyz="0 0 0.084525" rpy="0 ${-PI/2} ${PI}"/>
@@ -59,5 +59,5 @@
       <child link="left_gripper_base"/>
     </joint>
-    <xacro:Gripper name="left_gripper" collider_type="$(arg collider)"/>
+    <xacro:Gripper name="left" collider_type="$(arg collider)"/>
   </xacro:if>
   <xacro:if value="${selected_gripper_type == 'galbot_gripper'}">
