Commit message: 更新hitbot的include路径

File: galbot_charlie_description/urdf/galbot_charlie.urdf (robot description, URDF)
Before this commit: robot galbot_charlie, 64 links, 63 joints
Links:
- link left_gripper_base: geometry collision mesh filename=package://hitbot_description/meshes/Z-EFG-100/base.glb; visual mesh filename=package://hitbot_description/meshes/Z-EFG-100/base.glb
- link left_gripper_link1: geometry collision mesh filename=package://hitbot_description/meshes/Z-EFG-100/link1.glb; visual mesh filename=package://hitbot_description/meshes/Z-EFG-100/link1.glb
- link left_gripper_link2: geometry collision mesh filename=package://hitbot_description/meshes/Z-EFG-100/link2.glb; visual mesh filename=package://hitbot_description/meshes/Z-EFG-100/link2.glb
- link left_gripper_link3: geometry collision mesh filename=package://hitbot_description/meshes/Z-EFG-100/link3.glb; visual mesh filename=package://hitbot_description/meshes/Z-EFG-100/link3.glb
- link left_gripper_link4: geometry collision mesh filename=package://hitbot_description/meshes/Z-EFG-100/link4.glb; visual mesh filename=package://hitbot_description/meshes/Z-EFG-100/link4.glb
- link left_gripper_link5: geometry collision mesh filename=package://hitbot_description/meshes/Z-EFG-100/link5.glb; visual mesh filename=package://hitbot_description/meshes/Z-EFG-100/link5.glb
- link left_gripper_link6: geometry collision mesh filename=package://hitbot_description/meshes/Z-EFG-100/link6.glb; visual mesh filename=package://hitbot_description/meshes/Z-EFG-100/link6.glb
- link right_gripper_base: geometry collision mesh filename=package://hitbot_description/meshes/Z-EFG-100/base.glb; visual mesh filename=package://hitbot_description/meshes/Z-EFG-100/base.glb
- link right_gripper_link1: geometry collision mesh filename=package://hitbot_description/meshes/Z-EFG-100/link1.glb; visual mesh filename=package://hitbot_description/meshes/Z-EFG-100/link1.glb
- link right_gripper_link2: geometry collision mesh filename=package://hitbot_description/meshes/Z-EFG-100/link2.glb; visual mesh filename=package://hitbot_description/meshes/Z-EFG-100/link2.glb
- link right_gripper_link3: geometry collision mesh filename=package://hitbot_description/meshes/Z-EFG-100/link3.glb; visual mesh filename=package://hitbot_description/meshes/Z-EFG-100/link3.glb
- link right_gripper_link4: geometry collision mesh filename=package://hitbot_description/meshes/Z-EFG-100/link4.glb; visual mesh filename=package://hitbot_description/meshes/Z-EFG-100/link4.glb
- link right_gripper_link5: geometry collision mesh filename=package://hitbot_description/meshes/Z-EFG-100/link5.glb; visual mesh filename=package://hitbot_description/meshes/Z-EFG-100/link5.glb
- link right_gripper_link6: geometry collision mesh filename=package://hitbot_description/meshes/Z-EFG-100/link6.glb; visual mesh filename=package://hitbot_description/meshes/Z-EFG-100/link6.glb

File: galbot_foxtrot_description/urdf/galbot_foxtrot_hitbot.urdf (robot description, URDF)
Before this commit: robot galbot_one_foxtrot, 58 links, 57 joints
Links:
- link left_gripper_base: geometry collision mesh filename=package://hitbot_description/meshes/Z-EFG-100/base.glb; visual mesh filename=package://hitbot_description/meshes/Z-EFG-100/base.glb
- link left_gripper_link1: geometry collision mesh filename=package://hitbot_description/meshes/Z-EFG-100/link1.glb; visual mesh filename=package://hitbot_description/meshes/Z-EFG-100/link1.glb
- link left_gripper_link2: geometry collision mesh filename=package://hitbot_description/meshes/Z-EFG-100/link2.glb; visual mesh filename=package://hitbot_description/meshes/Z-EFG-100/link2.glb
- link left_gripper_link3: geometry collision mesh filename=package://hitbot_description/meshes/Z-EFG-100/link3.glb; visual mesh filename=package://hitbot_description/meshes/Z-EFG-100/link3.glb
- link left_gripper_link4: geometry collision mesh filename=package://hitbot_description/meshes/Z-EFG-100/link4.glb; visual mesh filename=package://hitbot_description/meshes/Z-EFG-100/link4.glb
- link left_gripper_link5: geometry collision mesh filename=package://hitbot_description/meshes/Z-EFG-100/link5.glb; visual mesh filename=package://hitbot_description/meshes/Z-EFG-100/link5.glb
- link left_gripper_link6: geometry collision mesh filename=package://hitbot_description/meshes/Z-EFG-100/link6.glb; visual mesh filename=package://hitbot_description/meshes/Z-EFG-100/link6.glb
- link right_gripper_base: geometry collision mesh filename=package://hitbot_description/meshes/Z-EFG-100/base.glb; visual mesh filename=package://hitbot_description/meshes/Z-EFG-100/base.glb
- link right_gripper_link1: geometry collision mesh filename=package://hitbot_description/meshes/Z-EFG-100/link1.glb; visual mesh filename=package://hitbot_description/meshes/Z-EFG-100/link1.glb
- link right_gripper_link2: geometry collision mesh filename=package://hitbot_description/meshes/Z-EFG-100/link2.glb; visual mesh filename=package://hitbot_description/meshes/Z-EFG-100/link2.glb
- link right_gripper_link3: geometry collision mesh filename=package://hitbot_description/meshes/Z-EFG-100/link3.glb; visual mesh filename=package://hitbot_description/meshes/Z-EFG-100/link3.glb
- link right_gripper_link4: geometry collision mesh filename=package://hitbot_description/meshes/Z-EFG-100/link4.glb; visual mesh filename=package://hitbot_description/meshes/Z-EFG-100/link4.glb
- link right_gripper_link5: geometry collision mesh filename=package://hitbot_description/meshes/Z-EFG-100/link5.glb; visual mesh filename=package://hitbot_description/meshes/Z-EFG-100/link5.glb
- link right_gripper_link6: geometry collision mesh filename=package://hitbot_description/meshes/Z-EFG-100/link6.glb; visual mesh filename=package://hitbot_description/meshes/Z-EFG-100/link6.glb

File: galbot_golf_description/urdf/galbot_golf_hitbot.urdf (robot description, URDF)
Before this commit: robot galbot_one_golf, 60 links, 59 joints
Links:
- link left_gripper_base: geometry collision mesh filename=package://hitbot_description/meshes/Z-EFG-100/base.glb; visual mesh filename=package://hitbot_description/meshes/Z-EFG-100/base.glb
- link left_gripper_link1: geometry collision mesh filename=package://hitbot_description/meshes/Z-EFG-100/link1.glb; visual mesh filename=package://hitbot_description/meshes/Z-EFG-100/link1.glb
- link left_gripper_link2: geometry collision mesh filename=package://hitbot_description/meshes/Z-EFG-100/link2.glb; visual mesh filename=package://hitbot_description/meshes/Z-EFG-100/link2.glb
- link left_gripper_link3: geometry collision mesh filename=package://hitbot_description/meshes/Z-EFG-100/link3.glb; visual mesh filename=package://hitbot_description/meshes/Z-EFG-100/link3.glb
- link left_gripper_link4: geometry collision mesh filename=package://hitbot_description/meshes/Z-EFG-100/link4.glb; visual mesh filename=package://hitbot_description/meshes/Z-EFG-100/link4.glb
- link left_gripper_link5: geometry collision mesh filename=package://hitbot_description/meshes/Z-EFG-100/link5.glb; visual mesh filename=package://hitbot_description/meshes/Z-EFG-100/link5.glb
- link left_gripper_link6: geometry collision mesh filename=package://hitbot_description/meshes/Z-EFG-100/link6.glb; visual mesh filename=package://hitbot_description/meshes/Z-EFG-100/link6.glb
- link right_gripper_base: geometry collision mesh filename=package://hitbot_description/meshes/Z-EFG-100/base.glb; visual mesh filename=package://hitbot_description/meshes/Z-EFG-100/base.glb
- link right_gripper_link1: geometry collision mesh filename=package://hitbot_description/meshes/Z-EFG-100/link1.glb; visual mesh filename=package://hitbot_description/meshes/Z-EFG-100/link1.glb
- link right_gripper_link2: geometry collision mesh filename=package://hitbot_description/meshes/Z-EFG-100/link2.glb; visual mesh filename=package://hitbot_description/meshes/Z-EFG-100/link2.glb
- link right_gripper_link3: geometry collision mesh filename=package://hitbot_description/meshes/Z-EFG-100/link3.glb; visual mesh filename=package://hitbot_description/meshes/Z-EFG-100/link3.glb
- link right_gripper_link4: geometry collision mesh filename=package://hitbot_description/meshes/Z-EFG-100/link4.glb; visual mesh filename=package://hitbot_description/meshes/Z-EFG-100/link4.glb
- link right_gripper_link5: geometry collision mesh filename=package://hitbot_description/meshes/Z-EFG-100/link5.glb; visual mesh filename=package://hitbot_description/meshes/Z-EFG-100/link5.glb
- link right_gripper_link6: geometry collision mesh filename=package://hitbot_description/meshes/Z-EFG-100/link6.glb; visual mesh filename=package://hitbot_description/meshes/Z-EFG-100/link6.glb

File: galbot_one_description/urdf/galbot_one.urdf (robot description, URDF)
Before this commit: robot galbot_one, 62 links, 61 joints
Links:
- link left_gripper_base: geometry collision mesh filename=package://hitbot_description/meshes/Z-EFG-100/base.glb; visual mesh filename=package://hitbot_description/meshes/Z-EFG-100/base.glb
- link left_gripper_link1: geometry collision mesh filename=package://hitbot_description/meshes/Z-EFG-100/link1.glb; visual mesh filename=package://hitbot_description/meshes/Z-EFG-100/link1.glb
- link left_gripper_link2: geometry collision mesh filename=package://hitbot_description/meshes/Z-EFG-100/link2.glb; visual mesh filename=package://hitbot_description/meshes/Z-EFG-100/link2.glb
- link left_gripper_link3: geometry collision mesh filename=package://hitbot_description/meshes/Z-EFG-100/link3.glb; visual mesh filename=package://hitbot_description/meshes/Z-EFG-100/link3.glb
- link left_gripper_link4: geometry collision mesh filename=package://hitbot_description/meshes/Z-EFG-100/link4.glb; visual mesh filename=package://hitbot_description/meshes/Z-EFG-100/link4.glb
- link left_gripper_link5: geometry collision mesh filename=package://hitbot_description/meshes/Z-EFG-100/link5.glb; visual mesh filename=package://hitbot_description/meshes/Z-EFG-100/link5.glb
- link left_gripper_link6: geometry collision mesh filename=package://hitbot_description/meshes/Z-EFG-100/link6.glb; visual mesh filename=package://hitbot_description/meshes/Z-EFG-100/link6.glb
- link right_gripper_base: geometry collision mesh filename=package://hitbot_description/meshes/Z-EFG-100/base.glb; visual mesh filename=package://hitbot_description/meshes/Z-EFG-100/base.glb
- link right_gripper_link1: geometry collision mesh filename=package://hitbot_description/meshes/Z-EFG-100/link1.glb; visual mesh filename=package://hitbot_description/meshes/Z-EFG-100/link1.glb
- link right_gripper_link2: geometry collision mesh filename=package://hitbot_description/meshes/Z-EFG-100/link2.glb; visual mesh filename=package://hitbot_description/meshes/Z-EFG-100/link2.glb
- link right_gripper_link3: geometry collision mesh filename=package://hitbot_description/meshes/Z-EFG-100/link3.glb; visual mesh filename=package://hitbot_description/meshes/Z-EFG-100/link3.glb
- link right_gripper_link4: geometry collision mesh filename=package://hitbot_description/meshes/Z-EFG-100/link4.glb; visual mesh filename=package://hitbot_description/meshes/Z-EFG-100/link4.glb
- link right_gripper_link5: geometry collision mesh filename=package://hitbot_description/meshes/Z-EFG-100/link5.glb; visual mesh filename=package://hitbot_description/meshes/Z-EFG-100/link5.glb
- link right_gripper_link6: geometry collision mesh filename=package://hitbot_description/meshes/Z-EFG-100/link6.glb; visual mesh filename=package://hitbot_description/meshes/Z-EFG-100/link6.glb

Commit message: move to mid360 glb

File: galbot_charlie_description/urdf/galbot_charlie.urdf (robot description, URDF)
Before this commit: robot galbot_charlie, 64 links, 63 joints
Links:
- link chassis_lidar: geometry visual mesh filename=package://sensor_models/meshes/livox/mid360.glb

File: galbot_charlie_description/urdf/galbot_charlie_galbot_gripper.urdf (robot description, URDF)
Before this commit: robot galbot_charlie, 66 links, 65 joints
Links:
- link chassis_lidar: geometry visual mesh filename=package://sensor_models/meshes/livox/mid360.glb

File: galbot_foxtrot_description/urdf/galbot_foxtrot.urdf (robot description, URDF)
Before this commit: robot galbot_one_foxtrot, 60 links, 59 joints
Links:
- link chassis_lidar: geometry visual mesh filename=package://sensor_models/meshes/livox/mid360.glb

File: galbot_foxtrot_description/urdf/galbot_foxtrot_hitbot.urdf (robot description, URDF)
Before this commit: robot galbot_one_foxtrot, 58 links, 57 joints
Links:
- link chassis_lidar: geometry visual mesh filename=package://sensor_models/meshes/livox/mid360.glb

File: galbot_foxtrot_description/xacro/components/chassis.xacro (robot description, xacro)
@@ -91,5 +91,5 @@
       <visual>
         <geometry>
-          <mesh filename="file://$(find sensor_models)/meshes/mid360/mid360.obj"/>
+          <mesh filename="file://$(find sensor_models)/meshes/livox/mid360.glb"/>
         </geometry>
       </visual>

File: galbot_golf_description/urdf/galbot_golf.urdf (robot description, URDF)
Before this commit: robot galbot_one_golf, 62 links, 61 joints
Links:
- link chassis_lidar: geometry visual mesh filename=package://sensor_models/meshes/livox/mid360.glb

File: galbot_golf_description/urdf/galbot_golf_hitbot.urdf (robot description, URDF)
Before this commit: robot galbot_one_golf, 60 links, 59 joints
Links:
- link chassis_lidar: geometry visual mesh filename=package://sensor_models/meshes/livox/mid360.glb

File: galbot_one_description/urdf/galbot_one.urdf (robot description, URDF)
Before this commit: robot galbot_one, 62 links, 61 joints
Links:
- link chassis_lidar: geometry visual mesh filename=package://sensor_models/meshes/livox/mid360.glb

File: galbot_one_description/urdf/galbot_one_galbot_gripper.urdf (robot description, URDF)
Before this commit: robot galbot_one, 64 links, 63 joints
Links:
- link chassis_lidar: geometry visual mesh filename=package://sensor_models/meshes/livox/mid360.glb

File: galbot_one_description/xacro/components/chassis.xacro (robot description, xacro)
@@ -85,5 +85,5 @@
       <visual>
         <geometry>
-          <mesh filename="file://$(find sensor_models)/meshes/mid360/mid360.obj"/>
+          <mesh filename="file://$(find sensor_models)/meshes/livox/mid360.glb"/>
         </geometry>
       </visual>

File: galbot_s1_description/urdf/galbot_s1.urdf (robot description, URDF)
Before this commit: robot galbot_s1, 60 links, 59 joints
Links:
- link chassis_lidar: geometry visual mesh filename=package://sensor_models/meshes/livox/mid360.glb
- link column_lidar: geometry visual mesh filename=package://sensor_models/meshes/livox/mid360.glb
- link head_lidar: geometry visual mesh filename=package://sensor_models/meshes/livox/mid360.glb

File: galbot_s1_description/xacro/components/column.xacro (robot description, xacro)
@@ -39,5 +39,5 @@
 			<visual>
 				<geometry>
-					<mesh filename="file://$(find sensor_models)/meshes/mid360/mid360.obj"/>
+					<mesh filename="file://$(find sensor_models)/meshes/livox/mid360.glb"/>
 				</geometry>
 			</visual>

File: galbot_s1_description/xacro/components/omni_chassis.xacro (robot description, xacro)
@@ -254,5 +254,5 @@
 			<visual>
 				<geometry>
-					<mesh filename="file://$(find sensor_models)/meshes/mid360/mid360.obj"/>
+					<mesh filename="file://$(find sensor_models)/meshes/livox/mid360.glb"/>
 				</geometry>
 			</visual>

File: galbot_s1_description/xacro/components/torso.xacro (robot description, xacro)
@@ -160,5 +160,5 @@
 			<visual>
 				<geometry>
-					<mesh filename="file://$(find sensor_models)/meshes/mid360/mid360.obj"/>
+					<mesh filename="file://$(find sensor_models)/meshes/livox/mid360.glb"/>
 				</geometry>
 			</visual>
